Commit message: Use simple shapes by default, reflect for left and right hands

File: ros/sandia_hand_description/robots/sandia_hand_both.urdf.xacro (robot description, xacro)
@@ -4,5 +4,7 @@
        xmlns:xacro="http://playerstage.sourceforge.net/gazebo/xmlschema/#interface"
        name="humanoid" >
-  <include filename="$(find sandia_hand_description)/urdf/sandia_hand.urdf.xacro" />
+  <!-- Commenting out urdf with meshes, using simple collision shapes instead -->
+  <!--<include filename="$(find sandia_hand_description)/urdf/sandia_hand.urdf.xacro" />-->
+  <include filename="$(find sandia_hand_description)/urdf/sandia_hand_simple_shapes.urdf.xacro" />
   <link name="base">
     <inertial>
@@ -24,8 +26,8 @@
     </collision>
   </link>
-  <xacro:sandia_hand side="right" parent="base">
+  <xacro:sandia_hand side="right" parent="base" reflect="1">
     <origin xyz="0 0.2 0.5" rpy="0 -1.57079 0"/>
   </xacro:sandia_hand>
-  <xacro:sandia_hand side="left" parent="base">
+  <xacro:sandia_hand side="left" parent="base" reflect="-1">
     <origin xyz="0 -0.2 0.5" rpy="0 -1.57079 0"/>
   </xacro:sandia_hand>

File: ros/sandia_hand_description/robots/sandia_hand_left.urdf.xacro (robot description, xacro)
@@ -4,5 +4,7 @@
        xmlns:xacro="http://playerstage.sourceforge.net/gazebo/xmlschema/#interface"
        name="humanoid" >
-  <include filename="$(find sandia_hand_description)/urdf/sandia_hand.urdf.xacro" />
+  <!-- Commenting out urdf with meshes, using simple collision shapes instead -->
+  <!--<include filename="$(find sandia_hand_description)/urdf/sandia_hand.urdf.xacro" />-->
+  <include filename="$(find sandia_hand_description)/urdf/sandia_hand_simple_shapes.urdf.xacro" />
   <link name="base">
     <inertial>
@@ -24,5 +26,5 @@
     </collision>
   </link>
-  <xacro:sandia_hand side="left" parent="base">
+  <xacro:sandia_hand side="left" parent="base" reflect="-1">
     <origin xyz="0 0 0.5" rpy="0 -1.57079 0"/>
   </xacro:sandia_hand>

File: ros/sandia_hand_description/robots/sandia_hand_right.urdf.xacro (robot description, xacro)
@@ -4,5 +4,7 @@
        xmlns:xacro="http://playerstage.sourceforge.net/gazebo/xmlschema/#interface"
        name="humanoid" >
-  <include filename="$(find sandia_hand_description)/urdf/sandia_hand.urdf.xacro" />
+  <!-- Commenting out urdf with meshes, using simple collision shapes instead -->
+  <!--<include filename="$(find sandia_hand_description)/urdf/sandia_hand.urdf.xacro" />-->
+  <include filename="$(find sandia_hand_description)/urdf/sandia_hand_simple_shapes.urdf.xacro" />
   <link name="base">
     <inertial>
@@ -24,5 +26,5 @@
     </collision>
   </link>
-  <xacro:sandia_hand side="right" parent="base">
+  <xacro:sandia_hand side="right" parent="base" reflect="1">
     <origin xyz="0 0 0.5" rpy="0 -1.57079 0"/>
   </xacro:sandia_hand>

File: ros/sandia_hand_description/urdf/sandia_hand_simple_shapes.urdf.xacro (robot description, xacro)
@@ -4,5 +4,6 @@
   <include filename="$(find sandia_hand_description)/urdf/sandia_hand.gazebo.xacro" />
   <include filename="$(find sandia_hand_description)/urdf/sandia_hand.transmission.xacro" />
-  <xacro:macro name="finger" params="idx x y z r p yaw side">
+  <xacro:property name="M_pi" value="3.1415926535897931" />
+  <xacro:macro name="finger" params="idx x y z r p yaw side reflect">
     <link name="${side}_f${idx}_base">
       <origin xyz="0 0 0" rpy="0 0 0"/>
@@ -36,5 +37,5 @@
       </collision>
       <collision>
-        <origin xyz="0.011 0 0.003" rpy="1.57 0 0"/>
+        <origin xyz="0.011 0 0.003" rpy="${M_pi/2} 0 0"/>
         <geometry>
           <cylinder radius="0.01" length="0.023" />
@@ -53,5 +54,5 @@
       </visual>
       <visual>
-        <origin xyz="0.011 0 0.003" rpy="1.57 0 0"/>
+        <origin xyz="0.011 0 0.003" rpy="${M_pi/2} 0 0"/>
         <geometry>
           <cylinder radius="0.01" length="0.023" />
@@ -91,5 +92,5 @@
       <!-- begin simple shape approximation of f1 -->
       <collision>
-        <origin xyz="0.024 0 0" rpy="0 1.57 0"/>
+        <origin xyz="0.024 0 0" rpy="0 ${M_pi/2} 0"/>
         <geometry>
           <cylinder radius="0.01" length="0.067" />
@@ -99,5 +100,5 @@
       <!-- begin visual shape approximation of f1 -->
       <visual>
-        <origin xyz="0.024 0 0" rpy="0 1.57 0"/>
+        <origin xyz="0.024 0 0" rpy="0 ${M_pi/2} 0"/>
         <geometry>
           <cylinder radius="0.01" length="0.067" />
@@ -145,5 +146,5 @@
       <!-- begin simple shape approximation of f2 -->
       <collision>
-        <origin xyz="0.024 0 0" rpy="0 1.57 0"/>
+        <origin xyz="0.024 0 0" rpy="0 ${M_pi/2} 0"/>
         <geometry>
           <cylinder radius="0.009" length="0.057" />
@@ -159,5 +160,5 @@
       <!-- begin visual shape approximation of f2 -->
       <visual>
-        <origin xyz="0.024 0 0" rpy="0 1.57 0"/>
+        <origin xyz="0.024 0 0" rpy="0 ${M_pi/2} 0"/>
         <geometry>
           <cylinder radius="0.009" length="0.057" />
@@ -210,8 +211,8 @@
     </joint>
     <joint name="${side}_f${idx}_j0" type="revolute">
-      <axis xyz="0 0 1"/>
+      <axis xyz="0 0 ${reflect}"/>
       <parent link="${side}_f${idx}_base"/>
       <child link="${side}_f${idx}_0"/>
-      <limit lower="-1.57079" upper="1.57079" effort="1" velocity="1"/>
+      <limit lower="-${M_pi/2}" upper="${M_pi/2}" effort="1" velocity="1"/>
       <safety_controller soft_lower_limit="${-1.57079-10.0}" soft_upper_limit="${1.57079+10.0}" k_position="1000.0" k_velocity="1000.0"/>
       <dynamics damping="0.1"/>
@@ -222,8 +223,8 @@
       <parent link="${side}_f${idx}_0"/>
       <child link="${side}_f${idx}_1"/>
-      <limit lower="-1.57079" upper="1.57079" effort="1" velocity="1"/>
+      <limit lower="-${M_pi/2}" upper="${M_pi/2}" effort="1" velocity="1"/>
       <safety_controller soft_lower_limit="${-1.57079-10.0}" soft_upper_limit="${1.57079+10.0}" k_position="1000.0" k_velocity="1000.0"/>
       <dynamics damping="0.1"/>
-      <origin xyz="0.028 0 0" rpy="1.57079 0 0"/>
+      <origin xyz="0.028 0 0" rpy="${M_pi/2} 0 0"/>
     </joint>
     <joint name="${side}_f${idx}_j2" type="revolute">
@@ -234,5 +235,5 @@
       <safety_controller soft_lower_limit="${-1.57079-10.0}" soft_upper_limit="${1.57079+10.0}" k_position="1000.0" k_velocity="1000.0"/>
       <dynamics damping="0.1"/>
-      <limit lower="-1.57079" upper="1.57079" effort="1" velocity="1"/>
+      <limit lower="-${M_pi/2}" upper="${M_pi/2}" effort="1" velocity="1"/>
     </joint>
     <joint name="${side}_f${idx}_fixed_accel" type="fixed">
@@ -244,14 +245,14 @@
       <parent link="${side}_f${idx}_1"/>
       <child link="${side}_f${idx}_1_accel"/>
-      <origin xyz="0.03 0 0" rpy="-1.5709 0 0"/>
+      <origin xyz="0.03 0 0" rpy="-${M_pi/2} 0 0"/>
     </joint>
     <joint name="${side}_f${idx}_2_accel" type="fixed">
       <parent link="${side}_f${idx}_2"/>
       <child link="${side}_f${idx}_2_accel"/>
-      <origin xyz="0.04 0 0" rpy="-1.5709 0 0"/>
+      <origin xyz="0.04 0 0" rpy="-${M_pi/2} 0 0"/>
     </joint>
     <xacro:finger_transmission side="${side}" idx="${idx}" x="${x}" y="${y}" z="${z}" r="${r}" p="${p}" yaw="${yaw}"/>
   </xacro:macro>
-  <xacro:macro name="sandia_hand" params="side parent *origin">
+  <xacro:macro name="sandia_hand" params="side parent reflect *origin">
     <link name="${side}_palm">
       <origin xyz="0 0 0" rpy="0 0 0"/>
@@ -263,5 +264,5 @@
       <!-- begin simple shape approximation of palm -->
       <collision>
-        <origin xyz="0.069 0.016 0.038" rpy="0 1.57 -0.9"/>
+        <origin xyz="0.069 ${0.016 * reflect} 0.038" rpy="0 ${M_pi/2} ${-0.9 * reflect}"/>
         <geometry>
           <cylinder radius="0.013" length="0.100" />
@@ -269,5 +270,5 @@
       </collision>
       <collision>
-        <origin xyz="0.064 0.008 0.021" rpy="0.41 0 -0.9"/>
+        <origin xyz="0.064 $(0.008 * reflect} 0.021" rpy="0.41 0 ${-0.9 * reflect}"/>
         <geometry>
           <box size="0.09 .035 .05" />
@@ -275,5 +276,5 @@
       </collision>
       <collision>
-        <origin xyz="0.02 0 -0.005" rpy="0 1.57 0"/>
+        <origin xyz="0.02 0 -0.005" rpy="0 ${M_pi/2} 0"/>
         <geometry>
           <cylinder radius="0.038" length="0.05" />
@@ -281,23 +282,23 @@
       </collision>
       <collision>
-        <origin xyz="0.11 -0.01 -0.005" rpy="0 0 0.37"/>
-        <geometry>
-          <box size="0.09 .03 .06" />
-        </geometry>
-      </collision>
-      <collision>
-        <origin xyz="0.09 0.02 -0.005" rpy="0 0 0.37"/>
-        <geometry>
-          <box size="0.09 .03 .06" />
-        </geometry>
-      </collision>
-      <collision>
-        <origin xyz="0.060 0.050 -0.005" rpy="0 0 0.37"/>
-        <geometry>
-          <box size="0.09 .03 .06" />
-        </geometry>
-      </collision>
-      <collision>
-        <origin xyz="0.044 -0.04 -0.005" rpy="0 0 0.79"/>
+        <origin xyz="0.11 ${-0.01*reflect} -0.005" rpy="0 0 ${0.37*reflect}"/>
+        <geometry>
+          <box size="0.09 .03 .06" />
+        </geometry>
+      </collision>
+      <collision>
+        <origin xyz="0.09 ${0.02*reflect} -0.005" rpy="0 0 ${0.37*reflect}"/>
+        <geometry>
+          <box size="0.09 .03 .06" />
+        </geometry>
+      </collision>
+      <collision>
+        <origin xyz="0.060 ${0.050*reflect} -0.005" rpy="0 0 ${0.37*reflect}"/>
+        <geometry>
+          <box size="0.09 .03 .06" />
+        </geometry>
+      </collision>
+      <collision>
+        <origin xyz="0.044 ${-0.04*reflect} -0.005" rpy="0 0 ${0.79*reflect}"/>
         <geometry>
           <box size="0.09 .03 .06" />
@@ -307,5 +308,5 @@
       <!-- begin visual shape approximation of palm -->
       <visual>
-        <origin xyz="0.069 0.016 0.038" rpy="0 1.57 -0.9"/>
+        <origin xyz="0.069 ${0.016*reflect} 0.038" rpy="0 ${M_pi/2} ${-0.9*reflect}"/>
         <geometry>
           <cylinder radius="0.013" length="0.100" />
@@ -316,5 +317,5 @@
       </visual>
       <visual>
-        <origin xyz="0.064 0.008 0.021" rpy="0.41 0 -0.9"/>
+        <origin xyz="0.064 ${0.008*reflect} 0.021" rpy="0.41 0 ${-0.9*reflect}"/>
         <geometry>
           <box size="0.09 .035 .05" />
@@ -325,5 +326,5 @@
       </visual>
       <visual>
-        <origin xyz="0.02 0 -0.005" rpy="0 1.57 0"/>
+        <origin xyz="0.02 0 -0.005" rpy="0 ${M_pi/2} 0"/>
         <geometry>
           <cylinder radius="0.038" length="0.05" />
@@ -334,32 +335,32 @@
       </visual>
       <visual>
-        <origin xyz="0.11 -0.01 -0.005" rpy="0 0 0.37"/>
-        <geometry>
-          <box size="0.09 .03 .06" />
-        </geometry>
-        <material name="${side}_sandia_hand_skin">
-          <color rgba="0.835 0.655 0.345 1.0"/>
-        </material>
-      </visual>
-      <visual>
-        <origin xyz="0.09 0.02 -0.005" rpy="0 0 0.37"/>
-        <geometry>
-          <box size="0.09 .03 .06" />
-        </geometry>
-        <material name="${side}_sandia_hand_skin">
-          <color rgba="0.835 0.655 0.345 1.0"/>
-        </material>
-      </visual>
-      <visual>
-        <origin xyz="0.060 0.050 -0.005" rpy="0 0 0.37"/>
-        <geometry>
-          <box size="0.09 .03 .06" />
-        </geometry>
-        <material name="${side}_sandia_hand_skin">
-          <color rgba="0.835 0.655 0.345 1.0"/>
-        </material>
-      </visual>
-      <visual>
-        <origin xyz="0.044 -0.04 -0.005" rpy="0 0 0.79"/>
+        <origin xyz="0.11 ${-0.01*reflect} -0.005" rpy="0 0 ${0.37*reflect}"/>
+        <geometry>
+          <box size="0.09 .03 .06" />
+        </geometry>
+        <material name="${side}_sandia_hand_skin">
+          <color rgba="0.835 0.655 0.345 1.0"/>
+        </material>
+      </visual>
+      <visual>
+        <origin xyz="0.09 ${0.02*reflect} -0.005" rpy="0 0 ${0.37*reflect}"/>
+        <geometry>
+          <box size="0.09 .03 .06" />
+        </geometry>
+        <material name="${side}_sandia_hand_skin">
+          <color rgba="0.835 0.655 0.345 1.0"/>
+        </material>
+      </visual>
+      <visual>
+        <origin xyz="0.060 ${0.050*reflect} -0.005" rpy="0 0 ${0.37*reflect}"/>
+        <geometry>
+          <box size="0.09 .03 .06" />
+        </geometry>
+        <material name="${side}_sandia_hand_skin">
+          <color rgba="0.835 0.655 0.345 1.0"/>
+        </material>
+      </visual>
+      <visual>
+        <origin xyz="0.044 ${-0.04*reflect} -0.005" rpy="0 0 ${0.79*reflect}"/>
         <geometry>
           <box size="0.09 .03 .06" />
@@ -395,8 +396,8 @@
       <insert_block name="origin" />
     </joint>
-    <xacro:finger side="${side}" idx="0" x="0.140" y="0.00000" z="0" r="0" p="0" yaw="0.3"/>
-    <xacro:finger side="${side}" idx="1" x="0.115" y="0.03122" z="0" r="0" p="0" yaw="0.3"/>
-    <xacro:finger side="${side}" idx="2" x="0.090" y="0.06245" z="0" r="0" p="0" yaw="0.3"/>
-    <xacro:finger side="${side}" idx="3" x="0.03995" y="-0.04383" z="0.014" r="0" p="-1.57079" yaw="-2.3562"/>
+    <xacro:finger side="${side}" idx="0" x="0.140" y="0.00000" z="0" r="0" p="0" yaw="${0.3*reflect}" reflect="${reflect}" />
+    <xacro:finger side="${side}" idx="1" x="0.115" y="${0.03122*reflect}" z="0" r="0" p="0" yaw="${0.3*reflect}" reflect="${reflect}" />
+    <xacro:finger side="${side}" idx="2" x="0.090" y="${0.06245*reflect}" z="0" r="0" p="0" yaw="${0.3*reflect}" reflect="${reflect}" />
+    <xacro:finger side="${side}" idx="3" x="0.03995" y="${-0.04383*reflect}" z="0.014" r="0" p="-${M_pi/2}" yaw="${-2.3562*reflect}" reflect="${reflect}" />
     <!-- not needed unless simulating the hand by itself
     <xacro:sandia_hand_gazebo side="${side}" />
