Commit message: try to fix camera topics for drcsim, without changing drcsim

File: ros/sandia_hand_description/robots/sandia_hand_both_on_box.urdf.xacro (robot description, xacro)
@@ -26,8 +26,18 @@
     </collision>
   </link>
-  <xacro:sandia_hand side="right" parent="base" reflect="1">
+  <joint name="r_hand_base" type="fixed">
+    <parent link="base"/>
+    <child link="r_hand"/>
+  </joint>
+  <link name="r_hand"/>
+  <joint name="l_hand_base" type="fixed">
+    <parent link="base"/>
+    <child link="l_hand"/>
+  </joint>
+  <link name="l_hand"/>
+  <xacro:sandia_hand side="right" parent="r_hand" reflect="1">
     <origin xyz="0 0.2 0.5" rpy="0 -1.57079 0"/>
   </xacro:sandia_hand>
-  <xacro:sandia_hand side="left" parent="base" reflect="-1">
+  <xacro:sandia_hand side="left" parent="l_hand" reflect="-1">
     <origin xyz="0 -0.2 0.5" rpy="0 -1.57079 0"/>
   </xacro:sandia_hand>

File: ros/sandia_hand_description/urdf/sandia_hand.gazebo.xacro (robot description, xacro)
@@ -64,5 +64,5 @@
   <xacro:property name="cam_d1" value="0.1" />
   <xacro:property name="cam_L1" value="0.09" />
-  <xacro:macro name="sandia_hand_cameras_gazebo" params="side reflect">
+  <xacro:macro name="sandia_hand_cameras_gazebo" params="side reflect parent">
     <joint name="${side}_palm_left_camera_frame_joint" type="fixed">
       <origin xyz="${(cam_L1+reflect*stereo_offset/2)*sin_theta} ${reflect*(cam_d1-(cam_L1+reflect*stereo_offset/2)*cos_theta)} 0.025"
@@ -123,5 +123,5 @@
           <alwaysOn>true</alwaysOn>
           <updateRate>0.0</updateRate>
-          <cameraName>sandia_hands/${side}_hand/camera</cameraName>
+          <cameraName>sandia_hands/${parent}/camera</cameraName>
           <imageTopicName>image_raw</imageTopicName>
           <cameraInfoTopicName>camera_info</cameraInfoTopicName>

File: ros/sandia_hand_description/urdf/sandia_hand_simple_shapes.urdf.xacro (robot description, xacro)
@@ -411,5 +411,5 @@
     -->
     <xacro:sandia_hand_gazebo side="${side}" />
-    <xacro:sandia_hand_cameras_gazebo side="${side}" reflect="${reflect}" />
+    <xacro:sandia_hand_cameras_gazebo side="${side}" reflect="${reflect}" parent="${parent}" />
   </xacro:macro>
 </robot>

Commit message: Add a new xacro parameter to sandia_hand_description, so that the revolute joints in fingers can be optionally set as fixed to simplify the dynamic model, while still supporting hand cameras

File: ros/sandia_hand_description/robots/sandia_hand_both_on_box.urdf.xacro (robot description, xacro)
@@ -36,8 +36,8 @@
   </joint>
   <link name="l_hand"/>
-  <xacro:sandia_hand side="right" parent="r_hand" reflect="1">
+  <xacro:sandia_hand side="right" parent="r_hand" reflect="1" joint_type="revolute">
     <origin xyz="0 0.2 0.5" rpy="0 -1.57079 0"/>
   </xacro:sandia_hand>
-  <xacro:sandia_hand side="left" parent="l_hand" reflect="-1">
+  <xacro:sandia_hand side="left" parent="l_hand" reflect="-1" joint_type="revolute">
     <origin xyz="0 -0.2 0.5" rpy="0 -1.57079 0"/>
   </xacro:sandia_hand>

File: ros/sandia_hand_description/robots/sandia_hand_left_on_box.urdf.xacro (robot description, xacro)
@@ -26,5 +26,5 @@
     </collision>
   </link>
-  <xacro:sandia_hand side="left" parent="base" reflect="-1">
+  <xacro:sandia_hand side="left" parent="base" reflect="-1" joint_type="revolute">
     <origin xyz="0 0 0.5" rpy="0 -1.57079 0"/>
   </xacro:sandia_hand>

File: ros/sandia_hand_description/robots/sandia_hand_stumps_on_box.urdf.xacro (robot description, xacro)
@@ -26,6 +26,19 @@
     </collision>
   </link>
-  <xacro:sandia_hand side="right" parent="base" reflect="1" joint_type="revolute">
-    <origin xyz="0 0 0.5" rpy="0 -1.57079 0"/>
+  <joint name="r_hand_base" type="fixed">
+    <parent link="base"/>
+    <child link="r_hand"/>
+  </joint>
+  <link name="r_hand"/>
+  <joint name="l_hand_base" type="fixed">
+    <parent link="base"/>
+    <child link="l_hand"/>
+  </joint>
+  <link name="l_hand"/>
+  <xacro:sandia_hand side="right" parent="r_hand" reflect="1" joint_type="fixed">
+    <origin xyz="0 0.2 0.5" rpy="0 -1.57079 0"/>
+  </xacro:sandia_hand>
+  <xacro:sandia_hand side="left" parent="l_hand" reflect="-1" joint_type="fixed">
+    <origin xyz="0 -0.2 0.5" rpy="0 -1.57079 0"/>
   </xacro:sandia_hand>
 </robot>

File: ros/sandia_hand_description/urdf/sandia_hand_simple_shapes.urdf.xacro (robot description, xacro)
@@ -5,5 +5,5 @@
   <include filename="$(find sandia_hand_description)/urdf/sandia_hand.transmission.xacro" />
   <xacro:property name="M_pi" value="3.1415926535897931" />
-  <xacro:macro name="finger" params="idx x y z r p yaw side reflect">
+  <xacro:macro name="finger" params="idx x y z r p yaw side reflect joint_type">
     <link name="${side}_f${idx}_base">
       <origin xyz="0 0 0" rpy="0 0 0"/>
@@ -215,5 +215,5 @@
       <origin xyz="${x} ${y} ${z}" rpy="${r} ${p} ${yaw}"/>
     </joint>
-    <joint name="${side}_f${idx}_j0" type="revolute">
+    <joint name="${side}_f${idx}_j0" type="${joint_type}">
       <axis xyz="0 0 ${reflect}"/>
       <parent link="${side}_f${idx}_base"/>
@@ -224,5 +224,5 @@
       <origin xyz="0 0 0" rpy="0 0 0"/>
     </joint>
-    <joint name="${side}_f${idx}_j1" type="revolute">
+    <joint name="${side}_f${idx}_j1" type="${joint_type}">
       <axis xyz="0 0 1"/>
       <parent link="${side}_f${idx}_0"/>
@@ -233,5 +233,5 @@
       <origin xyz="0.028 0 0" rpy="${M_pi/2} 0 0"/>
     </joint>
-    <joint name="${side}_f${idx}_j2" type="revolute">
+    <joint name="${side}_f${idx}_j2" type="${joint_type}">
       <axis xyz="0 0 1"/>
       <parent link="${side}_f${idx}_1"/>
@@ -260,5 +260,5 @@
     <xacro:finger_gazebo side="${side}" idx="${idx}"/>
   </xacro:macro>
-  <xacro:macro name="sandia_hand" params="side parent reflect *origin">
+  <xacro:macro name="sandia_hand" params="side parent reflect joint_type *origin">
     <link name="${side}_palm">
       <origin xyz="0 0 0" rpy="0 0 0"/>
@@ -403,8 +403,8 @@
       <insert_block name="origin" />
     </joint>
-    <xacro:finger side="${side}" idx="0" x="0.140" y="0.00000" z="0" r="0" p="0" yaw="${0.3*reflect}" reflect="${reflect}" />
-    <xacro:finger side="${side}" idx="1" x="0.115" y="${0.03122*reflect}" z="0" r="0" p="0" yaw="${0.3*reflect}" reflect="${reflect}" />
-    <xacro:finger side="${side}" idx="2" x="0.090" y="${0.06245*reflect}" z="0" r="0" p="0" yaw="${0.3*reflect}" reflect="${reflect}" />
-    <xacro:finger side="${side}" idx="3" x="0.03995" y="${-0.04383*reflect}" z="0.014" r="0" p="-${M_pi/2}" yaw="${-2.3562*reflect}" reflect="${reflect}" />
+    <xacro:finger side="${side}" idx="0" x="0.140" y="0.00000" z="0" r="0" p="0" yaw="${0.3*reflect}" reflect="${reflect}" joint_type="${joint_type}" />
+    <xacro:finger side="${side}" idx="1" x="0.115" y="${0.03122*reflect}" z="0" r="0" p="0" yaw="${0.3*reflect}" reflect="${reflect}" joint_type="${joint_type}" />
+    <xacro:finger side="${side}" idx="2" x="0.090" y="${0.06245*reflect}" z="0" r="0" p="0" yaw="${0.3*reflect}" reflect="${reflect}" joint_type="${joint_type}" />
+    <xacro:finger side="${side}" idx="3" x="0.03995" y="${-0.04383*reflect}" z="0.014" r="0" p="-${M_pi/2}" yaw="${-2.3562*reflect}" reflect="${reflect}" joint_type="${joint_type}" />
     <!-- not needed unless simulating the hand by itself
     <xacro:sandia_hand_gazebo_controller side="${side}" />

Commit message: Add another parameter to specify thumb angle, used to move thumbs out of camera frame when joint_type='fixed'

File: ros/sandia_hand_description/robots/sandia_hand_both_on_box.urdf.xacro (robot description, xacro)
@@ -36,8 +36,8 @@
   </joint>
   <link name="l_hand"/>
-  <xacro:sandia_hand side="right" parent="r_hand" reflect="1" joint_type="revolute">
+  <xacro:sandia_hand side="right" parent="r_hand" reflect="1" joint_type="revolute" thumb_angle="0">
     <origin xyz="0 0.2 0.5" rpy="0 -1.57079 0"/>
   </xacro:sandia_hand>
-  <xacro:sandia_hand side="left" parent="l_hand" reflect="-1" joint_type="revolute">
+  <xacro:sandia_hand side="left" parent="l_hand" reflect="-1" joint_type="revolute" thumb_angle="0">
     <origin xyz="0 -0.2 0.5" rpy="0 -1.57079 0"/>
   </xacro:sandia_hand>

File: ros/sandia_hand_description/robots/sandia_hand_left_on_box.urdf.xacro (robot description, xacro)
@@ -26,5 +26,5 @@
     </collision>
   </link>
-  <xacro:sandia_hand side="left" parent="base" reflect="-1" joint_type="revolute">
+  <xacro:sandia_hand side="left" parent="base" reflect="-1" joint_type="revolute" thumb_angle="0">
     <origin xyz="0 0 0.5" rpy="0 -1.57079 0"/>
   </xacro:sandia_hand>

File: ros/sandia_hand_description/robots/sandia_hand_right_on_box.urdf.xacro (robot description, xacro)
@@ -26,5 +26,5 @@
     </collision>
   </link>
-  <xacro:sandia_hand side="right" parent="base" reflect="1" joint_type="revolute">
+  <xacro:sandia_hand side="right" parent="base" reflect="1" joint_type="revolute" thumb_angle="0">
     <origin xyz="0 0 0.5" rpy="0 -1.57079 0"/>
   </xacro:sandia_hand>

File: ros/sandia_hand_description/robots/sandia_hand_stumps_on_box.urdf.xacro (robot description, xacro)
@@ -36,8 +36,8 @@
   </joint>
   <link name="l_hand"/>
-  <xacro:sandia_hand side="right" parent="r_hand" reflect="1" joint_type="fixed">
+  <xacro:sandia_hand side="right" parent="r_hand" reflect="1" joint_type="fixed" thumb_angle="1.57">
     <origin xyz="0 0.2 0.5" rpy="0 -1.57079 0"/>
   </xacro:sandia_hand>
-  <xacro:sandia_hand side="left" parent="l_hand" reflect="-1" joint_type="fixed">
+  <xacro:sandia_hand side="left" parent="l_hand" reflect="-1" joint_type="fixed" thumb_angle="1.57">
     <origin xyz="0 -0.2 0.5" rpy="0 -1.57079 0"/>
   </xacro:sandia_hand>

File: ros/sandia_hand_description/urdf/sandia_hand_simple_shapes.urdf.xacro (robot description, xacro)
@@ -260,5 +260,5 @@
     <xacro:finger_gazebo side="${side}" idx="${idx}"/>
   </xacro:macro>
-  <xacro:macro name="sandia_hand" params="side parent reflect joint_type *origin">
+  <xacro:macro name="sandia_hand" params="side parent reflect joint_type thumb_angle *origin">
     <link name="${side}_palm">
       <origin xyz="0 0 0" rpy="0 0 0"/>
@@ -406,5 +406,5 @@
     <xacro:finger side="${side}" idx="1" x="0.115" y="${0.03122*reflect}" z="0" r="0" p="0" yaw="${0.3*reflect}" reflect="${reflect}" joint_type="${joint_type}" />
     <xacro:finger side="${side}" idx="2" x="0.090" y="${0.06245*reflect}" z="0" r="0" p="0" yaw="${0.3*reflect}" reflect="${reflect}" joint_type="${joint_type}" />
-    <xacro:finger side="${side}" idx="3" x="0.03995" y="${-0.04383*reflect}" z="0.014" r="0" p="-${M_pi/2}" yaw="${-2.3562*reflect}" reflect="${reflect}" joint_type="${joint_type}" />
+    <xacro:finger side="${side}" idx="3" x="0.03995" y="${-0.04383*reflect}" z="0.014" r="0" p="-${M_pi/2 + thumb_angle}" yaw="${-(2.3562+thumb_angle)*reflect}" reflect="${reflect}" joint_type="${joint_type}" />
     <!-- not needed unless simulating the hand by itself
     <xacro:sandia_hand_gazebo_controller side="${side}" />

Commit message: Revert stump changes to sandia-hands until we're ready to do it for drcsim

File: ros/sandia_hand_description/robots/sandia_hand_both_on_box.urdf.xacro (robot description, xacro)
@@ -36,8 +36,8 @@
   </joint>
   <link name="l_hand"/>
-  <xacro:sandia_hand side="right" parent="r_hand" reflect="1" joint_type="revolute" thumb_angle="0">
+  <xacro:sandia_hand side="right" parent="r_hand" reflect="1"><!-- joint_type="revolute" thumb_angle="0"-->
     <origin xyz="0 0.2 0.5" rpy="0 -1.57079 0"/>
   </xacro:sandia_hand>
-  <xacro:sandia_hand side="left" parent="l_hand" reflect="-1" joint_type="revolute" thumb_angle="0">
+  <xacro:sandia_hand side="left" parent="l_hand" reflect="-1"><!-- joint_type="revolute" thumb_angle="0"-->
     <origin xyz="0 -0.2 0.5" rpy="0 -1.57079 0"/>
   </xacro:sandia_hand>

File: ros/sandia_hand_description/robots/sandia_hand_left_on_box.urdf.xacro (robot description, xacro)
@@ -26,5 +26,5 @@
     </collision>
   </link>
-  <xacro:sandia_hand side="left" parent="base" reflect="-1" joint_type="revolute" thumb_angle="0">
+  <xacro:sandia_hand side="left" parent="base" reflect="-1"><!-- joint_type="revolute" thumb_angle="0"-->
     <origin xyz="0 0 0.5" rpy="0 -1.57079 0"/>
   </xacro:sandia_hand>

File: ros/sandia_hand_description/robots/sandia_hand_right_on_box.urdf.xacro (robot description, xacro)
@@ -26,5 +26,5 @@
     </collision>
   </link>
-  <xacro:sandia_hand side="right" parent="base" reflect="1" joint_type="revolute" thumb_angle="0">
+  <xacro:sandia_hand side="right" parent="base" reflect="1"><!-- joint_type="revolute" thumb_angle="0"-->
     <origin xyz="0 0 0.5" rpy="0 -1.57079 0"/>
   </xacro:sandia_hand>

File: ros/sandia_hand_description/robots/sandia_hand_stumps_on_box.urdf.xacro (robot description, xacro)
@@ -36,8 +36,8 @@
   </joint>
   <link name="l_hand"/>
-  <xacro:sandia_hand side="right" parent="r_hand" reflect="1" joint_type="fixed" thumb_angle="1.57">
+  <xacro:sandia_hand side="right" parent="r_hand" reflect="1"><!-- joint_type="fixed" thumb_angle="1.57"-->
     <origin xyz="0 0.2 0.5" rpy="0 -1.57079 0"/>
   </xacro:sandia_hand>
-  <xacro:sandia_hand side="left" parent="l_hand" reflect="-1" joint_type="fixed" thumb_angle="1.57">
+  <xacro:sandia_hand side="left" parent="l_hand" reflect="-1"><!-- joint_type="fixed" thumb_angle="1.57"-->
     <origin xyz="0 -0.2 0.5" rpy="0 -1.57079 0"/>
   </xacro:sandia_hand>

File: ros/sandia_hand_description/urdf/sandia_hand_simple_shapes.urdf.xacro (robot description, xacro)
@@ -260,5 +260,8 @@
     <xacro:finger_gazebo side="${side}" idx="${idx}"/>
   </xacro:macro>
+  <!--
   <xacro:macro name="sandia_hand" params="side parent reflect joint_type thumb_angle *origin">
+  -->
+  <xacro:macro name="sandia_hand" params="side parent reflect *origin">
     <link name="${side}_palm">
       <origin xyz="0 0 0" rpy="0 0 0"/>
@@ -403,8 +406,14 @@
       <insert_block name="origin" />
     </joint>
+    <!--
     <xacro:finger side="${side}" idx="0" x="0.140" y="0.00000" z="0" r="0" p="0" yaw="${0.3*reflect}" reflect="${reflect}" joint_type="${joint_type}" />
     <xacro:finger side="${side}" idx="1" x="0.115" y="${0.03122*reflect}" z="0" r="0" p="0" yaw="${0.3*reflect}" reflect="${reflect}" joint_type="${joint_type}" />
     <xacro:finger side="${side}" idx="2" x="0.090" y="${0.06245*reflect}" z="0" r="0" p="0" yaw="${0.3*reflect}" reflect="${reflect}" joint_type="${joint_type}" />
     <xacro:finger side="${side}" idx="3" x="0.03995" y="${-0.04383*reflect}" z="0.014" r="0" p="-${M_pi/2 + thumb_angle}" yaw="${-(2.3562+thumb_angle)*reflect}" reflect="${reflect}" joint_type="${joint_type}" />
+    -->
+    <xacro:finger side="${side}" idx="0" x="0.140" y="0.00000" z="0" r="0" p="0" yaw="${0.3*reflect}" reflect="${reflect}" joint_type="revolute" />
+    <xacro:finger side="${side}" idx="1" x="0.115" y="${0.03122*reflect}" z="0" r="0" p="0" yaw="${0.3*reflect}" reflect="${reflect}" joint_type="revolute" />
+    <xacro:finger side="${side}" idx="2" x="0.090" y="${0.06245*reflect}" z="0" r="0" p="0" yaw="${0.3*reflect}" reflect="${reflect}" joint_type="revolute" />
+    <xacro:finger side="${side}" idx="3" x="0.03995" y="${-0.04383*reflect}" z="0.014" r="0" p="-${M_pi/2}" yaw="${-(2.3562)*reflect}" reflect="${reflect}" joint_type="joint_type" />
     <!-- not needed unless simulating the hand by itself
     <xacro:sandia_hand_gazebo_controller side="${side}" />

Commit message: Branch to use stumps with drcsim, requires simultaneous release

File: ros/sandia_hand_description/robots/sandia_hand_both_on_box.urdf.xacro (robot description, xacro)
@@ -36,8 +36,8 @@
   </joint>
   <link name="l_hand"/>
-  <xacro:sandia_hand side="right" parent="r_hand" reflect="1"><!-- joint_type="revolute" thumb_angle="0"-->
+  <xacro:sandia_hand side="right" parent="r_hand" reflect="1" joint_type="revolute" thumb_angle="0">
     <origin xyz="0 0.2 0.5" rpy="0 -1.57079 0"/>
   </xacro:sandia_hand>
-  <xacro:sandia_hand side="left" parent="l_hand" reflect="-1"><!-- joint_type="revolute" thumb_angle="0"-->
+  <xacro:sandia_hand side="left" parent="l_hand" reflect="-1" joint_type="revolute" thumb_angle="0">
     <origin xyz="0 -0.2 0.5" rpy="0 -1.57079 0"/>
   </xacro:sandia_hand>

File: ros/sandia_hand_description/robots/sandia_hand_left_on_box.urdf.xacro (robot description, xacro)
@@ -26,5 +26,5 @@
     </collision>
   </link>
-  <xacro:sandia_hand side="left" parent="base" reflect="-1"><!-- joint_type="revolute" thumb_angle="0"-->
+  <xacro:sandia_hand side="left" parent="base" reflect="-1" joint_type="revolute" thumb_angle="0">
     <origin xyz="0 0 0.5" rpy="0 -1.57079 0"/>
   </xacro:sandia_hand>

File: ros/sandia_hand_description/robots/sandia_hand_right_on_box.urdf.xacro (robot description, xacro)
@@ -26,5 +26,5 @@
     </collision>
   </link>
-  <xacro:sandia_hand side="right" parent="base" reflect="1"><!-- joint_type="revolute" thumb_angle="0"-->
+  <xacro:sandia_hand side="right" parent="base" reflect="1" joint_type="revolute" thumb_angle="0">
     <origin xyz="0 0 0.5" rpy="0 -1.57079 0"/>
   </xacro:sandia_hand>

File: ros/sandia_hand_description/robots/sandia_hand_stumps_on_box.urdf.xacro (robot description, xacro)
@@ -36,8 +36,8 @@
   </joint>
   <link name="l_hand"/>
-  <xacro:sandia_hand side="right" parent="r_hand" reflect="1"><!-- joint_type="fixed" thumb_angle="1.57"-->
+  <xacro:sandia_hand side="right" parent="r_hand" reflect="1" joint_type="fixed" thumb_angle="1.57">
     <origin xyz="0 0.2 0.5" rpy="0 -1.57079 0"/>
   </xacro:sandia_hand>
-  <xacro:sandia_hand side="left" parent="l_hand" reflect="-1"><!-- joint_type="fixed" thumb_angle="1.57"-->
+  <xacro:sandia_hand side="left" parent="l_hand" reflect="-1" joint_type="fixed" thumb_angle="1.57">
     <origin xyz="0 -0.2 0.5" rpy="0 -1.57079 0"/>
   </xacro:sandia_hand>

File: ros/sandia_hand_description/urdf/sandia_hand_simple_shapes.urdf.xacro (robot description, xacro)
@@ -9,5 +9,5 @@
   <xacro:property name="damping_coefficient_j2" value="30" />
   <xacro:property name="velocity_limit" value="100" />
-  <xacro:macro name="finger" params="idx x y z r p yaw side reflect">
+  <xacro:macro name="finger" params="idx x y z r p yaw side reflect joint_type">
     <link name="${side}_f${idx}_base">
       <origin xyz="0 0 0" rpy="0 0 0"/>
@@ -219,5 +219,5 @@
       <origin xyz="${x} ${y} ${z}" rpy="${r} ${p} ${yaw}"/>
     </joint>
-    <joint name="${side}_f${idx}_j0" type="revolute">
+    <joint name="${side}_f${idx}_j0" type="${joint_type}">
       <axis xyz="0 0 ${reflect}"/>
       <parent link="${side}_f${idx}_base"/>
@@ -228,5 +228,5 @@
       <origin xyz="0 0 0" rpy="0 0 0"/>
     </joint>
-    <joint name="${side}_f${idx}_j1" type="revolute">
+    <joint name="${side}_f${idx}_j1" type="${joint_type}">
       <axis xyz="0 0 1"/>
       <parent link="${side}_f${idx}_0"/>
@@ -237,5 +237,5 @@
       <origin xyz="0.028 0 0" rpy="${M_pi/2} 0 0"/>
     </joint>
-    <joint name="${side}_f${idx}_j2" type="revolute">
+    <joint name="${side}_f${idx}_j2" type="${joint_type}">
       <axis xyz="0 0 1"/>
       <parent link="${side}_f${idx}_1"/>
@@ -264,8 +264,5 @@
     <xacro:finger_gazebo side="${side}" idx="${idx}"/>
   </xacro:macro>
-  <!--
-  <xacro:macro name="sandia_hand" params="side parent reflect thumb_angle *origin">
-  -->
-  <xacro:macro name="sandia_hand" params="side parent reflect *origin">
+  <xacro:macro name="sandia_hand" params="side parent reflect joint_type thumb_angle *origin">
     <link name="${side}_palm">
       <origin xyz="0 0 0" rpy="0 0 0"/>
@@ -410,14 +407,8 @@
       <insert_block name="origin" />
     </joint>
-    <!--
-    <xacro:finger side="${side}" idx="0" x="0.140" y="0.00000" z="0" r="0" p="0" yaw="${0.3*reflect}" reflect="${reflect}" />
-    <xacro:finger side="${side}" idx="1" x="0.115" y="${0.03122*reflect}" z="0" r="0" p="0" yaw="${0.3*reflect}" reflect="${reflect}" />
-    <xacro:finger side="${side}" idx="2" x="0.090" y="${0.06245*reflect}" z="0" r="0" p="0" yaw="${0.3*reflect}" reflect="${reflect}" />
-    <xacro:finger side="${side}" idx="3" x="0.03995" y="${-0.04383*reflect}" z="0.014" r="0" p="-${M_pi/2 + thumb_angle}" yaw="${-(2.3562+thumb_angle)*reflect}" reflect="${reflect}" />
-    -->
-    <xacro:finger side="${side}" idx="0" x="0.140" y="0.00000" z="0" r="0" p="0" yaw="${0.3*reflect}" reflect="${reflect}" />
-    <xacro:finger side="${side}" idx="1" x="0.115" y="${0.03122*reflect}" z="0" r="0" p="0" yaw="${0.3*reflect}" reflect="${reflect}" />
-    <xacro:finger side="${side}" idx="2" x="0.090" y="${0.06245*reflect}" z="0" r="0" p="0" yaw="${0.3*reflect}" reflect="${reflect}" />
-    <xacro:finger side="${side}" idx="3" x="0.03995" y="${-0.04383*reflect}" z="0.014" r="0" p="-${M_pi/2}" yaw="${-(2.3562)*reflect}" reflect="${reflect}" />
+    <xacro:finger side="${side}" idx="0" x="0.140" y="0.00000" z="0" r="0" p="0" yaw="${0.3*reflect}" reflect="${reflect}" joint_type="${joint_type}"/>
+    <xacro:finger side="${side}" idx="1" x="0.115" y="${0.03122*reflect}" z="0" r="0" p="0" yaw="${0.3*reflect}" reflect="${reflect}" joint_type="${joint_type}"/>
+    <xacro:finger side="${side}" idx="2" x="0.090" y="${0.06245*reflect}" z="0" r="0" p="0" yaw="${0.3*reflect}" reflect="${reflect}" joint_type="${joint_type}"/>
+    <xacro:finger side="${side}" idx="3" x="0.03995" y="${-0.04383*reflect}" z="0.014" r="0" p="-${M_pi/2 + thumb_angle}" yaw="${-(2.3562+thumb_angle)*reflect}" reflect="${reflect}" joint_type="${joint_type}"/>
     <!-- not needed unless simulating the hand by itself
     <xacro:sandia_hand_gazebo_controller side="${side}" />
