Commit message: update package name references in urdf

File: ros/sandia_hand_description/urdf/sandia_hand.urdf.xacro (robot description, xacro)
@@ -31,5 +31,5 @@
         <origin xyz="0 0 0" rpy="0 0 0"/>
         <geometry>
-          <mesh filename="package://sandia_hand/meshes/f0.stl"/>
+          <mesh filename="package://sandia_hand_description/meshes/f0.stl"/>
         </geometry>
       </collision>
@@ -37,5 +37,5 @@
         <origin xyz="0 0 0" rpy="0 0 0"/>
         <geometry>
-          <mesh filename="package://sandia_hand/meshes/f0.stl"/>
+          <mesh filename="package://sandia_hand_description/meshes/f0.stl"/>
         </geometry>
         <material name="${side}_sandia_hand_skin_suntan">
@@ -54,5 +54,5 @@
         <origin xyz="0 0 0" rpy="0 0 0"/>
         <geometry>
-          <mesh filename="package://sandia_hand/meshes/f1.stl"/>
+          <mesh filename="package://sandia_hand_description/meshes/f1.stl"/>
         </geometry>
       </collision>
@@ -60,5 +60,5 @@
         <origin xyz="0 0 0" rpy="0 0 0"/>
         <geometry>
-          <mesh filename="package://sandia_hand/meshes/f1.stl"/>
+          <mesh filename="package://sandia_hand_description/meshes/f1.stl"/>
         </geometry>
         <material name="${side}_sandia_hand_skin">
@@ -85,5 +85,5 @@
         <origin xyz="0 0 0" rpy="0 0 0"/>
         <geometry>
-          <mesh filename="package://sandia_hand/meshes/f2.stl"/>
+          <mesh filename="package://sandia_hand_description/meshes/f2.stl"/>
         </geometry>
       </collision>
@@ -91,5 +91,5 @@
         <origin xyz="0 0 0" rpy="0 0 0"/>
         <geometry>
-          <mesh filename="package://sandia_hand/meshes/f2.stl"/>
+          <mesh filename="package://sandia_hand_description/meshes/f2.stl"/>
         </geometry>
         <material name="${side}_sandia_hand_skin_suntan">
@@ -166,5 +166,5 @@
         <origin xyz="0 0 0" rpy="0 0 0"/>
         <geometry>
-          <mesh filename="package://sandia_hand/meshes/palm.stl"/>
+          <mesh filename="package://sandia_hand_description/meshes/palm.stl"/>
         </geometry>
       </collision>
@@ -172,5 +172,5 @@
         <origin xyz="0 0 0" rpy="0 0 0"/>
         <geometry>
-          <mesh filename="package://sandia_hand/meshes/palm.stl"/>
+          <mesh filename="package://sandia_hand_description/meshes/palm.stl"/>
         </geometry>
         <material name="${side}_sandia_hand_skin">

Commit message: First pass at simple collision shapes for sandia hand

File: ros/sandia_hand_description/urdf/sandia_hand.urdf.xacro (robot description, xacro)
@@ -28,4 +28,51 @@
         <inertia ixx="0.01" ixy="0" ixz="0" iyy="0.01" iyz="0" izz="0.01"/>
       </inertial>
+      <!-- begin simple shape approximation of f0 -->
+      <collision>
+        <pose>0 0 0.003 0 0 0</pose>
+        <geometry>
+          <cylinder>
+            <radius>0.015</radius>
+            <length>0.023</length>
+          </cylinder>
+        </geometry>
+      </collision>
+      <collision>
+        <pose>0.011 0 0.003 1.57 0 0</pose>
+        <geometry>
+          <cylinder>
+            <radius>0.01</radius>
+            <length>0.023</length>
+          </cylinder>
+        </geometry>
+      </collision>
+      <!--   end simple shape approximation of f0 -->
+      <!-- begin visual shape approximation of f0 -->
+      <visual>
+        <pose>0 0 0.003 0 0 0</pose>
+        <geometry>
+          <cylinder>
+            <radius>0.015</radius>
+            <length>0.023</length>
+          </cylinder>
+        </geometry>
+        <material name="${side}_sandia_hand_skin_suntan">
+          <color rgba="0.7 0.4 0.2 1.0"/>
+        </material>
+      </visual>
+      <visual>
+        <pose>0.011 0 0.003 1.57 0 0</pose>
+        <geometry>
+          <cylinder>
+            <radius>0.01</radius>
+            <length>0.023</length>
+          </cylinder>
+        </geometry>
+        <material name="${side}_sandia_hand_skin_suntan">
+          <color rgba="0.7 0.4 0.2 1.0"/>
+        </material>
+      </visual>
+      <!--   end visual shape approximation of f0 -->
+      <!-- begin collision mesh of f0 ->
       <collision>
         <origin xyz="0 0 0" rpy="0 0 0"/>
@@ -34,4 +81,6 @@
         </geometry>
       </collision>
+      <!-   end collision mesh of f0 -->
+      <!-- begin visual mesh of f0 ->
       <visual>
         <origin xyz="0 0 0" rpy="0 0 0"/>
@@ -43,4 +92,5 @@
         </material>
       </visual>
+      <!-   end visual mesh of f0 -->
     </link>
     <link name="${side}_f${idx}_1">
@@ -51,4 +101,30 @@
         <inertia ixx="0.01" ixy="0" ixz="0" iyy="0.01" iyz="0" izz="0.01"/>
       </inertial>
+      <!-- begin simple shape approximation of f1 -->
+      <collision>
+        <pose>0.024 0 0 0 1.57 0</pose>
+        <geometry>
+          <cylinder>
+            <radius>0.01</radius>
+            <length>0.067</length>
+          </cylinder>
+        </geometry>
+      </collision>
+      <!--   end simple shape approximation of f1 -->
+      <!-- begin visual shape approximation of f1 -->
+      <visual>
+        <pose>0.024 0 0 0 1.57 0</pose>
+        <geometry>
+          <cylinder>
+            <radius>0.01</radius>
+            <length>0.067</length>
+          </cylinder>
+        </geometry>
+        <material name="${side}_sandia_hand_skin">
+          <color rgba="0.835 0.655 0.345 1.0"/>
+        </material>
+      </visual>
+      <!--   end visual shape approximation of f1 -->
+      <!-- begin collision mesh of f1 ->
       <collision>
         <origin xyz="0 0 0" rpy="0 0 0"/>
@@ -57,4 +133,6 @@
         </geometry>
       </collision>
+      <!-   end collision mesh of f1 -->
+      <!-- begin visual mesh of f1 ->
       <visual>
         <origin xyz="0 0 0" rpy="0 0 0"/>
@@ -66,4 +144,5 @@
         </material>
       </visual>
+      <!-   end visual mesh of f1 -->
     </link>
     <link name="${side}_f${idx}_1_accel">
@@ -82,4 +161,48 @@
         <inertia ixx="0.01" ixy="0" ixz="0" iyy="0.01" iyz="0" izz="0.01"/>
       </inertial>
+      <!-- begin simple shape approximation of f2 -->
+      <collision>
+        <pose>0.024 0 0 0 1.57 0</pose>
+        <geometry>
+          <cylinder>
+            <radius>0.009</radius>
+            <length>0.057</length>
+          </cylinder>
+        </geometry>
+      </collision>
+      <collision>
+        <pose>0.052 0 0 0 0 0</pose>
+        <geometry>
+          <sphere>
+            <radius>0.009</radius>
+          </sphere>
+        </geometry>
+      </collision>
+      <!--   end simple shape approximation of f2 -->
+      <!-- begin visual shape approximation of f2 -->
+      <visual>
+        <pose>0.024 0 0 0 1.57 0</pose>
+        <geometry>
+          <cylinder>
+            <radius>0.009</radius>
+            <length>0.057</length>
+          </cylinder>
+        </geometry>
+        <material name="${side}_sandia_hand_skin_suntan">
+          <color rgba="0.8 0.6 0.3 1.0"/>
+        </material>
+      </visual>
+      <visual>
+        <pose>0.052 0 0 0 0 0</pose>
+        <geometry>
+          <sphere>
+            <radius>0.009</radius>
+          </sphere>
+        </geometry>
+        <material name="${side}_sandia_hand_skin_suntan">
+          <color rgba="0.8 0.6 0.3 1.0"/>
+        </material>
+      </visual>
+      <!-- begin collision mesh of f2    ->
       <collision>
         <origin xyz="0 0 0" rpy="0 0 0"/>
@@ -88,4 +211,6 @@
         </geometry>
       </collision>
+      <!-   end collision mesh of f2 -->
+      <!-- begin visual mesh of f2    ->
       <visual>
         <origin xyz="0 0 0" rpy="0 0 0"/>
@@ -97,4 +222,5 @@
         </material>
       </visual>
+      <!-   end visual mesh of f2 -->
     </link>
     <link name="${side}_f${idx}_2_accel">
@@ -163,4 +289,146 @@
         <inertia ixx="0.01" ixy="0" ixz="0" iyy="0.01" iyz="0" izz="0.01"/>
       </inertial>
+      <!-- begin simple shape approximation of palm -->
+      <collision>
+        <pose>0.069 0.016 0.038 0 1.57 -0.9</pose>
+        <geometry>
+          <cylinder>
+            <radius>0.013</radius>
+            <length>0.100</length>
+          </cylinder>
+        </geometry>
+      </collision>
+      <collision>
+        <pose>0.064 0.008 0.021 0.41 0 -0.9</pose>
+        <geometry>
+          <box>
+            <size>0.09 .035 .05</size>
+          </box>
+        </geometry>
+      </collision>
+      <collision>
+        <pose>0.02 0 -0.005 0 1.57 0</pose>
+        <geometry>
+          <cylinder>
+            <radius>0.038</radius>
+            <length>0.05</length>
+          </cylinder>
+        </geometry>
+      </collision>
+      <collision>
+        <pose>0.11 -0.01 -0.005 0 0 0.37</pose>
+        <geometry>
+          <box>
+            <size>0.09 .03 .06</size>
+          </box>
+        </geometry>
+      </collision>
+      <collision>
+        <pose>0.09 0.02 -0.005 0 0 0.37</pose>
+        <geometry>
+          <box>
+            <size>0.09 .03 .06</size>
+          </box>
+        </geometry>
+      </collision>
+      <collision>
+        <pose>0.060 0.050 -0.005 0 0 0.37</pose>
+        <geometry>
+          <box>
+            <size>0.09 .03 .06</size>
+          </box>
+        </geometry>
+      </collision>
+      <collision>
+        <pose>0.044 -0.04 -0.005 0 0 0.79</pose>
+        <geometry>
+          <box>
+            <size>0.09 .03 .06</size>
+          </box>
+        </geometry>
+      </collision>
+      <!--   end simple shape approximation of palm -->
+      <!-- begin visual shape approximation of palm -->
+      <visual>
+        <pose>0.069 0.016 0.038 0 1.57 -0.9</pose>
+        <geometry>
+          <cylinder>
+            <radius>0.013</radius>
+            <length>0.100</length>
+          </cylinder>
+        </geometry>
+        <material name="${side}_sandia_hand_skin">
+          <color rgba="0.835 0.655 0.345 1.0"/>
+        </material>
+      </visual>
+      <visual>
+        <pose>0.064 0.008 0.021 0.41 0 -0.9</pose>
+        <geometry>
+          <box>
+            <size>0.09 .035 .05</size>
+          </box>
+        </geometry>
+        <material name="${side}_sandia_hand_skin">
+          <color rgba="0.835 0.655 0.345 1.0"/>
+        </material>
+      </visual>
+      <visual>
+        <pose>0.02 0 -0.005 0 1.57 0</pose>
+        <geometry>
+          <cylinder>
+            <radius>0.038</radius>
+            <length>0.05</length>
+          </cylinder>
+        </geometry>
+        <material name="${side}_sandia_hand_skin">
+          <color rgba="0.835 0.655 0.345 1.0"/>
+        </material>
+      </visual>
+      <visual>
+        <pose>0.11 -0.01 -0.005 0 0 0.37</pose>
+        <geometry>
+          <box>
+            <size>0.09 .03 .06</size>
+          </box>
+        </geometry>
+        <material name="${side}_sandia_hand_skin">
+          <color rgba="0.835 0.655 0.345 1.0"/>
+        </material>
+      </visual>
+      <visual>
+        <pose>0.09 0.02 -0.005 0 0 0.37</pose>
+        <geometry>
+          <box>
+            <size>0.09 .03 .06</size>
+          </box>
+        </geometry>
+        <material name="${side}_sandia_hand_skin">
+          <color rgba="0.835 0.655 0.345 1.0"/>
+        </material>
+      </visual>
+      <visual>
+        <pose>0.060 0.050 -0.005 0 0 0.37</pose>
+        <geometry>
+          <box>
+            <size>0.09 .03 .06</size>
+          </box>
+        </geometry>
+        <material name="${side}_sandia_hand_skin">
+          <color rgba="0.835 0.655 0.345 1.0"/>
+        </material>
+      </visual>
+      <visual>
+        <pose>0.044 -0.04 -0.005 0 0 0.79</pose>
+        <geometry>
+          <box>
+            <size>0.09 .03 .06</size>
+          </box>
+        </geometry>
+        <material name="${side}_sandia_hand_skin">
+          <color rgba="0.835 0.655 0.345 1.0"/>
+        </material>
+      </visual>
+      <!--   end visual shape approximation of palm -->
+      <!-- begin collision mesh of f2 ->
       <collision>
         <origin xyz="0 0 0" rpy="0 0 0"/>
@@ -169,4 +437,6 @@
         </geometry>
       </collision>
+      <!-   end collision mesh of f2 -->
+      <!-- begin visual mesh of f2    ->
       <visual>
         <origin xyz="0 0 0" rpy="0 0 0"/>
@@ -178,4 +448,5 @@
         </material>
       </visual>
+      <!-   end visual mesh of f2 -->
     </link>
     <joint name="${side}_sandia_hand_joint" type="fixed">

Commit message: Converted pose to origin for urdf

File: ros/sandia_hand_description/urdf/sandia_hand.urdf.xacro (robot description, xacro)
@@ -30,5 +30,5 @@
       <!-- begin simple shape approximation of f0 -->
       <collision>
-        <pose>0 0 0.003 0 0 0</pose>
+        <origin xyz="0 0 0.003" rpy="0 0 0"/>
         <geometry>
           <cylinder>
@@ -39,5 +39,5 @@
       </collision>
       <collision>
-        <pose>0.011 0 0.003 1.57 0 0</pose>
+        <origin xyz="0.011 0 0.003" rpy="1.57 0 0"/>
         <geometry>
           <cylinder>
@@ -50,5 +50,5 @@
       <!-- begin visual shape approximation of f0 -->
       <visual>
-        <pose>0 0 0.003 0 0 0</pose>
+        <origin xyz="0 0 0.003" rpy="0 0 0"/>
         <geometry>
           <cylinder>
@@ -62,5 +62,5 @@
       </visual>
       <visual>
-        <pose>0.011 0 0.003 1.57 0 0</pose>
+        <origin xyz="0.011 0 0.003" rpy="1.57 0 0"/>
         <geometry>
           <cylinder>
@@ -103,5 +103,5 @@
       <!-- begin simple shape approximation of f1 -->
       <collision>
-        <pose>0.024 0 0 0 1.57 0</pose>
+        <origin xyz="0.024 0 0" rpy="0 1.57 0"/>
         <geometry>
           <cylinder>
@@ -114,5 +114,5 @@
       <!-- begin visual shape approximation of f1 -->
       <visual>
-        <pose>0.024 0 0 0 1.57 0</pose>
+        <origin xyz="0.024 0 0" rpy="0 1.57 0"/>
         <geometry>
           <cylinder>
@@ -163,5 +163,5 @@
       <!-- begin simple shape approximation of f2 -->
       <collision>
-        <pose>0.024 0 0 0 1.57 0</pose>
+        <origin xyz="0.024 0 0" rpy="0 1.57 0"/>
         <geometry>
           <cylinder>
@@ -172,5 +172,5 @@
       </collision>
       <collision>
-        <pose>0.052 0 0 0 0 0</pose>
+        <origin xyz="0.052 0 0" rpy="0 0 0"/>
         <geometry>
           <sphere>
@@ -182,5 +182,5 @@
       <!-- begin visual shape approximation of f2 -->
       <visual>
-        <pose>0.024 0 0 0 1.57 0</pose>
+        <origin xyz="0.024 0 0" rpy="0 1.57 0"/>
         <geometry>
           <cylinder>
@@ -194,5 +194,5 @@
       </visual>
       <visual>
-        <pose>0.052 0 0 0 0 0</pose>
+        <origin xyz="0.052 0 0" rpy="0 0 0"/>
         <geometry>
           <sphere>
@@ -291,5 +291,5 @@
       <!-- begin simple shape approximation of palm -->
       <collision>
-        <pose>0.069 0.016 0.038 0 1.57 -0.9</pose>
+        <origin xyz="0.069 0.016 0.038" rpy="0 1.57 -0.9"/>
         <geometry>
           <cylinder>
@@ -300,5 +300,5 @@
       </collision>
       <collision>
-        <pose>0.064 0.008 0.021 0.41 0 -0.9</pose>
+        <origin xyz="0.064 0.008 0.021" rpy="0.41 0 -0.9"/>
         <geometry>
           <box>
@@ -308,5 +308,5 @@
       </collision>
       <collision>
-        <pose>0.02 0 -0.005 0 1.57 0</pose>
+        <origin xyz="0.02 0 -0.005" rpy="0 1.57 0"/>
         <geometry>
           <cylinder>
@@ -317,29 +317,29 @@
       </collision>
       <collision>
-        <pose>0.11 -0.01 -0.005 0 0 0.37</pose>
-        <geometry>
-          <box>
-            <size>0.09 .03 .06</size>
-          </box>
-        </geometry>
-      </collision>
-      <collision>
-        <pose>0.09 0.02 -0.005 0 0 0.37</pose>
-        <geometry>
-          <box>
-            <size>0.09 .03 .06</size>
-          </box>
-        </geometry>
-      </collision>
-      <collision>
-        <pose>0.060 0.050 -0.005 0 0 0.37</pose>
-        <geometry>
-          <box>
-            <size>0.09 .03 .06</size>
-          </box>
-        </geometry>
-      </collision>
-      <collision>
-        <pose>0.044 -0.04 -0.005 0 0 0.79</pose>
+        <origin xyz="0.11 -0.01 -0.005" rpy="0 0 0.37"/>
+        <geometry>
+          <box>
+            <size>0.09 .03 .06</size>
+          </box>
+        </geometry>
+      </collision>
+      <collision>
+        <origin xyz="0.09 0.02 -0.005" rpy="0 0 0.37"/>
+        <geometry>
+          <box>
+            <size>0.09 .03 .06</size>
+          </box>
+        </geometry>
+      </collision>
+      <collision>
+        <origin xyz="0.060 0.050 -0.005" rpy="0 0 0.37"/>
+        <geometry>
+          <box>
+            <size>0.09 .03 .06</size>
+          </box>
+        </geometry>
+      </collision>
+      <collision>
+        <origin xyz="0.044 -0.04 -0.005" rpy="0 0 0.79"/>
         <geometry>
           <box>
@@ -351,5 +351,5 @@
       <!-- begin visual shape approximation of palm -->
       <visual>
-        <pose>0.069 0.016 0.038 0 1.57 -0.9</pose>
+        <origin xyz="0.069 0.016 0.038" rpy="0 1.57 -0.9"/>
         <geometry>
           <cylinder>
@@ -363,5 +363,5 @@
       </visual>
       <visual>
-        <pose>0.064 0.008 0.021 0.41 0 -0.9</pose>
+        <origin xyz="0.064 0.008 0.021" rpy="0.41 0 -0.9"/>
         <geometry>
           <box>
@@ -374,5 +374,5 @@
       </visual>
       <visual>
-        <pose>0.02 0 -0.005 0 1.57 0</pose>
+        <origin xyz="0.02 0 -0.005" rpy="0 1.57 0"/>
         <geometry>
           <cylinder>
@@ -386,38 +386,38 @@
       </visual>
       <visual>
-        <pose>0.11 -0.01 -0.005 0 0 0.37</pose>
-        <geometry>
-          <box>
-            <size>0.09 .03 .06</size>
-          </box>
-        </geometry>
-        <material name="${side}_sandia_hand_skin">
-          <color rgba="0.835 0.655 0.345 1.0"/>
-        </material>
-      </visual>
-      <visual>
-        <pose>0.09 0.02 -0.005 0 0 0.37</pose>
-        <geometry>
-          <box>
-            <size>0.09 .03 .06</size>
-          </box>
-        </geometry>
-        <material name="${side}_sandia_hand_skin">
-          <color rgba="0.835 0.655 0.345 1.0"/>
-        </material>
-      </visual>
-      <visual>
-        <pose>0.060 0.050 -0.005 0 0 0.37</pose>
-        <geometry>
-          <box>
-            <size>0.09 .03 .06</size>
-          </box>
-        </geometry>
-        <material name="${side}_sandia_hand_skin">
-          <color rgba="0.835 0.655 0.345 1.0"/>
-        </material>
-      </visual>
-      <visual>
-        <pose>0.044 -0.04 -0.005 0 0 0.79</pose>
+        <origin xyz="0.11 -0.01 -0.005" rpy="0 0 0.37"/>
+        <geometry>
+          <box>
+            <size>0.09 .03 .06</size>
+          </box>
+        </geometry>
+        <material name="${side}_sandia_hand_skin">
+          <color rgba="0.835 0.655 0.345 1.0"/>
+        </material>
+      </visual>
+      <visual>
+        <origin xyz="0.09 0.02 -0.005" rpy="0 0 0.37"/>
+        <geometry>
+          <box>
+            <size>0.09 .03 .06</size>
+          </box>
+        </geometry>
+        <material name="${side}_sandia_hand_skin">
+          <color rgba="0.835 0.655 0.345 1.0"/>
+        </material>
+      </visual>
+      <visual>
+        <origin xyz="0.060 0.050 -0.005" rpy="0 0 0.37"/>
+        <geometry>
+          <box>
+            <size>0.09 .03 .06</size>
+          </box>
+        </geometry>
+        <material name="${side}_sandia_hand_skin">
+          <color rgba="0.835 0.655 0.345 1.0"/>
+        </material>
+      </visual>
+      <visual>
+        <origin xyz="0.044 -0.04 -0.005" rpy="0 0 0.79"/>
         <geometry>
           <box>
