Commit message: Fix shape syntax in urdf

File: ros/sandia_hand_description/urdf/sandia_hand.urdf.xacro (robot description, xacro)
@@ -32,8 +32,8 @@
         <origin xyz="0 0 0.003" rpy="0 0 0"/>
         <geometry>
-          <cylinder>
-            <radius>0.015</radius>
-            <length>0.023</length>
-          </cylinder>
+          <cylinder
+            radius="0.015"
+            length="0.023"
+          />
         </geometry>
       </collision>
@@ -41,8 +41,8 @@
         <origin xyz="0.011 0 0.003" rpy="1.57 0 0"/>
         <geometry>
-          <cylinder>
-            <radius>0.01</radius>
-            <length>0.023</length>
-          </cylinder>
+          <cylinder
+            radius="0.01"
+            length="0.023"
+          />
         </geometry>
       </collision>
@@ -52,8 +52,8 @@
         <origin xyz="0 0 0.003" rpy="0 0 0"/>
         <geometry>
-          <cylinder>
-            <radius>0.015</radius>
-            <length>0.023</length>
-          </cylinder>
+          <cylinder
+            radius="0.015"
+            length="0.023"
+          />
         </geometry>
         <material name="${side}_sandia_hand_skin_suntan">
@@ -64,8 +64,8 @@
         <origin xyz="0.011 0 0.003" rpy="1.57 0 0"/>
         <geometry>
-          <cylinder>
-            <radius>0.01</radius>
-            <length>0.023</length>
-          </cylinder>
+          <cylinder
+            radius="0.01"
+            length="0.023"
+          />
         </geometry>
         <material name="${side}_sandia_hand_skin_suntan">
@@ -105,8 +105,8 @@
         <origin xyz="0.024 0 0" rpy="0 1.57 0"/>
         <geometry>
-          <cylinder>
-            <radius>0.01</radius>
-            <length>0.067</length>
-          </cylinder>
+          <cylinder
+            radius="0.01"
+            length="0.067"
+          />
         </geometry>
       </collision>
@@ -116,8 +116,8 @@
         <origin xyz="0.024 0 0" rpy="0 1.57 0"/>
         <geometry>
-          <cylinder>
-            <radius>0.01</radius>
-            <length>0.067</length>
-          </cylinder>
+          <cylinder
+            radius="0.01"
+            length="0.067"
+          />
         </geometry>
         <material name="${side}_sandia_hand_skin">
@@ -165,8 +165,8 @@
         <origin xyz="0.024 0 0" rpy="0 1.57 0"/>
         <geometry>
-          <cylinder>
-            <radius>0.009</radius>
-            <length>0.057</length>
-          </cylinder>
+          <cylinder
+            radius="0.009"
+            length="0.057"
+          />
         </geometry>
       </collision>
@@ -174,7 +174,5 @@
         <origin xyz="0.052 0 0" rpy="0 0 0"/>
         <geometry>
-          <sphere>
-            <radius>0.009</radius>
-          </sphere>
+          <sphere radius="0.009" />
         </geometry>
       </collision>
@@ -184,8 +182,8 @@
         <origin xyz="0.024 0 0" rpy="0 1.57 0"/>
         <geometry>
-          <cylinder>
-            <radius>0.009</radius>
-            <length>0.057</length>
-          </cylinder>
+          <cylinder
+            radius="0.009"
+            length="0.057"
+          />
         </geometry>
         <material name="${side}_sandia_hand_skin_suntan">
@@ -196,7 +194,5 @@
         <origin xyz="0.052 0 0" rpy="0 0 0"/>
         <geometry>
-          <sphere>
-            <radius>0.009</radius>
-          </sphere>
+          <sphere radius="0.009" />
         </geometry>
         <material name="${side}_sandia_hand_skin_suntan">
@@ -293,8 +289,8 @@
         <origin xyz="0.069 0.016 0.038" rpy="0 1.57 -0.9"/>
         <geometry>
-          <cylinder>
-            <radius>0.013</radius>
-            <length>0.100</length>
-          </cylinder>
+          <cylinder
+            radius="0.013"
+            length="0.100"
+          />
         </geometry>
       </collision>
@@ -302,7 +298,5 @@
         <origin xyz="0.064 0.008 0.021" rpy="0.41 0 -0.9"/>
         <geometry>
-          <box>
-            <size>0.09 .035 .05</size>
-          </box>
+          <box size="0.09 .035 .05" />
         </geometry>
       </collision>
@@ -310,8 +304,8 @@
         <origin xyz="0.02 0 -0.005" rpy="0 1.57 0"/>
         <geometry>
-          <cylinder>
-            <radius>0.038</radius>
-            <length>0.05</length>
-          </cylinder>
+          <cylinder
+            radius="0.038"
+            length="0.05"
+          />
         </geometry>
       </collision>
@@ -319,7 +313,5 @@
         <origin xyz="0.11 -0.01 -0.005" rpy="0 0 0.37"/>
         <geometry>
-          <box>
-            <size>0.09 .03 .06</size>
-          </box>
+          <box size="0.09 .03 .06" />
         </geometry>
       </collision>
@@ -327,7 +319,5 @@
         <origin xyz="0.09 0.02 -0.005" rpy="0 0 0.37"/>
         <geometry>
-          <box>
-            <size>0.09 .03 .06</size>
-          </box>
+          <box size="0.09 .03 .06" />
         </geometry>
       </collision>
@@ -335,7 +325,5 @@
         <origin xyz="0.060 0.050 -0.005" rpy="0 0 0.37"/>
         <geometry>
-          <box>
-            <size>0.09 .03 .06</size>
-          </box>
+          <box size="0.09 .03 .06" />
         </geometry>
       </collision>
@@ -343,7 +331,5 @@
         <origin xyz="0.044 -0.04 -0.005" rpy="0 0 0.79"/>
         <geometry>
-          <box>
-            <size>0.09 .03 .06</size>
-          </box>
+          <box size="0.09 .03 .06" />
         </geometry>
       </collision>
@@ -353,8 +339,8 @@
         <origin xyz="0.069 0.016 0.038" rpy="0 1.57 -0.9"/>
         <geometry>
-          <cylinder>
-            <radius>0.013</radius>
-            <length>0.100</length>
-          </cylinder>
+          <cylinder
+            radius="0.013"
+            length="0.100"
+          />
         </geometry>
         <material name="${side}_sandia_hand_skin">
@@ -365,7 +351,5 @@
         <origin xyz="0.064 0.008 0.021" rpy="0.41 0 -0.9"/>
         <geometry>
-          <box>
-            <size>0.09 .035 .05</size>
-          </box>
+          <box size="0.09 .035 .05" />
         </geometry>
         <material name="${side}_sandia_hand_skin">
@@ -376,8 +360,8 @@
         <origin xyz="0.02 0 -0.005" rpy="0 1.57 0"/>
         <geometry>
-          <cylinder>
-            <radius>0.038</radius>
-            <length>0.05</length>
-          </cylinder>
+          <cylinder
+            radius="0.038"
+            length="0.05"
+          />
         </geometry>
         <material name="${side}_sandia_hand_skin">
@@ -388,7 +372,5 @@
         <origin xyz="0.11 -0.01 -0.005" rpy="0 0 0.37"/>
         <geometry>
-          <box>
-            <size>0.09 .03 .06</size>
-          </box>
+          <box size="0.09 .03 .06" />
         </geometry>
         <material name="${side}_sandia_hand_skin">
@@ -399,7 +381,5 @@
         <origin xyz="0.09 0.02 -0.005" rpy="0 0 0.37"/>
         <geometry>
-          <box>
-            <size>0.09 .03 .06</size>
-          </box>
+          <box size="0.09 .03 .06" />
         </geometry>
         <material name="${side}_sandia_hand_skin">
@@ -410,7 +390,5 @@
         <origin xyz="0.060 0.050 -0.005" rpy="0 0 0.37"/>
         <geometry>
-          <box>
-            <size>0.09 .03 .06</size>
-          </box>
+          <box size="0.09 .03 .06" />
         </geometry>
         <material name="${side}_sandia_hand_skin">
@@ -421,7 +399,5 @@
         <origin xyz="0.044 -0.04 -0.005" rpy="0 0 0.79"/>
         <geometry>
-          <box>
-            <size>0.09 .03 .06</size>
-          </box>
+          <box size="0.09 .03 .06" />
         </geometry>
         <material name="${side}_sandia_hand_skin">

Commit message: address drcsim issue #400 (https://bitbucket.org/osrf/drcsim/issue/400/accurate-models-for-atlas-irobot-and) by copying inertia from sandia_hand_simple_shapes.urdf.xacro into sandia_hand.urdf.xacro.

File: ros/sandia_hand_description/urdf/sandia_hand.urdf.xacro (robot description, xacro)
@@ -4,11 +4,18 @@
   <xacro:include filename="$(find sandia_hand_description)/urdf/sandia_hand.gazebo.xacro" />
   <xacro:include filename="$(find sandia_hand_description)/urdf/sandia_hand.transmission.xacro" />
-  <xacro:macro name="finger" params="idx x y z r p yaw side">
+  <xacro:property name="M_pi" value="3.1415926535897931" />
+  <xacro:property name="damping_coefficient_j0" value="1.0" />
+  <xacro:property name="damping_coefficient_j1" value="1.0" />
+  <xacro:property name="damping_coefficient_j2" value="1.0" />
+  <xacro:property name="velocity_limit" value="-1" />
+  <xacro:macro name="finger" params="idx x y z r p yaw side reflect joint_type">
     <link name="${side}_f${idx}_base">
       <origin xyz="0 0 0" rpy="0 0 0"/>
       <inertial>
-        <mass value="0.1"/>
-        <origin xyz="0 0 0"/>
-        <inertia ixx="0.01" ixy="0" ixz="0" iyy="0.01" iyz="0" izz="0.01"/>
+        <!-- total mass is 2.303 kg, palm is about 1.303 kg, distribute the rest into _base -->
+        <mass value="0.250"/> <!-- (2.303 - 1.303) / 4 -->
+        <origin xyz="0 0 0"/>
+        <!-- model as sphere with radius of 1cm -->
+        <inertia ixx="0.00001" ixy="0" ixz="0" iyy="0.00001" iyz="0" izz="0.00001"/>
       </inertial>
     </link>
@@ -16,7 +23,7 @@
       <origin xyz="0 0 0" rpy="0 0 0"/>
       <inertial>
-        <mass value="0.1"/>
-        <origin xyz="0 0 0"/>
-        <inertia ixx="0.01" ixy="0" ixz="0" iyy="0.01" iyz="0" izz="0.01"/>
+        <mass value="0.01"/>
+        <origin xyz="0 0 0"/>
+        <inertia ixx="0.000001" ixy="0" ixz="0" iyy="0.000001" iyz="0" izz="0.000001"/>
       </inertial>
     </link>
@@ -24,7 +31,8 @@
       <origin xyz="0 0 0" rpy="0 0 0"/>
       <inertial>
-        <mass value="0.1"/>
-        <origin xyz="0 0 0"/>
-        <inertia ixx="0.01" ixy="0" ixz="0" iyy="0.01" iyz="0" izz="0.01"/>
+        <mass value="0.106"/> <!-- F1 -->
+        <origin xyz="0 0 0"/>
+        <!-- solid cylinder -->
+        <inertia ixx="0.000011925" ixy="0" ixz="0" iyy="0.00011505" iyz="0" izz="0.00011505"/>
       </inertial>
       <collision>
@@ -47,7 +55,8 @@
       <origin xyz="0 0 0" rpy="0 0 0"/>
       <inertial>
-        <mass value="0.1"/>
-        <origin xyz="0 0 0"/>
-        <inertia ixx="0.01" ixy="0" ixz="0" iyy="0.01" iyz="0" izz="0.01"/>
+        <mass value="0.033"/> <!-- F2 -->
+        <origin xyz="0 0 0"/>
+        <!-- solid cylinder -->
+        <inertia ixx="0.00000165" ixy="0" ixz="0" iyy="0.00001316975" iyz="0" izz="0.00001316975"/>
       </inertial>
       <collision>
@@ -70,7 +79,7 @@
       <origin xyz="0 0 0" rpy="0 0 0"/>
       <inertial>
-        <mass value="0.1"/>
-        <origin xyz="0 0 0"/>
-        <inertia ixx="0.01" ixy="0" ixz="0" iyy="0.01" iyz="0" izz="0.01"/>
+        <mass value="0.01"/>
+        <origin xyz="0 0 0"/>
+        <inertia ixx="0.000001" ixy="0" ixz="0" iyy="0.000001" iyz="0" izz="0.000001"/>
       </inertial>
     </link>
@@ -78,7 +87,8 @@
       <origin xyz="0 0 0" rpy="0 0 0"/>
       <inertial>
-        <mass value="0.1"/>
-        <origin xyz="0 0 0"/>
-        <inertia ixx="0.01" ixy="0" ixz="0" iyy="0.01" iyz="0" izz="0.01"/>
+        <mass value="0.033"/>  <!-- F3 -->
+        <origin xyz="0 0 0"/>
+        <!-- solid cylinder -->
+        <inertia ixx="0.0000013365" ixy="0" ixz="0" iyy="0.000009603" iyz="0" izz="0.000009603"/>
       </inertial>
       <collision>
@@ -101,7 +111,7 @@
       <origin xyz="0 0 0" rpy="0 0 0"/>
       <inertial>
-        <mass value="0.1"/>
-        <origin xyz="0 0 0"/>
-        <inertia ixx="0.01" ixy="0" ixz="0" iyy="0.01" iyz="0" izz="0.01"/>
+        <mass value="0.01"/>
+        <origin xyz="0 0 0"/>
+        <inertia ixx="0.000001" ixy="0" ixz="0" iyy="0.000001" iyz="0" izz="0.000001"/>
       </inertial>
     </link>
@@ -111,23 +121,23 @@
       <origin xyz="${x} ${y} ${z}" rpy="${r} ${p} ${yaw}"/>
     </joint>
-    <joint name="${side}_f${idx}_j0" type="revolute">
-      <axis xyz="0 0 1"/>
+    <joint name="${side}_f${idx}_j0" type="${joint_type}">
+      <axis xyz="0 0 ${reflect}"/>
       <parent link="${side}_f${idx}_base"/>
       <child link="${side}_f${idx}_0"/>
-      <limit lower="-1.57079" upper="1.57079" effort="1" velocity="1"/>
+      <limit lower="-${M_pi/2}" upper="${M_pi/2}" effort="11" velocity="${velocity_limit}"/>
       <safety_controller soft_lower_limit="${-1.57079-10.0}" soft_upper_limit="${1.57079+10.0}" k_position="1000.0" k_velocity="1000.0"/>
-      <dynamics damping="0.1"/>
-      <origin xyz="0 0 0" rpy="0 0 0"/>
-    </joint>
-    <joint name="${side}_f${idx}_j1" type="revolute">
+      <dynamics damping="${damping_coefficient_j0}"/>
+      <origin xyz="0 0 0" rpy="0 0 0"/>
+    </joint>
+    <joint name="${side}_f${idx}_j1" type="${joint_type}">
       <axis xyz="0 0 1"/>
       <parent link="${side}_f${idx}_0"/>
       <child link="${side}_f${idx}_1"/>
-      <limit lower="-1.57079" upper="1.57079" effort="1" velocity="1"/>
+      <limit lower="-${M_pi/2}" upper="${M_pi/2}" effort="28" velocity="${velocity_limit}"/>
       <safety_controller soft_lower_limit="${-1.57079-10.0}" soft_upper_limit="${1.57079+10.0}" k_position="1000.0" k_velocity="1000.0"/>
-      <dynamics damping="0.1"/>
-      <origin xyz="0.028 0 0" rpy="1.57079 0 0"/>
-    </joint>
-    <joint name="${side}_f${idx}_j2" type="revolute">
+      <dynamics damping="${damping_coefficient_j1}"/>
+      <origin xyz="0.028 0 0" rpy="${M_pi/2} 0 0"/>
+    </joint>
+    <joint name="${side}_f${idx}_j2" type="${joint_type}">
       <axis xyz="0 0 1"/>
       <parent link="${side}_f${idx}_1"/>
@@ -135,6 +145,6 @@
       <origin xyz="0.05 0 0" rpy="0 0 0"/>
       <safety_controller soft_lower_limit="${-1.57079-10.0}" soft_upper_limit="${1.57079+10.0}" k_position="1000.0" k_velocity="1000.0"/>
-      <dynamics damping="0.1"/>
-      <limit lower="-1.57079" upper="1.57079" effort="1" velocity="1"/>
+      <dynamics damping="${damping_coefficient_j2}"/>
+      <limit lower="-${M_pi/2}" upper="${M_pi/2}" effort="28" velocity="${velocity_limit}"/>
     </joint>
     <joint name="${side}_f${idx}_fixed_accel" type="fixed">
@@ -146,21 +156,22 @@
       <parent link="${side}_f${idx}_1"/>
       <child link="${side}_f${idx}_1_accel"/>
-      <origin xyz="0.03 0 0" rpy="-1.5709 0 0"/>
+      <origin xyz="0.03 0 0" rpy="-${M_pi/2} 0 0"/>
     </joint>
     <joint name="${side}_f${idx}_2_accel" type="fixed">
       <parent link="${side}_f${idx}_2"/>
       <child link="${side}_f${idx}_2_accel"/>
-      <origin xyz="0.04 0 0" rpy="-1.5709 0 0"/>
+      <origin xyz="0.04 0 0" rpy="-${M_pi/2} 0 0"/>
     </joint>
     <xacro:finger_transmission side="${side}" idx="${idx}" x="${x}" y="${y}" z="${z}" r="${r}" p="${p}" yaw="${yaw}"/>
     <xacro:finger_gazebo side="${side}" idx="${idx}"/>
   </xacro:macro>
-  <xacro:macro name="sandia_hand" params="side parent *origin">
+  <xacro:macro name="sandia_hand" params="side parent reflect joint_type thumb_angle *origin">
     <link name="${side}_palm">
       <origin xyz="0 0 0" rpy="0 0 0"/>
       <inertial>
-        <mass value="0.1"/>
-        <origin xyz="0 0 0"/>
-        <inertia ixx="0.01" ixy="0" ixz="0" iyy="0.01" iyz="0" izz="0.01"/>
+        <mass value="1.303"/>
+        <origin xyz="0 0 0"/>
+        <!-- solid sphere with 5cm radius -->
+        <inertia ixx="0.001303" ixy="0" ixz="0" iyy="0.001303" iyz="0" izz="0.001303"/>
       </inertial>
       <collision>
@@ -185,12 +196,15 @@
       <insert_block name="origin" />
     </joint>
-    <xacro:finger side="${side}" idx="0" x="0.140" y="0.00000" z="0" r="0" p="0" yaw="0.3"/>
-    <xacro:finger side="${side}" idx="1" x="0.115" y="0.03122" z="0" r="0" p="0" yaw="0.3"/>
-    <xacro:finger side="${side}" idx="2" x="0.090" y="0.06245" z="0" r="0" p="0" yaw="0.3"/>
-    <xacro:finger side="${side}" idx="3" x="0.03995" y="-0.04383" z="0.014" r="0" p="-1.57079" yaw="-2.3562"/>
+    <xacro:finger side="${side}" idx="0" x="0.140" y="0.00000" z="0" r="0" p="0" yaw="${0.3*reflect}" reflect="${reflect}" joint_type="${joint_type}"/>
+    <xacro:finger side="${side}" idx="1" x="0.115" y="${0.03122*reflect}" z="0" r="0" p="0" yaw="${0.3*reflect}" reflect="${reflect}" joint_type="${joint_type}"/>
+    <xacro:finger side="${side}" idx="2" x="0.090" y="${0.06245*reflect}" z="0" r="0" p="0" yaw="${0.3*reflect}" reflect="${reflect}" joint_type="${joint_type}"/>
+    <xacro:finger side="${side}" idx="3" x="0.03995" y="${-0.04383*reflect}" z="0.014" r="0" p="-${M_pi/2 + thumb_angle}" yaw="${-(2.3562+thumb_angle)*reflect}" reflect="${reflect}" joint_type="${joint_type}"/>
     <!-- not needed unless simulating the hand by itself
     <xacro:sandia_hand_gazebo_controller side="${side}" />
     -->
     <xacro:sandia_hand_gazebo side="${side}" />
+    <xacro:sandia_hand_cameras_gazebo side="${side}" reflect="${reflect}" parent="${parent}" />
+    <xacro:sandia_hand_tactile_sensors_gazebo side="${side}" parent="${parent}" />
+    <xacro:sandia_hand_imu_sensor_gazebo parent="${parent}" />
   </xacro:macro>
 </robot>
