Commit message: Isolate simple collision shape changes to separate file

File: ros/sandia_hand_description/urdf/sandia_hand_simple_shapes.urdf.xacro (robot description, xacro)
@@ -28,4 +28,51 @@
         <inertia ixx="0.01" ixy="0" ixz="0" iyy="0.01" iyz="0" izz="0.01"/>
       </inertial>
+      <!-- begin simple shape approximation of f0 -->
+      <collision>
+        <origin xyz="0 0 0.003" rpy="0 0 0"/>
+        <geometry>
+          <cylinder
+            radius="0.015"
+            length="0.023"
+          />
+        </geometry>
+      </collision>
+      <collision>
+        <origin xyz="0.011 0 0.003" rpy="1.57 0 0"/>
+        <geometry>
+          <cylinder
+            radius="0.01"
+            length="0.023"
+          />
+        </geometry>
+      </collision>
+      <!--   end simple shape approximation of f0 -->
+      <!-- begin visual shape approximation of f0 -->
+      <visual>
+        <origin xyz="0 0 0.003" rpy="0 0 0"/>
+        <geometry>
+          <cylinder
+            radius="0.015"
+            length="0.023"
+          />
+        </geometry>
+        <material name="${side}_sandia_hand_skin_suntan">
+          <color rgba="0.7 0.4 0.2 1.0"/>
+        </material>
+      </visual>
+      <visual>
+        <origin xyz="0.011 0 0.003" rpy="1.57 0 0"/>
+        <geometry>
+          <cylinder
+            radius="0.01"
+            length="0.023"
+          />
+        </geometry>
+        <material name="${side}_sandia_hand_skin_suntan">
+          <color rgba="0.7 0.4 0.2 1.0"/>
+        </material>
+      </visual>
+      <!--   end visual shape approximation of f0 -->
+      <!-- begin collision mesh of f0 ->
       <collision>
         <origin xyz="0 0 0" rpy="0 0 0"/>
@@ -34,4 +81,6 @@
         </geometry>
       </collision>
+      <!-   end collision mesh of f0 -->
+      <!-- begin visual mesh of f0 ->
       <visual>
         <origin xyz="0 0 0" rpy="0 0 0"/>
@@ -43,4 +92,5 @@
         </material>
       </visual>
+      <!-   end visual mesh of f0 -->
     </link>
     <link name="${side}_f${idx}_1">
@@ -51,4 +101,30 @@
         <inertia ixx="0.01" ixy="0" ixz="0" iyy="0.01" iyz="0" izz="0.01"/>
       </inertial>
+      <!-- begin simple shape approximation of f1 -->
+      <collision>
+        <origin xyz="0.024 0 0" rpy="0 1.57 0"/>
+        <geometry>
+          <cylinder
+            radius="0.01"
+            length="0.067"
+          />
+        </geometry>
+      </collision>
+      <!--   end simple shape approximation of f1 -->
+      <!-- begin visual shape approximation of f1 -->
+      <visual>
+        <origin xyz="0.024 0 0" rpy="0 1.57 0"/>
+        <geometry>
+          <cylinder
+            radius="0.01"
+            length="0.067"
+          />
+        </geometry>
+        <material name="${side}_sandia_hand_skin">
+          <color rgba="0.835 0.655 0.345 1.0"/>
+        </material>
+      </visual>
+      <!--   end visual shape approximation of f1 -->
+      <!-- begin collision mesh of f1 ->
       <collision>
         <origin xyz="0 0 0" rpy="0 0 0"/>
@@ -57,4 +133,6 @@
         </geometry>
       </collision>
+      <!-   end collision mesh of f1 -->
+      <!-- begin visual mesh of f1 ->
       <visual>
         <origin xyz="0 0 0" rpy="0 0 0"/>
@@ -66,4 +144,5 @@
         </material>
       </visual>
+      <!-   end visual mesh of f1 -->
     </link>
     <link name="${side}_f${idx}_1_accel">
@@ -82,4 +161,44 @@
         <inertia ixx="0.01" ixy="0" ixz="0" iyy="0.01" iyz="0" izz="0.01"/>
       </inertial>
+      <!-- begin simple shape approximation of f2 -->
+      <collision>
+        <origin xyz="0.024 0 0" rpy="0 1.57 0"/>
+        <geometry>
+          <cylinder
+            radius="0.009"
+            length="0.057"
+          />
+        </geometry>
+      </collision>
+      <collision>
+        <origin xyz="0.052 0 0" rpy="0 0 0"/>
+        <geometry>
+          <sphere radius="0.009" />
+        </geometry>
+      </collision>
+      <!--   end simple shape approximation of f2 -->
+      <!-- begin visual shape approximation of f2 -->
+      <visual>
+        <origin xyz="0.024 0 0" rpy="0 1.57 0"/>
+        <geometry>
+          <cylinder
+            radius="0.009"
+            length="0.057"
+          />
+        </geometry>
+        <material name="${side}_sandia_hand_skin_suntan">
+          <color rgba="0.8 0.6 0.3 1.0"/>
+        </material>
+      </visual>
+      <visual>
+        <origin xyz="0.052 0 0" rpy="0 0 0"/>
+        <geometry>
+          <sphere radius="0.009" />
+        </geometry>
+        <material name="${side}_sandia_hand_skin_suntan">
+          <color rgba="0.8 0.6 0.3 1.0"/>
+        </material>
+      </visual>
+      <!-- begin collision mesh of f2    ->
       <collision>
         <origin xyz="0 0 0" rpy="0 0 0"/>
@@ -88,4 +207,6 @@
         </geometry>
       </collision>
+      <!-   end collision mesh of f2 -->
+      <!-- begin visual mesh of f2    ->
       <visual>
         <origin xyz="0 0 0" rpy="0 0 0"/>
@@ -97,4 +218,5 @@
         </material>
       </visual>
+      <!-   end visual mesh of f2 -->
     </link>
     <link name="${side}_f${idx}_2_accel">
@@ -163,4 +285,126 @@
         <inertia ixx="0.01" ixy="0" ixz="0" iyy="0.01" iyz="0" izz="0.01"/>
       </inertial>
+      <!-- begin simple shape approximation of palm -->
+      <collision>
+        <origin xyz="0.069 0.016 0.038" rpy="0 1.57 -0.9"/>
+        <geometry>
+          <cylinder
+            radius="0.013"
+            length="0.100"
+          />
+        </geometry>
+      </collision>
+      <collision>
+        <origin xyz="0.064 0.008 0.021" rpy="0.41 0 -0.9"/>
+        <geometry>
+          <box size="0.09 .035 .05" />
+        </geometry>
+      </collision>
+      <collision>
+        <origin xyz="0.02 0 -0.005" rpy="0 1.57 0"/>
+        <geometry>
+          <cylinder
+            radius="0.038"
+            length="0.05"
+          />
+        </geometry>
+      </collision>
+      <collision>
+        <origin xyz="0.11 -0.01 -0.005" rpy="0 0 0.37"/>
+        <geometry>
+          <box size="0.09 .03 .06" />
+        </geometry>
+      </collision>
+      <collision>
+        <origin xyz="0.09 0.02 -0.005" rpy="0 0 0.37"/>
+        <geometry>
+          <box size="0.09 .03 .06" />
+        </geometry>
+      </collision>
+      <collision>
+        <origin xyz="0.060 0.050 -0.005" rpy="0 0 0.37"/>
+        <geometry>
+          <box size="0.09 .03 .06" />
+        </geometry>
+      </collision>
+      <collision>
+        <origin xyz="0.044 -0.04 -0.005" rpy="0 0 0.79"/>
+        <geometry>
+          <box size="0.09 .03 .06" />
+        </geometry>
+      </collision>
+      <!--   end simple shape approximation of palm -->
+      <!-- begin visual shape approximation of palm -->
+      <visual>
+        <origin xyz="0.069 0.016 0.038" rpy="0 1.57 -0.9"/>
+        <geometry>
+          <cylinder
+            radius="0.013"
+            length="0.100"
+          />
+        </geometry>
+        <material name="${side}_sandia_hand_skin">
+          <color rgba="0.835 0.655 0.345 1.0"/>
+        </material>
+      </visual>
+      <visual>
+        <origin xyz="0.064 0.008 0.021" rpy="0.41 0 -0.9"/>
+        <geometry>
+          <box size="0.09 .035 .05" />
+        </geometry>
+        <material name="${side}_sandia_hand_skin">
+          <color rgba="0.835 0.655 0.345 1.0"/>
+        </material>
+      </visual>
+      <visual>
+        <origin xyz="0.02 0 -0.005" rpy="0 1.57 0"/>
+        <geometry>
+          <cylinder
+            radius="0.038"
+            length="0.05"
+          />
+        </geometry>
+        <material name="${side}_sandia_hand_skin">
+          <color rgba="0.835 0.655 0.345 1.0"/>
+        </material>
+      </visual>
+      <visual>
+        <origin xyz="0.11 -0.01 -0.005" rpy="0 0 0.37"/>
+        <geometry>
+          <box size="0.09 .03 .06" />
+        </geometry>
+        <material name="${side}_sandia_hand_skin">
+          <color rgba="0.835 0.655 0.345 1.0"/>
+        </material>
+      </visual>
+      <visual>
+        <origin xyz="0.09 0.02 -0.005" rpy="0 0 0.37"/>
+        <geometry>
+          <box size="0.09 .03 .06" />
+        </geometry>
+        <material name="${side}_sandia_hand_skin">
+          <color rgba="0.835 0.655 0.345 1.0"/>
+        </material>
+      </visual>
+      <visual>
+        <origin xyz="0.060 0.050 -0.005" rpy="0 0 0.37"/>
+        <geometry>
+          <box size="0.09 .03 .06" />
+        </geometry>
+        <material name="${side}_sandia_hand_skin">
+          <color rgba="0.835 0.655 0.345 1.0"/>
+        </material>
+      </visual>
+      <visual>
+        <origin xyz="0.044 -0.04 -0.005" rpy="0 0 0.79"/>
+        <geometry>
+          <box size="0.09 .03 .06" />
+        </geometry>
+        <material name="${side}_sandia_hand_skin">
+          <color rgba="0.835 0.655 0.345 1.0"/>
+        </material>
+      </visual>
+      <!--   end visual shape approximation of palm -->
+      <!-- begin collision mesh of f2 ->
       <collision>
         <origin xyz="0 0 0" rpy="0 0 0"/>
@@ -169,4 +413,6 @@
         </geometry>
       </collision>
+      <!-   end collision mesh of f2 -->
+      <!-- begin visual mesh of f2    ->
       <visual>
         <origin xyz="0 0 0" rpy="0 0 0"/>
@@ -178,4 +424,5 @@
         </material>
       </visual>
+      <!-   end visual mesh of f2 -->
     </link>
     <joint name="${side}_sandia_hand_joint" type="fixed">

Commit message: Put cylinder elements on a single line

File: ros/sandia_hand_description/urdf/sandia_hand_simple_shapes.urdf.xacro (robot description, xacro)
@@ -32,8 +32,5 @@
         <origin xyz="0 0 0.003" rpy="0 0 0"/>
         <geometry>
-          <cylinder
-            radius="0.015"
-            length="0.023"
-          />
+          <cylinder radius="0.015" length="0.023" />
         </geometry>
       </collision>
@@ -41,8 +38,5 @@
         <origin xyz="0.011 0 0.003" rpy="1.57 0 0"/>
         <geometry>
-          <cylinder
-            radius="0.01"
-            length="0.023"
-          />
+          <cylinder radius="0.01" length="0.023" />
         </geometry>
       </collision>
@@ -52,8 +46,5 @@
         <origin xyz="0 0 0.003" rpy="0 0 0"/>
         <geometry>
-          <cylinder
-            radius="0.015"
-            length="0.023"
-          />
+          <cylinder radius="0.015" length="0.023" />
         </geometry>
         <material name="${side}_sandia_hand_skin_suntan">
@@ -64,8 +55,5 @@
         <origin xyz="0.011 0 0.003" rpy="1.57 0 0"/>
         <geometry>
-          <cylinder
-            radius="0.01"
-            length="0.023"
-          />
+          <cylinder radius="0.01" length="0.023" />
         </geometry>
         <material name="${side}_sandia_hand_skin_suntan">
@@ -105,8 +93,5 @@
         <origin xyz="0.024 0 0" rpy="0 1.57 0"/>
         <geometry>
-          <cylinder
-            radius="0.01"
-            length="0.067"
-          />
+          <cylinder radius="0.01" length="0.067" />
         </geometry>
       </collision>
@@ -116,8 +101,5 @@
         <origin xyz="0.024 0 0" rpy="0 1.57 0"/>
         <geometry>
-          <cylinder
-            radius="0.01"
-            length="0.067"
-          />
+          <cylinder radius="0.01" length="0.067" />
         </geometry>
         <material name="${side}_sandia_hand_skin">
@@ -165,8 +147,5 @@
         <origin xyz="0.024 0 0" rpy="0 1.57 0"/>
         <geometry>
-          <cylinder
-            radius="0.009"
-            length="0.057"
-          />
+          <cylinder radius="0.009" length="0.057" />
         </geometry>
       </collision>
@@ -182,8 +161,5 @@
         <origin xyz="0.024 0 0" rpy="0 1.57 0"/>
         <geometry>
-          <cylinder
-            radius="0.009"
-            length="0.057"
-          />
+          <cylinder radius="0.009" length="0.057" />
         </geometry>
         <material name="${side}_sandia_hand_skin_suntan">
@@ -289,8 +265,5 @@
         <origin xyz="0.069 0.016 0.038" rpy="0 1.57 -0.9"/>
         <geometry>
-          <cylinder
-            radius="0.013"
-            length="0.100"
-          />
+          <cylinder radius="0.013" length="0.100" />
         </geometry>
       </collision>
@@ -304,8 +277,5 @@
         <origin xyz="0.02 0 -0.005" rpy="0 1.57 0"/>
         <geometry>
-          <cylinder
-            radius="0.038"
-            length="0.05"
-          />
+          <cylinder radius="0.038" length="0.05" />
         </geometry>
       </collision>
@@ -339,8 +309,5 @@
         <origin xyz="0.069 0.016 0.038" rpy="0 1.57 -0.9"/>
         <geometry>
-          <cylinder
-            radius="0.013"
-            length="0.100"
-          />
+          <cylinder radius="0.013" length="0.100" />
         </geometry>
         <material name="${side}_sandia_hand_skin">
@@ -360,8 +327,5 @@
         <origin xyz="0.02 0 -0.005" rpy="0 1.57 0"/>
         <geometry>
-          <cylinder
-            radius="0.038"
-            length="0.05"
-          />
+          <cylinder radius="0.038" length="0.05" />
         </geometry>
         <material name="${side}_sandia_hand_skin">

Commit message: Bracket error in xacro

File: ros/sandia_hand_description/urdf/sandia_hand_simple_shapes.urdf.xacro (robot description, xacro)
@@ -270,5 +270,5 @@
       </collision>
       <collision>
-        <origin xyz="0.064 $(0.008 * reflect} 0.021" rpy="0.41 0 ${-0.9 * reflect}"/>
+        <origin xyz="0.064 ${0.008 * reflect} 0.021" rpy="0.41 0 ${-0.9 * reflect}"/>
         <geometry>
           <box size="0.09 .035 .05" />

Commit message: Add group names to collisions in sandia_hand_simple_shapes to prevent a million warnings when loading gazebo

File: ros/sandia_hand_description/urdf/sandia_hand_simple_shapes.urdf.xacro (robot description, xacro)
@@ -30,5 +30,5 @@
       </inertial>
       <!-- begin simple shape approximation of f0 -->
-      <collision>
+      <collision group="default">
         <origin xyz="0 0 0.003" rpy="0 0 0"/>
         <geometry>
@@ -36,5 +36,5 @@
         </geometry>
       </collision>
-      <collision>
+      <collision group="other">
         <origin xyz="0.011 0 0.003" rpy="${M_pi/2} 0 0"/>
         <geometry>
@@ -64,5 +64,5 @@
       <!--   end visual shape approximation of f0 -->
       <!-- begin collision mesh of f0 ->
-      <collision>
+      <collision group="default">
         <origin xyz="0 0 0" rpy="0 0 0"/>
         <geometry>
@@ -91,5 +91,5 @@
       </inertial>
       <!-- begin simple shape approximation of f1 -->
-      <collision>
+      <collision group="default">
         <origin xyz="0.024 0 0" rpy="0 ${M_pi/2} 0"/>
         <geometry>
@@ -110,5 +110,5 @@
       <!--   end visual shape approximation of f1 -->
       <!-- begin collision mesh of f1 ->
-      <collision>
+      <collision group="default">
         <origin xyz="0 0 0" rpy="0 0 0"/>
         <geometry>
@@ -145,5 +145,5 @@
       </inertial>
       <!-- begin simple shape approximation of f2 -->
-      <collision>
+      <collision group="default">
         <origin xyz="0.024 0 0" rpy="0 ${M_pi/2} 0"/>
         <geometry>
@@ -151,5 +151,5 @@
         </geometry>
       </collision>
-      <collision>
+      <collision group="other">
         <origin xyz="0.052 0 0" rpy="0 0 0"/>
         <geometry>
@@ -178,5 +178,5 @@
       </visual>
       <!-- begin collision mesh of f2    ->
-      <collision>
+      <collision group="default">
         <origin xyz="0 0 0" rpy="0 0 0"/>
         <geometry>
@@ -263,5 +263,5 @@
       </inertial>
       <!-- begin simple shape approximation of palm -->
-      <collision>
+      <collision group="default">
         <origin xyz="0.069 ${0.016 * reflect} 0.038" rpy="0 ${M_pi/2} ${-0.9 * reflect}"/>
         <geometry>
@@ -269,5 +269,5 @@
         </geometry>
       </collision>
-      <collision>
+      <collision group="other">
         <origin xyz="0.064 ${0.008 * reflect} 0.021" rpy="0.41 0 ${-0.9 * reflect}"/>
         <geometry>
@@ -275,5 +275,5 @@
         </geometry>
       </collision>
-      <collision>
+      <collision group="other">
         <origin xyz="0.02 0 -0.005" rpy="0 ${M_pi/2} 0"/>
         <geometry>
@@ -281,5 +281,5 @@
         </geometry>
       </collision>
-      <collision>
+      <collision group="other">
         <origin xyz="0.11 ${-0.01*reflect} -0.005" rpy="0 0 ${0.37*reflect}"/>
         <geometry>
@@ -287,5 +287,5 @@
         </geometry>
       </collision>
-      <collision>
+      <collision group="other">
         <origin xyz="0.09 ${0.02*reflect} -0.005" rpy="0 0 ${0.37*reflect}"/>
         <geometry>
@@ -293,5 +293,5 @@
         </geometry>
       </collision>
-      <collision>
+      <collision group="other">
         <origin xyz="0.060 ${0.050*reflect} -0.005" rpy="0 0 ${0.37*reflect}"/>
         <geometry>
@@ -299,5 +299,5 @@
         </geometry>
       </collision>
-      <collision>
+      <collision group="other">
         <origin xyz="0.044 ${-0.04*reflect} -0.005" rpy="0 0 ${0.79*reflect}"/>
         <geometry>
@@ -372,5 +372,5 @@
       <!--   end visual shape approximation of palm -->
       <!-- begin collision mesh of f2 ->
-      <collision>
+      <collision group="default">
         <origin xyz="0 0 0" rpy="0 0 0"/>
         <geometry>

Commit message: a simple eigengrasp based controller just for demonstration/strawman purposes.

File: ros/sandia_hand_description/urdf/sandia_hand_simple_shapes.urdf.xacro (robot description, xacro)
@@ -9,5 +9,5 @@
       <origin xyz="0 0 0" rpy="0 0 0"/>
       <inertial>
-        <mass value="0.1"/>
+        <mass value="0.35"/>
         <origin xyz="0 0 0"/>
         <inertia ixx="0.01" ixy="0" ixz="0" iyy="0.01" iyz="0" izz="0.01"/>
@@ -17,5 +17,5 @@
       <origin xyz="0 0 0" rpy="0 0 0"/>
       <inertial>
-        <mass value="0.1"/>
+        <mass value="0.001"/>
         <origin xyz="0 0 0"/>
         <inertia ixx="0.01" ixy="0" ixz="0" iyy="0.01" iyz="0" izz="0.01"/>
@@ -25,5 +25,5 @@
       <origin xyz="0 0 0" rpy="0 0 0"/>
       <inertial>
-        <mass value="0.1"/>
+        <mass value="0.05"/>
         <origin xyz="0 0 0"/>
         <inertia ixx="0.01" ixy="0" ixz="0" iyy="0.01" iyz="0" izz="0.01"/>
@@ -86,5 +86,5 @@
       <origin xyz="0 0 0" rpy="0 0 0"/>
       <inertial>
-        <mass value="0.1"/>
+        <mass value="0.05"/>
         <origin xyz="0 0 0"/>
         <inertia ixx="0.01" ixy="0" ixz="0" iyy="0.01" iyz="0" izz="0.01"/>
@@ -132,5 +132,5 @@
       <origin xyz="0 0 0" rpy="0 0 0"/>
       <inertial>
-        <mass value="0.1"/>
+        <mass value="0.001"/>
         <origin xyz="0 0 0"/>
         <inertia ixx="0.01" ixy="0" ixz="0" iyy="0.01" iyz="0" izz="0.01"/>
@@ -140,5 +140,5 @@
       <origin xyz="0 0 0" rpy="0 0 0"/>
       <inertial>
-        <mass value="0.1"/>
+        <mass value="0.05"/>
         <origin xyz="0 0 0"/>
         <inertia ixx="0.01" ixy="0" ixz="0" iyy="0.01" iyz="0" izz="0.01"/>
@@ -200,5 +200,5 @@
       <origin xyz="0 0 0" rpy="0 0 0"/>
       <inertial>
-        <mass value="0.1"/>
+        <mass value="0.001"/>
         <origin xyz="0 0 0"/>
         <inertia ixx="0.01" ixy="0" ixz="0" iyy="0.01" iyz="0" izz="0.01"/>
@@ -216,5 +216,5 @@
       <limit lower="-${M_pi/2}" upper="${M_pi/2}" effort="1" velocity="1"/>
       <safety_controller soft_lower_limit="${-1.57079-10.0}" soft_upper_limit="${1.57079+10.0}" k_position="1000.0" k_velocity="1000.0"/>
-      <dynamics damping="0.1"/>
+      <dynamics damping="0.2"/>
       <origin xyz="0 0 0" rpy="0 0 0"/>
     </joint>
@@ -225,5 +225,5 @@
       <limit lower="-${M_pi/2}" upper="${M_pi/2}" effort="1" velocity="1"/>
       <safety_controller soft_lower_limit="${-1.57079-10.0}" soft_upper_limit="${1.57079+10.0}" k_position="1000.0" k_velocity="1000.0"/>
-      <dynamics damping="0.1"/>
+      <dynamics damping="0.2"/>
       <origin xyz="0.028 0 0" rpy="${M_pi/2} 0 0"/>
     </joint>
@@ -234,5 +234,5 @@
       <origin xyz="0.05 0 0" rpy="0 0 0"/>
       <safety_controller soft_lower_limit="${-1.57079-10.0}" soft_upper_limit="${1.57079+10.0}" k_position="1000.0" k_velocity="1000.0"/>
-      <dynamics damping="0.1"/>
+      <dynamics damping="0.2"/>
       <limit lower="-${M_pi/2}" upper="${M_pi/2}" effort="1" velocity="1"/>
     </joint>
@@ -258,5 +258,5 @@
       <origin xyz="0 0 0" rpy="0 0 0"/>
       <inertial>
-        <mass value="0.1"/>
+        <mass value="0.3"/>
         <origin xyz="0 0 0"/>
         <inertia ixx="0.01" ixy="0" ixz="0" iyy="0.01" iyz="0" izz="0.01"/>
