Commit message: for issue #1, install sandia hand meshes as gazebo model resource

File: ros/sandia_hand_description/urdf/sandia_hand_simple_shapes.urdf.xacro (robot description, xacro)
@@ -43,9 +43,8 @@
       </collision>
       <!--   end simple shape approximation of f0 -->
-      <!-- begin visual shape approximation of f0 -->
-      <visual>
-        <origin xyz="0 0 0.003" rpy="0 0 0"/>
-        <geometry>
-          <cylinder radius="0.015" length="0.023" />
+      <visual>
+        <origin xyz="0 0 0" rpy="0 0 0"/>
+        <geometry>
+          <mesh filename="package://sandia_hand_description/meshes/f0.stl"/>
         </geometry>
         <material name="${side}_sandia_hand_skin_suntan">
@@ -53,33 +52,4 @@
         </material>
       </visual>
-      <visual>
-        <origin xyz="0.011 0 0.003" rpy="${M_pi/2} 0 0"/>
-        <geometry>
-          <cylinder radius="0.01" length="0.023" />
-        </geometry>
-        <material name="${side}_sandia_hand_skin_suntan">
-          <color rgba="0.7 0.4 0.2 1.0"/>
-        </material>
-      </visual>
-      <!--   end visual shape approximation of f0 -->
-      <!-- begin collision mesh of f0 ->
-      <collision group="default">
-        <origin xyz="0 0 0" rpy="0 0 0"/>
-        <geometry>
-          <mesh filename="package://sandia_hand_description/meshes/f0.stl"/>
-        </geometry>
-      </collision>
-      <!-   end collision mesh of f0 -->
-      <!-- begin visual mesh of f0 ->
-      <visual>
-        <origin xyz="0 0 0" rpy="0 0 0"/>
-        <geometry>
-          <mesh filename="package://sandia_hand_description/meshes/f0.stl"/>
-        </geometry>
-        <material name="${side}_sandia_hand_skin_suntan">
-          <color rgba="0.7 0.4 0.2 1.0"/>
-        </material>
-      </visual>
-      <!-   end visual mesh of f0 -->
     </link>
     <link name="${side}_f${idx}_1">
@@ -98,9 +68,16 @@
       </collision>
       <!--   end simple shape approximation of f1 -->
-      <!-- begin visual shape approximation of f1 -->
-      <visual>
-        <origin xyz="0.024 0 0" rpy="0 ${M_pi/2} 0"/>
-        <geometry>
-          <cylinder radius="0.01" length="0.067" />
+      <!-- begin collision mesh of f1 ->
+      <collision group="default">
+        <origin xyz="0 0 0" rpy="0 0 0"/>
+        <geometry>
+          <mesh filename="package://sandia_hand_description/meshes/f1.stl"/>
+        </geometry>
+      </collision>
+      <!-   end collision mesh of f1 -->
+      <visual>
+        <origin xyz="0 0 0" rpy="0 0 0"/>
+        <geometry>
+          <mesh filename="package://sandia_hand_description/meshes/f1.stl"/>
         </geometry>
         <material name="${side}_sandia_hand_skin">
@@ -108,24 +85,4 @@
         </material>
       </visual>
-      <!--   end visual shape approximation of f1 -->
-      <!-- begin collision mesh of f1 ->
-      <collision group="default">
-        <origin xyz="0 0 0" rpy="0 0 0"/>
-        <geometry>
-          <mesh filename="package://sandia_hand_description/meshes/f1.stl"/>
-        </geometry>
-      </collision>
-      <!-   end collision mesh of f1 -->
-      <!-- begin visual mesh of f1 ->
-      <visual>
-        <origin xyz="0 0 0" rpy="0 0 0"/>
-        <geometry>
-          <mesh filename="package://sandia_hand_description/meshes/f1.stl"/>
-        </geometry>
-        <material name="${side}_sandia_hand_skin">
-          <color rgba="0.835 0.655 0.345 1.0"/>
-        </material>
-      </visual>
-      <!-   end visual mesh of f1 -->
     </link>
     <link name="${side}_f${idx}_1_accel">
@@ -158,9 +115,16 @@
       </collision>
       <!--   end simple shape approximation of f2 -->
-      <!-- begin visual shape approximation of f2 -->
-      <visual>
-        <origin xyz="0.024 0 0" rpy="0 ${M_pi/2} 0"/>
-        <geometry>
-          <cylinder radius="0.009" length="0.057" />
+      <!-- begin collision mesh of f2    ->
+      <collision group="default">
+        <origin xyz="0 0 0" rpy="0 0 0"/>
+        <geometry>
+          <mesh filename="package://sandia_hand_description/meshes/f2.stl"/>
+        </geometry>
+      </collision>
+      <!-   end collision mesh of f2 -->
+      <visual>
+        <origin xyz="0 0 0" rpy="0 0 0"/>
+        <geometry>
+          <mesh filename="package://sandia_hand_description/meshes/f2.stl"/>
         </geometry>
         <material name="${side}_sandia_hand_skin_suntan">
@@ -168,32 +132,4 @@
         </material>
       </visual>
-      <visual>
-        <origin xyz="0.052 0 0" rpy="0 0 0"/>
-        <geometry>
-          <sphere radius="0.009" />
-        </geometry>
-        <material name="${side}_sandia_hand_skin_suntan">
-          <color rgba="0.8 0.6 0.3 1.0"/>
-        </material>
-      </visual>
-      <!-- begin collision mesh of f2    ->
-      <collision group="default">
-        <origin xyz="0 0 0" rpy="0 0 0"/>
-        <geometry>
-          <mesh filename="package://sandia_hand_description/meshes/f2.stl"/>
-        </geometry>
-      </collision>
-      <!-   end collision mesh of f2 -->
-      <!-- begin visual mesh of f2    ->
-      <visual>
-        <origin xyz="0 0 0" rpy="0 0 0"/>
-        <geometry>
-          <mesh filename="package://sandia_hand_description/meshes/f2.stl"/>
-        </geometry>
-        <material name="${side}_sandia_hand_skin_suntan">
-          <color rgba="0.8 0.6 0.3 1.0"/>
-        </material>
-      </visual>
-      <!-   end visual mesh of f2 -->
     </link>
     <link name="${side}_f${idx}_2_accel">
@@ -306,9 +242,17 @@
       </collision>
       <!--   end simple shape approximation of palm -->
-      <!-- begin visual shape approximation of palm -->
-      <visual>
-        <origin xyz="0.069 ${0.016*reflect} 0.038" rpy="0 ${M_pi/2} ${-0.9*reflect}"/>
-        <geometry>
-          <cylinder radius="0.013" length="0.100" />
+      <!--   end visual shape approximation of palm -->
+      <!-- begin collision mesh of f2 ->
+      <collision group="default">
+        <origin xyz="0 0 0" rpy="0 0 0"/>
+        <geometry>
+          <mesh filename="package://sandia_hand_description/meshes/palm.stl"/>
+        </geometry>
+      </collision>
+      <!-   end collision mesh of f2 -->
+      <visual>
+        <origin xyz="0 0 0" rpy="0 0 0"/>
+        <geometry>
+          <mesh filename="package://sandia_hand_description/meshes/palm.stl"/>
         </geometry>
         <material name="${side}_sandia_hand_skin">
@@ -316,78 +260,4 @@
         </material>
       </visual>
-      <visual>
-        <origin xyz="0.064 ${0.008*reflect} 0.021" rpy="0.41 0 ${-0.9*reflect}"/>
-        <geometry>
-          <box size="0.09 .035 .05" />
-        </geometry>
-        <material name="${side}_sandia_hand_skin">
-          <color rgba="0.835 0.655 0.345 1.0"/>
-        </material>
-      </visual>
-      <visual>
-        <origin xyz="0.02 0 -0.005" rpy="0 ${M_pi/2} 0"/>
-        <geometry>
-          <cylinder radius="0.038" length="0.05" />
-        </geometry>
-        <material name="${side}_sandia_hand_skin">
-          <color rgba="0.835 0.655 0.345 1.0"/>
-        </material>
-      </visual>
-      <visual>
-        <origin xyz="0.11 ${-0.01*reflect} -0.005" rpy="0 0 ${0.37*reflect}"/>
-        <geometry>
-          <box size="0.09 .03 .06" />
-        </geometry>
-        <material name="${side}_sandia_hand_skin">
-          <color rgba="0.835 0.655 0.345 1.0"/>
-        </material>
-      </visual>
-      <visual>
-        <origin xyz="0.09 ${0.02*reflect} -0.005" rpy="0 0 ${0.37*reflect}"/>
-        <geometry>
-          <box size="0.09 .03 .06" />
-        </geometry>
-        <material name="${side}_sandia_hand_skin">
-          <color rgba="0.835 0.655 0.345 1.0"/>
-        </material>
-      </visual>
-      <visual>
-        <origin xyz="0.060 ${0.050*reflect} -0.005" rpy="0 0 ${0.37*reflect}"/>
-        <geometry>
-          <box size="0.09 .03 .06" />
-        </geometry>
-        <material name="${side}_sandia_hand_skin">
-          <color rgba="0.835 0.655 0.345 1.0"/>
-        </material>
-      </visual>
-      <visual>
-        <origin xyz="0.044 ${-0.04*reflect} -0.005" rpy="0 0 ${0.79*reflect}"/>
-        <geometry>
-          <box size="0.09 .03 .06" />
-        </geometry>
-        <material name="${side}_sandia_hand_skin">
-          <color rgba="0.835 0.655 0.345 1.0"/>
-        </material>
-      </visual>
-      <!--   end visual shape approximation of palm -->
-      <!-- begin collision mesh of f2 ->
-      <collision group="default">
-        <origin xyz="0 0 0" rpy="0 0 0"/>
-        <geometry>
-          <mesh filename="package://sandia_hand_description/meshes/palm.stl"/>
-        </geometry>
-      </collision>
-      <!-   end collision mesh of f2 -->
-      <!-- begin visual mesh of f2    ->
-      <visual>
-        <origin xyz="0 0 0" rpy="0 0 0"/>
-        <geometry>
-          <mesh filename="package://sandia_hand_description/meshes/palm.stl"/>
-        </geometry>
-        <material name="${side}_sandia_hand_skin">
-          <color rgba="0.835 0.655 0.345 1.0"/>
-        </material>
-      </visual>
-      <!-   end visual mesh of f2 -->
     </link>
     <joint name="${side}_sandia_hand_joint" type="fixed">

Commit message: looking at inertia updates.

File: ros/sandia_hand_description/urdf/sandia_hand_simple_shapes.urdf.xacro (robot description, xacro)
@@ -9,5 +9,5 @@
       <origin xyz="0 0 0" rpy="0 0 0"/>
       <inertial>
-        <mass value="0.35"/>
+        <mass value="0.250"/> <!-- (2.303 - 1.303) / 4 -->
         <origin xyz="0 0 0"/>
         <inertia ixx="0.01" ixy="0" ixz="0" iyy="0.01" iyz="0" izz="0.01"/>
@@ -25,5 +25,5 @@
       <origin xyz="0 0 0" rpy="0 0 0"/>
       <inertial>
-        <mass value="0.05"/>
+        <mass value="0.106"/> <!-- F1 -->
         <origin xyz="0 0 0"/>
         <inertia ixx="0.01" ixy="0" ixz="0" iyy="0.01" iyz="0" izz="0.01"/>
@@ -86,5 +86,5 @@
       <origin xyz="0 0 0" rpy="0 0 0"/>
       <inertial>
-        <mass value="0.05"/>
+        <mass value="0.033"/> <!-- F2 -->
         <origin xyz="0 0 0"/>
         <inertia ixx="0.01" ixy="0" ixz="0" iyy="0.01" iyz="0" izz="0.01"/>
@@ -140,5 +140,5 @@
       <origin xyz="0 0 0" rpy="0 0 0"/>
       <inertial>
-        <mass value="0.05"/>
+        <mass value="0.033"/>  <!-- F3 -->
         <origin xyz="0 0 0"/>
         <inertia ixx="0.01" ixy="0" ixz="0" iyy="0.01" iyz="0" izz="0.01"/>
@@ -258,7 +258,8 @@
       <origin xyz="0 0 0" rpy="0 0 0"/>
       <inertial>
-        <mass value="0.3"/>
-        <origin xyz="0 0 0"/>
-        <inertia ixx="0.01" ixy="0" ixz="0" iyy="0.01" iyz="0" izz="0.01"/>
+        <mass value="1.303"/>
+        <origin xyz="0 0 0"/>
+        <!-- solid sphere with 5cm radius -->
+        <inertia ixx="0.002303" ixy="0" ixz="0" iyy="0.002303" iyz="0" izz="0.002303"/>
       </inertial>
       <!-- begin simple shape approximation of palm -->

Commit message: first cut at realistic inertia

File: ros/sandia_hand_description/urdf/sandia_hand_simple_shapes.urdf.xacro (robot description, xacro)
@@ -9,7 +9,9 @@
       <origin xyz="0 0 0" rpy="0 0 0"/>
       <inertial>
+        <!-- total mass is 2.303 kg, palm is about 1.303 kg, distribute the rest into _base -->
         <mass value="0.250"/> <!-- (2.303 - 1.303) / 4 -->
         <origin xyz="0 0 0"/>
-        <inertia ixx="0.01" ixy="0" ixz="0" iyy="0.01" iyz="0" izz="0.01"/>
+        <!-- model as sphere with radius of 1cm -->
+        <inertia ixx="0.00001" ixy="0" ixz="0" iyy="0.00001" iyz="0" izz="0.00001"/>
       </inertial>
     </link>
@@ -17,7 +19,7 @@
       <origin xyz="0 0 0" rpy="0 0 0"/>
       <inertial>
-        <mass value="0.001"/>
-        <origin xyz="0 0 0"/>
-        <inertia ixx="0.01" ixy="0" ixz="0" iyy="0.01" iyz="0" izz="0.01"/>
+        <mass value="0.01"/>
+        <origin xyz="0 0 0"/>
+        <inertia ixx="0.000001" ixy="0" ixz="0" iyy="0.000001" iyz="0" izz="0.000001"/>
       </inertial>
     </link>
@@ -27,5 +29,6 @@
         <mass value="0.106"/> <!-- F1 -->
         <origin xyz="0 0 0"/>
-        <inertia ixx="0.01" ixy="0" ixz="0" iyy="0.01" iyz="0" izz="0.01"/>
+        <!-- solid cylinder -->
+        <inertia izz="0.000011925" ixy="0" ixz="0" iyy="0.00011505" iyz="0" ixx="0.00011505"/>
       </inertial>
       <!-- begin simple shape approximation of f0 -->
@@ -88,5 +91,6 @@
         <mass value="0.033"/> <!-- F2 -->
         <origin xyz="0 0 0"/>
-        <inertia ixx="0.01" ixy="0" ixz="0" iyy="0.01" iyz="0" izz="0.01"/>
+        <!-- solid cylinder -->
+        <inertia ixx="0.00000165" ixy="0" ixz="0" iyy="0.00001316975" iyz="0" izz="0.00001316975"/>
       </inertial>
       <!-- begin simple shape approximation of f1 -->
@@ -132,7 +136,7 @@
       <origin xyz="0 0 0" rpy="0 0 0"/>
       <inertial>
-        <mass value="0.001"/>
-        <origin xyz="0 0 0"/>
-        <inertia ixx="0.01" ixy="0" ixz="0" iyy="0.01" iyz="0" izz="0.01"/>
+        <mass value="0.01"/>
+        <origin xyz="0 0 0"/>
+        <inertia ixx="0.000001" ixy="0" ixz="0" iyy="0.000001" iyz="0" izz="0.000001"/>
       </inertial>
     </link>
@@ -142,5 +146,6 @@
         <mass value="0.033"/>  <!-- F3 -->
         <origin xyz="0 0 0"/>
-        <inertia ixx="0.01" ixy="0" ixz="0" iyy="0.01" iyz="0" izz="0.01"/>
+        <!-- solid cylinder -->
+        <inertia ixx="0.0000013365" ixy="0" ixz="0" iyy="0.000009603" iyz="0" izz="0.000009603"/>
       </inertial>
       <!-- begin simple shape approximation of f2 -->
@@ -200,7 +205,7 @@
       <origin xyz="0 0 0" rpy="0 0 0"/>
       <inertial>
-        <mass value="0.001"/>
-        <origin xyz="0 0 0"/>
-        <inertia ixx="0.01" ixy="0" ixz="0" iyy="0.01" iyz="0" izz="0.01"/>
+        <mass value="0.01"/>
+        <origin xyz="0 0 0"/>
+        <inertia ixx="0.000001" ixy="0" ixz="0" iyy="0.000001" iyz="0" izz="0.000001"/>
       </inertial>
     </link>
@@ -261,5 +266,5 @@
         <origin xyz="0 0 0"/>
         <!-- solid sphere with 5cm radius -->
-        <inertia ixx="0.002303" ixy="0" ixz="0" iyy="0.002303" iyz="0" izz="0.002303"/>
+        <inertia ixx="0.001303" ixy="0" ixz="0" iyy="0.001303" iyz="0" izz="0.001303"/>
       </inertial>
       <!-- begin simple shape approximation of palm -->

Commit message: tune damping and gains

File: ros/sandia_hand_description/urdf/sandia_hand_simple_shapes.urdf.xacro (robot description, xacro)
@@ -219,7 +219,7 @@
       <parent link="${side}_f${idx}_base"/>
       <child link="${side}_f${idx}_0"/>
-      <limit lower="-${M_pi/2}" upper="${M_pi/2}" effort="1" velocity="1"/>
+      <limit lower="-${M_pi/2}" upper="${M_pi/2}" effort="11" velocity="1"/>
       <safety_controller soft_lower_limit="${-1.57079-10.0}" soft_upper_limit="${1.57079+10.0}" k_position="1000.0" k_velocity="1000.0"/>
-      <dynamics damping="0.2"/>
+      <dynamics damping="30.0"/>
       <origin xyz="0 0 0" rpy="0 0 0"/>
     </joint>
@@ -228,7 +228,7 @@
       <parent link="${side}_f${idx}_0"/>
       <child link="${side}_f${idx}_1"/>
-      <limit lower="-${M_pi/2}" upper="${M_pi/2}" effort="1" velocity="1"/>
+      <limit lower="-${M_pi/2}" upper="${M_pi/2}" effort="28" velocity="1"/>
       <safety_controller soft_lower_limit="${-1.57079-10.0}" soft_upper_limit="${1.57079+10.0}" k_position="1000.0" k_velocity="1000.0"/>
-      <dynamics damping="0.2"/>
+      <dynamics damping="30.0"/>
       <origin xyz="0.028 0 0" rpy="${M_pi/2} 0 0"/>
     </joint>
@@ -239,6 +239,6 @@
       <origin xyz="0.05 0 0" rpy="0 0 0"/>
       <safety_controller soft_lower_limit="${-1.57079-10.0}" soft_upper_limit="${1.57079+10.0}" k_position="1000.0" k_velocity="1000.0"/>
-      <dynamics damping="0.2"/>
-      <limit lower="-${M_pi/2}" upper="${M_pi/2}" effort="1" velocity="1"/>
+      <dynamics damping="30.0"/>
+      <limit lower="-${M_pi/2}" upper="${M_pi/2}" effort="28" velocity="1"/>
     </joint>
     <joint name="${side}_f${idx}_fixed_accel" type="fixed">

Commit message: testing damping reduction

File: ros/sandia_hand_description/urdf/sandia_hand_simple_shapes.urdf.xacro (robot description, xacro)
@@ -5,4 +5,6 @@
   <include filename="$(find sandia_hand_description)/urdf/sandia_hand.transmission.xacro" />
   <xacro:property name="M_pi" value="3.1415926535897931" />
+  <xacro:property name="damping_coefficient" value="20" />
+  <xacro:property name="velocity_limit" value="1" />
   <xacro:macro name="finger" params="idx x y z r p yaw side reflect">
     <link name="${side}_f${idx}_base">
@@ -219,7 +221,7 @@
       <parent link="${side}_f${idx}_base"/>
       <child link="${side}_f${idx}_0"/>
-      <limit lower="-${M_pi/2}" upper="${M_pi/2}" effort="11" velocity="1"/>
+      <limit lower="-${M_pi/2}" upper="${M_pi/2}" effort="11" velocity="${velocity_limit}"/>
       <safety_controller soft_lower_limit="${-1.57079-10.0}" soft_upper_limit="${1.57079+10.0}" k_position="1000.0" k_velocity="1000.0"/>
-      <dynamics damping="30.0"/>
+      <dynamics damping="${damping_coefficient}"/>
       <origin xyz="0 0 0" rpy="0 0 0"/>
     </joint>
@@ -228,7 +230,7 @@
       <parent link="${side}_f${idx}_0"/>
       <child link="${side}_f${idx}_1"/>
-      <limit lower="-${M_pi/2}" upper="${M_pi/2}" effort="28" velocity="1"/>
+      <limit lower="-${M_pi/2}" upper="${M_pi/2}" effort="28" velocity="${velocity_limit}"/>
       <safety_controller soft_lower_limit="${-1.57079-10.0}" soft_upper_limit="${1.57079+10.0}" k_position="1000.0" k_velocity="1000.0"/>
-      <dynamics damping="30.0"/>
+      <dynamics damping="${damping_coefficient}"/>
       <origin xyz="0.028 0 0" rpy="${M_pi/2} 0 0"/>
     </joint>
@@ -239,6 +241,6 @@
       <origin xyz="0.05 0 0" rpy="0 0 0"/>
       <safety_controller soft_lower_limit="${-1.57079-10.0}" soft_upper_limit="${1.57079+10.0}" k_position="1000.0" k_velocity="1000.0"/>
-      <dynamics damping="30.0"/>
-      <limit lower="-${M_pi/2}" upper="${M_pi/2}" effort="28" velocity="1"/>
+      <dynamics damping="${damping_coefficient}"/>
+      <limit lower="-${M_pi/2}" upper="${M_pi/2}" effort="28" velocity="${velocity_limit}"/>
     </joint>
     <joint name="${side}_f${idx}_fixed_accel" type="fixed">

Commit message: fix moi for F1 (izz and ixx were backwards).  increase velocity limit from 1 to 100.

File: ros/sandia_hand_description/urdf/sandia_hand_simple_shapes.urdf.xacro (robot description, xacro)
@@ -5,6 +5,8 @@
   <include filename="$(find sandia_hand_description)/urdf/sandia_hand.transmission.xacro" />
   <xacro:property name="M_pi" value="3.1415926535897931" />
-  <xacro:property name="damping_coefficient" value="20" />
-  <xacro:property name="velocity_limit" value="1" />
+  <xacro:property name="damping_coefficient_j0" value="30" />
+  <xacro:property name="damping_coefficient_j1" value="30" />
+  <xacro:property name="damping_coefficient_j2" value="30" />
+  <xacro:property name="velocity_limit" value="100" />
   <xacro:macro name="finger" params="idx x y z r p yaw side reflect">
     <link name="${side}_f${idx}_base">
@@ -32,5 +34,5 @@
         <origin xyz="0 0 0"/>
         <!-- solid cylinder -->
-        <inertia izz="0.000011925" ixy="0" ixz="0" iyy="0.00011505" iyz="0" ixx="0.00011505"/>
+        <inertia ixx="0.000011925" ixy="0" ixz="0" iyy="0.00011505" iyz="0" izz="0.00011505"/>
       </inertial>
       <!-- begin simple shape approximation of f0 -->
@@ -223,5 +225,5 @@
       <limit lower="-${M_pi/2}" upper="${M_pi/2}" effort="11" velocity="${velocity_limit}"/>
       <safety_controller soft_lower_limit="${-1.57079-10.0}" soft_upper_limit="${1.57079+10.0}" k_position="1000.0" k_velocity="1000.0"/>
-      <dynamics damping="${damping_coefficient}"/>
+      <dynamics damping="${damping_coefficient_j0}"/>
       <origin xyz="0 0 0" rpy="0 0 0"/>
     </joint>
@@ -232,5 +234,5 @@
       <limit lower="-${M_pi/2}" upper="${M_pi/2}" effort="28" velocity="${velocity_limit}"/>
       <safety_controller soft_lower_limit="${-1.57079-10.0}" soft_upper_limit="${1.57079+10.0}" k_position="1000.0" k_velocity="1000.0"/>
-      <dynamics damping="${damping_coefficient}"/>
+      <dynamics damping="${damping_coefficient_j1}"/>
       <origin xyz="0.028 0 0" rpy="${M_pi/2} 0 0"/>
     </joint>
@@ -241,5 +243,5 @@
       <origin xyz="0.05 0 0" rpy="0 0 0"/>
       <safety_controller soft_lower_limit="${-1.57079-10.0}" soft_upper_limit="${1.57079+10.0}" k_position="1000.0" k_velocity="1000.0"/>
-      <dynamics damping="${damping_coefficient}"/>
+      <dynamics damping="${damping_coefficient_j2}"/>
       <limit lower="-${M_pi/2}" upper="${M_pi/2}" effort="28" velocity="${velocity_limit}"/>
     </joint>
