Commit message: fix merge from revert_stump

File: ros/sandia_hand_description/urdf/sandia_hand_simple_shapes.urdf.xacro (robot description, xacro)
@@ -9,5 +9,5 @@
   <xacro:property name="damping_coefficient_j2" value="30" />
   <xacro:property name="velocity_limit" value="100" />
-  <xacro:macro name="finger" params="idx x y z r p yaw side reflect joint_type">
+  <xacro:macro name="finger" params="idx x y z r p yaw side reflect">
     <link name="${side}_f${idx}_base">
       <origin xyz="0 0 0" rpy="0 0 0"/>
@@ -219,5 +219,5 @@
       <origin xyz="${x} ${y} ${z}" rpy="${r} ${p} ${yaw}"/>
     </joint>
-    <joint name="${side}_f${idx}_j0" type="${joint_type}">
+    <joint name="${side}_f${idx}_j0" type="revolute">
       <axis xyz="0 0 ${reflect}"/>
       <parent link="${side}_f${idx}_base"/>
@@ -228,5 +228,5 @@
       <origin xyz="0 0 0" rpy="0 0 0"/>
     </joint>
-    <joint name="${side}_f${idx}_j1" type="${joint_type}">
+    <joint name="${side}_f${idx}_j1" type="revolute">
       <axis xyz="0 0 1"/>
       <parent link="${side}_f${idx}_0"/>
@@ -237,5 +237,5 @@
       <origin xyz="0.028 0 0" rpy="${M_pi/2} 0 0"/>
     </joint>
-    <joint name="${side}_f${idx}_j2" type="${joint_type}">
+    <joint name="${side}_f${idx}_j2" type="revolute">
       <axis xyz="0 0 1"/>
       <parent link="${side}_f${idx}_1"/>
@@ -265,5 +265,5 @@
   </xacro:macro>
   <!--
-  <xacro:macro name="sandia_hand" params="side parent reflect joint_type thumb_angle *origin">
+  <xacro:macro name="sandia_hand" params="side parent reflect thumb_angle *origin">
   -->
   <xacro:macro name="sandia_hand" params="side parent reflect *origin">
@@ -411,13 +411,13 @@
     </joint>
     <!--
-    <xacro:finger side="${side}" idx="0" x="0.140" y="0.00000" z="0" r="0" p="0" yaw="${0.3*reflect}" reflect="${reflect}" joint_type="${joint_type}" />
-    <xacro:finger side="${side}" idx="1" x="0.115" y="${0.03122*reflect}" z="0" r="0" p="0" yaw="${0.3*reflect}" reflect="${reflect}" joint_type="${joint_type}" />
-    <xacro:finger side="${side}" idx="2" x="0.090" y="${0.06245*reflect}" z="0" r="0" p="0" yaw="${0.3*reflect}" reflect="${reflect}" joint_type="${joint_type}" />
-    <xacro:finger side="${side}" idx="3" x="0.03995" y="${-0.04383*reflect}" z="0.014" r="0" p="-${M_pi/2 + thumb_angle}" yaw="${-(2.3562+thumb_angle)*reflect}" reflect="${reflect}" joint_type="${joint_type}" />
+    <xacro:finger side="${side}" idx="0" x="0.140" y="0.00000" z="0" r="0" p="0" yaw="${0.3*reflect}" reflect="${reflect}" />
+    <xacro:finger side="${side}" idx="1" x="0.115" y="${0.03122*reflect}" z="0" r="0" p="0" yaw="${0.3*reflect}" reflect="${reflect}" />
+    <xacro:finger side="${side}" idx="2" x="0.090" y="${0.06245*reflect}" z="0" r="0" p="0" yaw="${0.3*reflect}" reflect="${reflect}" />
+    <xacro:finger side="${side}" idx="3" x="0.03995" y="${-0.04383*reflect}" z="0.014" r="0" p="-${M_pi/2 + thumb_angle}" yaw="${-(2.3562+thumb_angle)*reflect}" reflect="${reflect}" />
     -->
-    <xacro:finger side="${side}" idx="0" x="0.140" y="0.00000" z="0" r="0" p="0" yaw="${0.3*reflect}" reflect="${reflect}" joint_type="revolute" />
-    <xacro:finger side="${side}" idx="1" x="0.115" y="${0.03122*reflect}" z="0" r="0" p="0" yaw="${0.3*reflect}" reflect="${reflect}" joint_type="revolute" />
-    <xacro:finger side="${side}" idx="2" x="0.090" y="${0.06245*reflect}" z="0" r="0" p="0" yaw="${0.3*reflect}" reflect="${reflect}" joint_type="revolute" />
-    <xacro:finger side="${side}" idx="3" x="0.03995" y="${-0.04383*reflect}" z="0.014" r="0" p="-${M_pi/2}" yaw="${-(2.3562)*reflect}" reflect="${reflect}" joint_type="joint_type" />
+    <xacro:finger side="${side}" idx="0" x="0.140" y="0.00000" z="0" r="0" p="0" yaw="${0.3*reflect}" reflect="${reflect}" />
+    <xacro:finger side="${side}" idx="1" x="0.115" y="${0.03122*reflect}" z="0" r="0" p="0" yaw="${0.3*reflect}" reflect="${reflect}" />
+    <xacro:finger side="${side}" idx="2" x="0.090" y="${0.06245*reflect}" z="0" r="0" p="0" yaw="${0.3*reflect}" reflect="${reflect}" />
+    <xacro:finger side="${side}" idx="3" x="0.03995" y="${-0.04383*reflect}" z="0.014" r="0" p="-${M_pi/2}" yaw="${-(2.3562)*reflect}" reflect="${reflect}" />
     <!-- not needed unless simulating the hand by itself
     <xacro:sandia_hand_gazebo_controller side="${side}" />

Commit message: adaptive damping set at -5 nms/rad for finger joints in simulation.

File: ros/sandia_hand_description/urdf/sandia_hand_simple_shapes.urdf.xacro (robot description, xacro)
@@ -5,7 +5,7 @@
   <include filename="$(find sandia_hand_description)/urdf/sandia_hand.transmission.xacro" />
   <xacro:property name="M_pi" value="3.1415926535897931" />
-  <xacro:property name="damping_coefficient_j0" value="30" />
-  <xacro:property name="damping_coefficient_j1" value="30" />
-  <xacro:property name="damping_coefficient_j2" value="30" />
+  <xacro:property name="damping_coefficient_j0" value="-5" />
+  <xacro:property name="damping_coefficient_j1" value="-5" />
+  <xacro:property name="damping_coefficient_j2" value="-5" />
   <xacro:property name="velocity_limit" value="-1" />
   <xacro:macro name="finger" params="idx x y z r p yaw side reflect">

Commit message: reduce default damping to 0.1 Nms/rad, adaptive

File: ros/sandia_hand_description/urdf/sandia_hand_simple_shapes.urdf.xacro (robot description, xacro)
@@ -5,7 +5,7 @@
   <include filename="$(find sandia_hand_description)/urdf/sandia_hand.transmission.xacro" />
   <xacro:property name="M_pi" value="3.1415926535897931" />
-  <xacro:property name="damping_coefficient_j0" value="-5" />
-  <xacro:property name="damping_coefficient_j1" value="-5" />
-  <xacro:property name="damping_coefficient_j2" value="-5" />
+  <xacro:property name="damping_coefficient_j0" value="-0.1" />
+  <xacro:property name="damping_coefficient_j1" value="-0.1" />
+  <xacro:property name="damping_coefficient_j2" value="-0.1" />
   <xacro:property name="velocity_limit" value="-1" />
   <xacro:macro name="finger" params="idx x y z r p yaw side reflect">

Commit message: increase damping to 2.5 for stability

File: ros/sandia_hand_description/urdf/sandia_hand_simple_shapes.urdf.xacro (robot description, xacro)
@@ -5,7 +5,7 @@
   <include filename="$(find sandia_hand_description)/urdf/sandia_hand.transmission.xacro" />
   <xacro:property name="M_pi" value="3.1415926535897931" />
-  <xacro:property name="damping_coefficient_j0" value="-0.1" />
-  <xacro:property name="damping_coefficient_j1" value="-0.1" />
-  <xacro:property name="damping_coefficient_j2" value="-0.1" />
+  <xacro:property name="damping_coefficient_j0" value="-2.5" />
+  <xacro:property name="damping_coefficient_j1" value="-2.5" />
+  <xacro:property name="damping_coefficient_j2" value="-2.5" />
   <xacro:property name="velocity_limit" value="-1" />
   <xacro:macro name="finger" params="idx x y z r p yaw side reflect">

Commit message: reducing damping to 1.0 Nms/rad.

File: ros/sandia_hand_description/urdf/sandia_hand_simple_shapes.urdf.xacro (robot description, xacro)
@@ -5,7 +5,7 @@
   <include filename="$(find sandia_hand_description)/urdf/sandia_hand.transmission.xacro" />
   <xacro:property name="M_pi" value="3.1415926535897931" />
-  <xacro:property name="damping_coefficient_j0" value="2.0" />
-  <xacro:property name="damping_coefficient_j1" value="2.0" />
-  <xacro:property name="damping_coefficient_j2" value="2.0" />
+  <xacro:property name="damping_coefficient_j0" value="1.0" />
+  <xacro:property name="damping_coefficient_j1" value="1.0" />
+  <xacro:property name="damping_coefficient_j2" value="1.0" />
   <xacro:property name="velocity_limit" value="-1" />
   <xacro:macro name="finger" params="idx x y z r p yaw side reflect">

Commit message: Expand visuals to match soft collision shapes

File: ros/sandia_hand_description/urdf/sandia_hand_simple_shapes.urdf.xacro (robot description, xacro)
@@ -171,5 +171,5 @@
         <origin xyz="0.024 0 0" rpy="0 ${M_pi/2} 0"/>
         <geometry>
-          <cylinder radius="0.009" length="0.057" />
+          <cylinder radius="0.014" length="0.057" />
         </geometry>
         <material name="${side}_sandia_hand_skin_suntan">
@@ -180,5 +180,5 @@
         <origin xyz="0.052 0 0" rpy="0 0 0"/>
         <geometry>
-          <sphere radius="0.009" />
+          <sphere radius="0.014" />
         </geometry>
         <material name="${side}_sandia_hand_skin_suntan">
@@ -227,18 +227,4 @@
         </geometry>
       </collision>
-      <!--
-      <visual>
-        <origin xyz="0.024 0 0" rpy="0 ${M_pi/2} 0"/>
-        <geometry>
-          <cylinder radius="0.014" length="0.057" />
-        </geometry>
-      </visual>
-      <visual>
-        <origin xyz="0.052 0 0" rpy="0 0 0"/>
-        <geometry>
-          <sphere radius="0.014" />
-        </geometry>
-      </visual>
-      -->
     </link>
     <joint name="${side}_f${idx}_base" type="fixed">
@@ -354,5 +340,5 @@
         <origin xyz="0.069 ${0.016*reflect} 0.038" rpy="0 ${M_pi/2} ${-0.9*reflect}"/>
         <geometry>
-          <cylinder radius="0.013" length="0.100" />
+          <cylinder radius="0.018" length="0.100" />
         </geometry>
         <material name="${side}_sandia_hand_skin">
@@ -381,5 +367,5 @@
         <origin xyz="0.11 ${-0.01*reflect} -0.005" rpy="0 0 ${0.37*reflect}"/>
         <geometry>
-          <box size="0.09 .03 .06" />
+          <box size="0.09 .03 .07" />
         </geometry>
         <material name="${side}_sandia_hand_skin">
@@ -390,5 +376,5 @@
         <origin xyz="0.09 ${0.02*reflect} -0.005" rpy="0 0 ${0.37*reflect}"/>
         <geometry>
-          <box size="0.09 .03 .06" />
+          <box size="0.09 .03 .07" />
         </geometry>
         <material name="${side}_sandia_hand_skin">
@@ -399,5 +385,5 @@
         <origin xyz="0.060 ${0.050*reflect} -0.005" rpy="0 0 ${0.37*reflect}"/>
         <geometry>
-          <box size="0.09 .03 .06" />
+          <box size="0.09 .03 .07" />
         </geometry>
         <material name="${side}_sandia_hand_skin">

Commit message: Fix reflection bug in one of sandia-hand collision/visual shapes

File: ros/sandia_hand_description/urdf/sandia_hand_simple_shapes.urdf.xacro (robot description, xacro)
@@ -281,5 +281,5 @@
       </collision>
       <collision group="other">
-        <origin xyz="0.064 ${0.008 * reflect} 0.021" rpy="0.41 0 ${-0.9 * reflect}"/>
+        <origin xyz="0.064 ${0.008 * reflect} 0.021" rpy="${0.41 * reflect} 0 ${-0.9 * reflect}"/>
         <geometry>
           <box size="0.09 .035 .05" />
@@ -328,5 +328,5 @@
       </visual>
       <visual>
-        <origin xyz="0.064 ${0.008*reflect} 0.021" rpy="0.41 0 ${-0.9*reflect}"/>
+        <origin xyz="0.064 ${0.008*reflect} 0.021" rpy="${0.41 * reflect} 0 ${-0.9*reflect}"/>
         <geometry>
           <box size="0.09 .035 .05" />

Commit message: Removed collision groups

File: ros/sandia_hand_description/urdf/sandia_hand_simple_shapes.urdf.xacro (robot description, xacro)
@@ -37,5 +37,5 @@
       </inertial>
       <!-- begin simple shape approximation of f0 -->
-      <collision group="default">
+      <collision>
         <origin xyz="0 0 0.003" rpy="0 0 0"/>
         <geometry>
@@ -43,5 +43,5 @@
         </geometry>
       </collision>
-      <collision group="other">
+      <collision>
         <origin xyz="0.011 0 0.003" rpy="${M_pi/2} 0 0"/>
         <geometry>
@@ -71,5 +71,5 @@
       <!--   end visual shape approximation of f0 -->
       <!-- begin collision mesh of f0 ->
-      <collision group="default">
+      <collision>
         <origin xyz="0 0 0" rpy="0 0 0"/>
         <geometry>
@@ -99,5 +99,5 @@
       </inertial>
       <!-- begin simple shape approximation of f1 -->
-      <collision group="default">
+      <collision>
         <origin xyz="0.024 0 0" rpy="0 ${M_pi/2} 0"/>
         <geometry>
@@ -118,5 +118,5 @@
       <!--   end visual shape approximation of f1 -->
       <!-- begin collision mesh of f1 ->
-      <collision group="default">
+      <collision>
         <origin xyz="0 0 0" rpy="0 0 0"/>
         <geometry>
@@ -154,5 +154,5 @@
       </inertial>
       <!-- begin simple shape approximation of f2 -->
-      <collision group="default">
+      <collision>
         <origin xyz="0.024 0 0" rpy="0 ${M_pi/2} 0"/>
         <geometry>
@@ -160,5 +160,5 @@
         </geometry>
       </collision>
-      <collision group="other">
+      <collision>
         <origin xyz="0.052 0 0" rpy="0 0 0"/>
         <geometry>
@@ -187,5 +187,5 @@
       </visual>
       <!-- begin collision mesh of f2    ->
-      <collision group="default">
+      <collision>
         <origin xyz="0 0 0" rpy="0 0 0"/>
         <geometry>
@@ -274,5 +274,5 @@
       </inertial>
       <!-- begin simple shape approximation of palm -->
-      <collision group="default">
+      <collision>
         <origin xyz="0.069 ${0.016 * reflect} 0.038" rpy="0 ${M_pi/2} ${-0.9 * reflect}"/>
         <geometry>
@@ -280,5 +280,5 @@
         </geometry>
       </collision>
-      <collision group="other">
+      <collision>
         <origin xyz="0.064 ${0.008 * reflect} 0.021" rpy="${0.41 * reflect} 0 ${-0.9 * reflect}"/>
         <geometry>
@@ -286,5 +286,5 @@
         </geometry>
       </collision>
-      <collision group="other">
+      <collision>
         <origin xyz="0.02 0 -0.005" rpy="0 ${M_pi/2} 0"/>
         <geometry>
@@ -292,5 +292,5 @@
         </geometry>
       </collision>
-      <collision group="other">
+      <collision>
         <origin xyz="0.11 ${-0.01*reflect} -0.005" rpy="0 0 ${0.37*reflect}"/>
         <geometry>
@@ -298,5 +298,5 @@
         </geometry>
       </collision>
-      <collision group="other">
+      <collision>
         <origin xyz="0.09 ${0.02*reflect} -0.005" rpy="0 0 ${0.37*reflect}"/>
         <geometry>
@@ -304,5 +304,5 @@
         </geometry>
       </collision>
-      <collision group="other">
+      <collision>
         <origin xyz="0.060 ${0.050*reflect} -0.005" rpy="0 0 ${0.37*reflect}"/>
         <geometry>
@@ -310,5 +310,5 @@
         </geometry>
       </collision>
-      <collision group="other">
+      <collision>
         <origin xyz="0.044 ${-0.04*reflect} -0.005" rpy="0 0 ${0.79*reflect}"/>
         <geometry>
@@ -383,5 +383,5 @@
       <!--   end visual shape approximation of palm -->
       <!-- begin collision mesh of f2 ->
-      <collision group="default">
+      <collision>
         <origin xyz="0 0 0" rpy="0 0 0"/>
         <geometry>
