Commit message: increase finger inertia until we can teleop to grab the drill.

File: ros/sandia_hand_description/urdf/sandia_hand.gazebo.xacro (robot description, xacro)
@@ -2,4 +2,22 @@
 <robot name="sandia_hand"
        xmlns:xacro="http://www.ros.org/wiki/xacro">
+  <xacro:macro name="finger_gazebo" params="side idx">
+    <gazebo reference ="${side}_f${idx}_base">
+      <mu1>0.9</mu1>
+      <mu2>0.9</mu2>
+    </gazebo>
+    <gazebo reference="${side}_f${idx}_0">
+      <mu1>0.9</mu1>
+      <mu2>0.9</mu2>
+    </gazebo>
+    <gazebo reference="${side}_f${idx}_1">
+      <mu1>0.9</mu1>
+      <mu2>0.9</mu2>
+    </gazebo>
+    <gazebo reference="${side}_f${idx}_2">
+      <mu1>0.9</mu1>
+      <mu2>0.9</mu2>
+    </gazebo>
+  </xacro:macro>
   <xacro:macro name="sandia_hand_gazebo" params="side">
     <gazebo>
@@ -9,4 +27,8 @@
       </plugin>
     </gazebo>
+    <gazebo reference="${side}_palm">
+      <mu1>0.9</mu1>
+      <mu2>0.9</mu2>
+    </gazebo>
   </xacro:macro>
 </robot>

File: ros/sandia_hand_description/urdf/sandia_hand_simple_shapes.urdf.xacro (robot description, xacro)
@@ -13,5 +13,5 @@
         <origin xyz="0 0 0"/>
         <!-- model as sphere with radius of 1cm -->
-        <inertia ixx="0.00001" ixy="0" ixz="0" iyy="0.00001" iyz="0" izz="0.00001"/>
+        <inertia ixx="0.001" ixy="0" ixz="0" iyy="0.001" iyz="0" izz="0.001"/>
       </inertial>
     </link>
@@ -21,5 +21,5 @@
         <mass value="0.01"/>
         <origin xyz="0 0 0"/>
-        <inertia ixx="0.000001" ixy="0" ixz="0" iyy="0.000001" iyz="0" izz="0.000001"/>
+        <inertia ixx="0.0001" ixy="0" ixz="0" iyy="0.0001" iyz="0" izz="0.0001"/>
       </inertial>
     </link>
@@ -30,5 +30,5 @@
         <origin xyz="0 0 0"/>
         <!-- solid cylinder -->
-        <inertia izz="0.000011925" ixy="0" ixz="0" iyy="0.00011505" iyz="0" ixx="0.00011505"/>
+        <inertia ixx="0.011505" izz="0.0011925" ixy="0" ixz="0" iyy="0.011505" iyz="0"/>
       </inertial>
       <!-- begin simple shape approximation of f0 -->
@@ -92,5 +92,5 @@
         <origin xyz="0 0 0"/>
         <!-- solid cylinder -->
-        <inertia ixx="0.00000165" ixy="0" ixz="0" iyy="0.00001316975" iyz="0" izz="0.00001316975"/>
+        <inertia ixx="0.000165" ixy="0" ixz="0" iyy="0.001316975" iyz="0" izz="0.001316975"/>
       </inertial>
       <!-- begin simple shape approximation of f1 -->
@@ -138,5 +138,5 @@
         <mass value="0.01"/>
         <origin xyz="0 0 0"/>
-        <inertia ixx="0.000001" ixy="0" ixz="0" iyy="0.000001" iyz="0" izz="0.000001"/>
+        <inertia ixx="0.0001" ixy="0" ixz="0" iyy="0.0001" iyz="0" izz="0.0001"/>
       </inertial>
     </link>
@@ -147,5 +147,5 @@
         <origin xyz="0 0 0"/>
         <!-- solid cylinder -->
-        <inertia ixx="0.0000013365" ixy="0" ixz="0" iyy="0.000009603" iyz="0" izz="0.000009603"/>
+        <inertia ixx="0.00013365" ixy="0" ixz="0" iyy="0.0009603" iyz="0" izz="0.0009603"/>
       </inertial>
       <!-- begin simple shape approximation of f2 -->
@@ -207,5 +207,5 @@
         <mass value="0.01"/>
         <origin xyz="0 0 0"/>
-        <inertia ixx="0.000001" ixy="0" ixz="0" iyy="0.000001" iyz="0" izz="0.000001"/>
+        <inertia ixx="0.0001" ixy="0" ixz="0" iyy="0.0001" iyz="0" izz="0.0001"/>
       </inertial>
     </link>
@@ -221,5 +221,5 @@
       <limit lower="-${M_pi/2}" upper="${M_pi/2}" effort="1" velocity="1"/>
       <safety_controller soft_lower_limit="${-1.57079-10.0}" soft_upper_limit="${1.57079+10.0}" k_position="1000.0" k_velocity="1000.0"/>
-      <dynamics damping="0.2"/>
+      <dynamics damping="0.01"/>
       <origin xyz="0 0 0" rpy="0 0 0"/>
     </joint>
@@ -230,5 +230,5 @@
       <limit lower="-${M_pi/2}" upper="${M_pi/2}" effort="1" velocity="1"/>
       <safety_controller soft_lower_limit="${-1.57079-10.0}" soft_upper_limit="${1.57079+10.0}" k_position="1000.0" k_velocity="1000.0"/>
-      <dynamics damping="0.2"/>
+      <dynamics damping="0.01"/>
       <origin xyz="0.028 0 0" rpy="${M_pi/2} 0 0"/>
     </joint>
@@ -239,5 +239,5 @@
       <origin xyz="0.05 0 0" rpy="0 0 0"/>
       <safety_controller soft_lower_limit="${-1.57079-10.0}" soft_upper_limit="${1.57079+10.0}" k_position="1000.0" k_velocity="1000.0"/>
-      <dynamics damping="0.2"/>
+      <dynamics damping="0.01"/>
       <limit lower="-${M_pi/2}" upper="${M_pi/2}" effort="1" velocity="1"/>
     </joint>
@@ -257,4 +257,5 @@
       <origin xyz="0.04 0 0" rpy="-${M_pi/2} 0 0"/>
     </joint>
+    <xacro:finger_gazebo side="${side}" idx="${idx}"/>
     <xacro:finger_transmission side="${side}" idx="${idx}" x="${x}" y="${y}" z="${z}" r="${r}" p="${p}" yaw="${yaw}"/>
   </xacro:macro>

Commit message: add urdf cfmDamping option.  load xacro macros for gazebo elements for hand.

File: ros/sandia_hand_description/urdf/sandia_hand.gazebo.xacro (robot description, xacro)
@@ -9,4 +9,5 @@
       <kd>1.0</kd>
       <maxVel>0.1</maxVel>
+      <minDepth>0.0</minDepth>
       <minDepth>0.0</minDepth>
     </gazebo>
@@ -35,6 +36,21 @@
       <minDepth>0.0</minDepth>
     </gazebo>
+    <gazebo reference="${side}_f${idx}_j0">
+      <cfmDamping>1</cfmDamping>
+    </gazebo>
+    <gazebo reference="${side}_f${idx}_j1">
+      <cfmDamping>1</cfmDamping>
+    </gazebo>
+    <gazebo reference="${side}_f${idx}_j2">
+      <cfmDamping>1</cfmDamping>
+    </gazebo>
   </xacro:macro>
   <xacro:macro name="sandia_hand_gazebo" params="side">
+    <gazebo reference="${side}_palm">
+      <mu1>0.9</mu1>
+      <mu2>0.9</mu2>
+    </gazebo>
+  </xacro:macro>
+  <xacro:macro name="sandia_hand_gazebo_controller" params="side">
     <gazebo>
       <plugin filename="libgazebo_ros_controller_manager.so" name="gazebo_ros_controller_manager">
@@ -43,8 +59,4 @@
       </plugin>
     </gazebo>
-    <gazebo reference="${side}_palm">
-      <mu1>0.9</mu1>
-      <mu2>0.9</mu2>
-    </gazebo>
   </xacro:macro>
 </robot>

File: ros/sandia_hand_description/urdf/sandia_hand.urdf.xacro (robot description, xacro)
@@ -154,4 +154,5 @@
     </joint>
     <xacro:finger_transmission side="${side}" idx="${idx}" x="${x}" y="${y}" z="${z}" r="${r}" p="${p}" yaw="${yaw}"/>
+    <xacro:finger_gazebo side="${side}" idx="${idx}"/>
   </xacro:macro>
   <xacro:macro name="sandia_hand" params="side parent *origin">
@@ -189,6 +190,7 @@
     <xacro:finger side="${side}" idx="3" x="0.03995" y="-0.04383" z="0.014" r="0" p="-1.57079" yaw="-2.3562"/>
     <!-- not needed unless simulating the hand by itself
+    <xacro:sandia_hand_gazebo_controller side="${side}" />
+    -->
     <xacro:sandia_hand_gazebo side="${side}" />
-    -->
   </xacro:macro>
 </robot>

File: ros/sandia_hand_description/urdf/sandia_hand_simple_shapes.urdf.xacro (robot description, xacro)
@@ -258,4 +258,5 @@
     </joint>
     <xacro:finger_transmission side="${side}" idx="${idx}" x="${x}" y="${y}" z="${z}" r="${r}" p="${p}" yaw="${yaw}"/>
+    <xacro:finger_gazebo side="${side}" idx="${idx}"/>
   </xacro:macro>
   <xacro:macro name="sandia_hand" params="side parent reflect *origin">

Commit message: Start adding cameras to hands, currently only works for left hand

File: ros/sandia_hand_description/urdf/sandia_hand.gazebo.xacro (robot description, xacro)
@@ -51,4 +51,116 @@
     </gazebo>
   </xacro:macro>
+  <!-- begin cameras -->
+  <xacro:property name="M_pi" value="3.1415926535897931" />
+  <!-- the following properties are used to adjust the camera location -->
+  <!-- theta specifies the inclination of the stereo axis -->
+  <!-- sin_theta and cos_theta are manually entered since xacro doesn't do trig -->
+  <xacro:property name="theta" value="0.6708" />
+  <xacro:property name="sin_theta" value="0.62161284558" />
+  <xacro:property name="cos_theta" value="0.78332462632" />
+  <!-- stereo offset of 40 mm -->
+  <xacro:property name="stereo_offset" value="0.04" />
+  <!-- cam_d1 and cam_L1 are lengths that adjust the camera position -->
+  <xacro:property name="cam_d1" value="0.1" />
+  <xacro:property name="cam_L1" value="0.07" />
+  <xacro:macro name="sandia_hand_cameras_gazebo" params="side">
+    <joint name="left_camera_frame_joint" type="fixed">
+      <origin xyz="${cam_L1*sin_theta} ${-cam_d1+cam_L1*cos_theta} 0.025"
+              rpy="${-theta} -${M_pi/2} ${M_pi}"/>
+      <parent link="${side}_palm"/>
+      <child link="left_camera_frame"/>
+    </joint>
+    <link name="left_camera_frame">
+      <inertial>
+        <mass value="0.01"/>
+        <origin xyz="0 0 0"/>
+        <inertia ixx="0.0001" ixy="0.0" ixz="0.0" iyy="0.0001" iyz="0.0" izz="0.0001"/>
+      </inertial>
+      <visual group="default">
+        <origin xyz="0 0 0" rpy="0 0 0"/>
+        <geometry>
+          <box size="0.003 0.010 0.007" />
+        </geometry>
+      </visual>
+    </link>
+    <joint name="left_camera_optical_frame_joint" type="fixed">
+      <origin rpy="${-M_pi/2} 0.0 ${-M_pi/2}" xyz="0 0 0"/>
+      <parent link="left_camera_frame"/>
+      <child link="left_camera_optical_frame"/>
+    </joint>
+    <link name="left_camera_optical_frame"/>
+    <gazebo reference="left_camera_frame">
+      <sensor name="stereo_camera" type="multicamera">
+        <update_rate>60.0</update_rate>
+        <camera name="left">
+          <!-- 72 degrees -->
+          <horizontal_fov>${72 * M_pi / 180}</horizontal_fov>
+          <image>
+            <width>752</width>
+            <height>480</height>
+            <format>L_INT8</format>
+          </image>
+          <clip>
+            <near>0.02</near>
+            <far>100</far>
+          </clip>
+        </camera>
+        <camera name="right">
+          <pose>0 ${stereo_offset} 0  0 0 0</pose>
+          <!-- 72 degrees -->
+          <horizontal_fov>${72 * M_pi / 180}</horizontal_fov>
+          <image>
+            <width>752</width>
+            <height>480</height>
+            <format>L_INT8</format>
+          </image>
+          <clip>
+            <near>0.02</near>
+            <far>100</far>
+          </clip>
+        </camera>
+        <plugin filename="libgazebo_ros_multicamera.so" name="stereo_camera_controller">
+          <alwaysOn>true</alwaysOn>
+          <updateRate>0.0</updateRate>
+          <cameraName>sandia_hand/${side}_hand/camera</cameraName>
+          <imageTopicName>image_raw</imageTopicName>
+          <cameraInfoTopicName>camera_info</cameraInfoTopicName>
+          <frameName>left_camera_optical_frame</frameName>
+          <hackBaseline>0.07</hackBaseline>
+          <distortionK1>0.0</distortionK1>
+          <distortionK2>0.0</distortionK2>
+          <distortionK3>0.0</distortionK3>
+          <distortionT1>0.0</distortionT1>
+          <distortionT2>0.0</distortionT2>
+        </plugin>
+      </sensor>
+    </gazebo>
+    <joint name="right_camera_frame_joint" type="fixed">
+      <origin xyz="${(cam_L1+stereo_offset)*sin_theta} ${-cam_d1+(cam_L1+stereo_offset)*cos_theta} 0.025"
+              rpy="${-theta} -${M_pi/2} ${M_pi}"/>
+      <parent link="${side}_palm"/>
+      <child link="right_camera_frame"/>
+    </joint>
+    <link name="right_camera_frame">
+      <inertial>
+        <mass value="0.01"/>
+        <origin xyz="0 0 0"/>
+        <inertia ixx="0.0001" ixy="0.0" ixz="0.0" iyy="0.0001" iyz="0.0" izz="0.0001"/>
+      </inertial>
+      <visual group="default">
+        <origin xyz="0 0 0" rpy="0 0 0"/>
+        <geometry>
+          <box size="0.003 0.010 0.007" />
+        </geometry>
+      </visual>
+    </link>
+    <joint name="right_camera_optical_frame_joint" type="fixed">
+      <origin rpy="${-M_pi/2} 0.0 ${-M_pi/2}" xyz="0 0 0"/>
+      <parent link="right_camera_frame"/>
+      <child link="right_camera_optical_frame"/>
+    </joint>
+    <link name="right_camera_optical_frame"/>
+  </xacro:macro>
+  <!-- end cameras -->
   <xacro:macro name="sandia_hand_gazebo_controller" params="side">
     <gazebo>

File: ros/sandia_hand_description/urdf/sandia_hand_simple_shapes.urdf.xacro (robot description, xacro)
@@ -411,4 +411,5 @@
     -->
     <xacro:sandia_hand_gazebo side="${side}" />
+    <xacro:sandia_hand_cameras_gazebo side="${side}" />
   </xacro:macro>
 </robot>

Commit message: add reflect tag to cameras xacro

File: ros/sandia_hand_description/urdf/sandia_hand.gazebo.xacro (robot description, xacro)
@@ -64,8 +64,8 @@
   <xacro:property name="cam_d1" value="0.1" />
   <xacro:property name="cam_L1" value="0.07" />
-  <xacro:macro name="sandia_hand_cameras_gazebo" params="side">
+  <xacro:macro name="sandia_hand_cameras_gazebo" params="side reflect">
     <joint name="left_camera_frame_joint" type="fixed">
-      <origin xyz="${cam_L1*sin_theta} ${-cam_d1+cam_L1*cos_theta} 0.025"
-              rpy="${-theta} -${M_pi/2} ${M_pi}"/>
+      <origin xyz="${cam_L1*sin_theta} ${reflect*cam_d1 - reflect*cam_L1*cos_theta} 0.025"
+              rpy="${reflect*theta} -${M_pi/2} ${M_pi}"/>
       <parent link="${side}_palm"/>
       <child link="left_camera_frame"/>

File: ros/sandia_hand_description/urdf/sandia_hand_simple_shapes.urdf.xacro (robot description, xacro)
@@ -411,5 +411,5 @@
     -->
     <xacro:sandia_hand_gazebo side="${side}" />
-    <xacro:sandia_hand_cameras_gazebo side="${side}" />
+    <xacro:sandia_hand_cameras_gazebo side="${side}" reflect="${reflect}" />
   </xacro:macro>
 </robot>

Commit message: Split stereo_offset between left and right cameras

File: ros/sandia_hand_description/urdf/sandia_hand.gazebo.xacro (robot description, xacro)
@@ -63,9 +63,9 @@
   <!-- cam_d1 and cam_L1 are lengths that adjust the camera position -->
   <xacro:property name="cam_d1" value="0.1" />
-  <xacro:property name="cam_L1" value="0.07" />
+  <xacro:property name="cam_L1" value="0.09" />
   <xacro:macro name="sandia_hand_cameras_gazebo" params="side reflect">
     <joint name="left_camera_frame_joint" type="fixed">
-      <origin xyz="${cam_L1*sin_theta} ${reflect*cam_d1 - reflect*cam_L1*cos_theta} 0.025"
-              rpy="${reflect*theta} -${M_pi/2} ${M_pi}"/>
+      <origin xyz="${(cam_L1-stereo_offset/2)*sin_theta} ${cam_d1 - (cam_L1-stereo_offset/2)*cos_theta} 0.025"
+              rpy="${theta} -${M_pi/2} ${M_pi}"/>
       <parent link="${side}_palm"/>
       <child link="left_camera_frame"/>
@@ -137,5 +137,5 @@
     </gazebo>
     <joint name="right_camera_frame_joint" type="fixed">
-      <origin xyz="${(cam_L1+stereo_offset)*sin_theta} ${-cam_d1+(cam_L1+stereo_offset)*cos_theta} 0.025"
+      <origin xyz="${(cam_L1+stereo_offset/2)*sin_theta} ${-cam_d1+(cam_L1+stereo_offset/2)*cos_theta} 0.025"
               rpy="${-theta} -${M_pi/2} ${M_pi}"/>
       <parent link="${side}_palm"/>

Commit message: Reflect stereo camera location and angle

File: ros/sandia_hand_description/urdf/sandia_hand.gazebo.xacro (robot description, xacro)
@@ -66,6 +66,6 @@
   <xacro:macro name="sandia_hand_cameras_gazebo" params="side reflect">
     <joint name="left_camera_frame_joint" type="fixed">
-      <origin xyz="${(cam_L1-stereo_offset/2)*sin_theta} ${cam_d1 - (cam_L1-stereo_offset/2)*cos_theta} 0.025"
-              rpy="${theta} -${M_pi/2} ${M_pi}"/>
+      <origin xyz="${(cam_L1+reflect*stereo_offset/2)*sin_theta} ${cam_d1 - (cam_L1+reflect*stereo_offset/2)*cos_theta} 0.025"
+              rpy="${-reflect*theta} -${M_pi/2} ${M_pi}"/>
       <parent link="${side}_palm"/>
       <child link="left_camera_frame"/>
@@ -137,6 +137,6 @@
     </gazebo>
     <joint name="right_camera_frame_joint" type="fixed">
-      <origin xyz="${(cam_L1+stereo_offset/2)*sin_theta} ${-cam_d1+(cam_L1+stereo_offset/2)*cos_theta} 0.025"
-              rpy="${-theta} -${M_pi/2} ${M_pi}"/>
+      <origin xyz="${(cam_L1-reflect*stereo_offset/2)*sin_theta} ${-cam_d1+(cam_L1-reflect*stereo_offset/2)*cos_theta} 0.025"
+              rpy="${reflect*theta} -${M_pi/2} ${M_pi}"/>
       <parent link="${side}_palm"/>
       <child link="right_camera_frame"/>

Commit message: Fix camera naming conflicts and reflections

File: ros/sandia_hand_description/urdf/sandia_hand.gazebo.xacro (robot description, xacro)
@@ -65,11 +65,11 @@
   <xacro:property name="cam_L1" value="0.09" />
   <xacro:macro name="sandia_hand_cameras_gazebo" params="side reflect">
-    <joint name="left_camera_frame_joint" type="fixed">
-      <origin xyz="${(cam_L1+reflect*stereo_offset/2)*sin_theta} ${cam_d1 - (cam_L1+reflect*stereo_offset/2)*cos_theta} 0.025"
-              rpy="${-reflect*theta} -${M_pi/2} ${M_pi}"/>
+    <joint name="${side}_palm_left_camera_frame_joint" type="fixed">
+      <origin xyz="${(cam_L1+reflect*stereo_offset/2)*sin_theta} ${reflect*(cam_d1-(cam_L1+reflect*stereo_offset/2)*cos_theta)} 0.025"
+              rpy="${reflect*theta} -${M_pi/2} ${M_pi}"/>
       <parent link="${side}_palm"/>
-      <child link="left_camera_frame"/>
+      <child link="${side}_palm_left_camera_frame"/>
     </joint>
-    <link name="left_camera_frame">
+    <link name="${side}_palm_left_camera_frame">
       <inertial>
         <mass value="0.01"/>
@@ -84,12 +84,12 @@
       </visual>
     </link>
-    <joint name="left_camera_optical_frame_joint" type="fixed">
+    <joint name="${side}_palm_left_camera_optical_frame_joint" type="fixed">
       <origin rpy="${-M_pi/2} 0.0 ${-M_pi/2}" xyz="0 0 0"/>
-      <parent link="left_camera_frame"/>
-      <child link="left_camera_optical_frame"/>
+      <parent link="${side}_palm_left_camera_frame"/>
+      <child link="${side}_palm_left_camera_optical_frame"/>
     </joint>
-    <link name="left_camera_optical_frame"/>
-    <gazebo reference="left_camera_frame">
-      <sensor name="stereo_camera" type="multicamera">
+    <link name="${side}_palm_left_camera_optical_frame"/>
+    <gazebo reference="${side}_palm_left_camera_frame">
+      <sensor name="${side}_palm_stereo_camera" type="multicamera">
         <update_rate>60.0</update_rate>
         <camera name="left">
@@ -99,5 +99,5 @@
             <width>752</width>
             <height>480</height>
-            <format>L_INT8</format>
+            <format>L8</format>
           </image>
           <clip>
@@ -113,5 +113,5 @@
             <width>752</width>
             <height>480</height>
-            <format>L_INT8</format>
+            <format>L8</format>
           </image>
           <clip>
@@ -126,5 +126,5 @@
           <imageTopicName>image_raw</imageTopicName>
           <cameraInfoTopicName>camera_info</cameraInfoTopicName>
-          <frameName>left_camera_optical_frame</frameName>
+          <frameName>${side}_palm_left_camera_optical_frame</frameName>
           <hackBaseline>0.07</hackBaseline>
           <distortionK1>0.0</distortionK1>
@@ -136,11 +136,11 @@
       </sensor>
     </gazebo>
-    <joint name="right_camera_frame_joint" type="fixed">
-      <origin xyz="${(cam_L1-reflect*stereo_offset/2)*sin_theta} ${-cam_d1+(cam_L1-reflect*stereo_offset/2)*cos_theta} 0.025"
+    <joint name="${side}_palm_right_camera_frame_joint" type="fixed">
+      <origin xyz="${(cam_L1-reflect*stereo_offset/2)*sin_theta} ${reflect*(cam_d1-(cam_L1-reflect*stereo_offset/2)*cos_theta)} 0.025"
               rpy="${reflect*theta} -${M_pi/2} ${M_pi}"/>
       <parent link="${side}_palm"/>
-      <child link="right_camera_frame"/>
+      <child link="${side}_palm_right_camera_frame"/>
     </joint>
-    <link name="right_camera_frame">
+    <link name="${side}_palm_right_camera_frame">
       <inertial>
         <mass value="0.01"/>
@@ -155,10 +155,10 @@
       </visual>
     </link>
-    <joint name="right_camera_optical_frame_joint" type="fixed">
+    <joint name="${side}_palm_right_camera_optical_frame_joint" type="fixed">
       <origin rpy="${-M_pi/2} 0.0 ${-M_pi/2}" xyz="0 0 0"/>
-      <parent link="right_camera_frame"/>
-      <child link="right_camera_optical_frame"/>
+      <parent link="${side}_palm_right_camera_frame"/>
+      <child link="${side}_palm_right_camera_optical_frame"/>
     </joint>
-    <link name="right_camera_optical_frame"/>
+    <link name="${side}_palm_right_camera_optical_frame"/>
   </xacro:macro>
   <!-- end cameras -->

Commit message: Xacro-parameterize more of the sandia hand properties

File: ros/sandia_hand_description/urdf/sandia_hand.gazebo.xacro (robot description, xacro)
@@ -90,4 +90,11 @@
     </joint>
     <link name="${side}_palm_left_camera_optical_frame"/>
+    <!-- 72 degrees -->
+    <xacro:property name="horizontal_fov_degrees" value="72" />
+    <xacro:property name="image_width" value="752" />
+    <xacro:property name="image_height" value="480" />
+    <xacro:property name="image_format" value="L8" />
+    <xacro:property name="clip_near" value="0.02" />
+    <xacro:property name="clip_far" value="100" />
     <gazebo reference="${side}_palm_left_camera_frame">
       <sensor name="${side}_palm_stereo_camera" type="multicamera">
@@ -95,27 +102,26 @@
         <camera name="left">
           <!-- 72 degrees -->
-          <horizontal_fov>${72 * M_pi / 180}</horizontal_fov>
+          <horizontal_fov>${horizontal_fov_degrees * M_pi / 180}</horizontal_fov>
           <image>
-            <width>752</width>
-            <height>480</height>
-            <format>L8</format>
+            <width>${image_width}</width>
+            <height>${image_height}</height>
+            <format>${image_format}</format>
           </image>
           <clip>
-            <near>0.02</near>
-            <far>100</far>
+            <near>${clip_near}</near>
+            <far>${clip_far}</far>
           </clip>
         </camera>
         <camera name="right">
           <pose>0 ${-stereo_offset} 0  0 0 0</pose>
-          <!-- 72 degrees -->
-          <horizontal_fov>${72 * M_pi / 180}</horizontal_fov>
+          <horizontal_fov>${horizontal_fov_degrees * M_pi / 180}</horizontal_fov>
           <image>
-            <width>752</width>
-            <height>480</height>
-            <format>L8</format>
+            <width>${image_width}</width>
+            <height>${image_height}</height>
+            <format>${image_format}</format>
           </image>
           <clip>
-            <near>0.02</near>
-            <far>100</far>
+            <near>${clip_near}</near>
+            <far>${clip_far}</far>
           </clip>
         </camera>
