Commit message: Add gaussian noise to sandia hand cameras

File: ros/sandia_hand_description/urdf/sandia_hand.gazebo.xacro (robot description, xacro)
@@ -97,9 +97,17 @@
     <xacro:property name="clip_near" value="0.02" />
     <xacro:property name="clip_far" value="100" />
+    <!-- Noise is sampled independently per pixel on each frame.
+         That pixel's noise value is added to each of its color
+         channels, which at that point lie in the range [0,1].
+         The stddev value of 0.007 is based on experimental data
+         from a camera in a Sandia hand pointed at a static scene
+         in a couple of different lighting conditions.  -->
+    <xacro:property name="noise_type" value="gaussian" />
+    <xacro:property name="noise_mean" value="0.0" />
+    <xacro:property name="noise_stddev" value="0.007" />
     <gazebo reference="${side}_palm_left_camera_frame">
       <sensor name="${side}_palm_stereo_camera" type="multicamera">
         <update_rate>60.0</update_rate>
         <camera name="left">
-          <!-- 72 degrees -->
           <horizontal_fov>${horizontal_fov_degrees * M_pi / 180}</horizontal_fov>
           <image>
@@ -112,4 +120,9 @@
             <far>${clip_far}</far>
           </clip>
+          <noise>
+            <type>${noise_type}</type>
+            <mean>${noise_mean}</mean>
+            <stddev>${noise_stddev}</stddev>
+          </noise>
         </camera>
         <camera name="right">
@@ -125,4 +138,9 @@
             <far>${clip_far}</far>
           </clip>
+          <noise>
+            <type>${noise_type}</type>
+            <mean>${noise_mean}</mean>
+            <stddev>${noise_stddev}</stddev>
+          </noise>
         </camera>
         <plugin filename="libgazebo_ros_multicamera.so" name="stereo_camera_controller">

Commit message: Fix build: xacro properties cannot be defined inside a xacro macro

File: ros/sandia_hand_description/urdf/sandia_hand.gazebo.xacro (robot description, xacro)
@@ -64,4 +64,20 @@
   <xacro:property name="cam_d1" value="0.1" />
   <xacro:property name="cam_L1" value="0.09" />
+  <!-- 72 degrees -->
+  <xacro:property name="horizontal_fov_degrees" value="72.0" />
+  <xacro:property name="image_width" value="752" />
+  <xacro:property name="image_height" value="480" />
+  <xacro:property name="image_format" value="L8" />
+  <xacro:property name="clip_near" value="0.02" />
+  <xacro:property name="clip_far" value="100" />
+  <!-- Noise is sampled independently per pixel on each frame.
+       That pixel's noise value is added to each of its color
+       channels, which at that point lie in the range [0,1].
+       The stddev value of 0.007 is based on experimental data
+       from a camera in a Sandia hand pointed at a static scene
+       in a couple of different lighting conditions.  -->
+  <xacro:property name="noise_type" value="gaussian" />
+  <xacro:property name="noise_mean" value="0.0" />
+  <xacro:property name="noise_stddev" value="0.007" />
   <xacro:macro name="sandia_hand_cameras_gazebo" params="side reflect parent">
     <joint name="${side}_palm_left_camera_frame_joint" type="fixed">
@@ -90,20 +106,4 @@
     </joint>
     <link name="${side}_palm_left_camera_optical_frame"/>
-    <!-- 72 degrees -->
-    <xacro:property name="horizontal_fov_degrees" value="72" />
-    <xacro:property name="image_width" value="752" />
-    <xacro:property name="image_height" value="480" />
-    <xacro:property name="image_format" value="L8" />
-    <xacro:property name="clip_near" value="0.02" />
-    <xacro:property name="clip_far" value="100" />
-    <!-- Noise is sampled independently per pixel on each frame.
-         That pixel's noise value is added to each of its color
-         channels, which at that point lie in the range [0,1].
-         The stddev value of 0.007 is based on experimental data
-         from a camera in a Sandia hand pointed at a static scene
-         in a couple of different lighting conditions.  -->
-    <xacro:property name="noise_type" value="gaussian" />
-    <xacro:property name="noise_mean" value="0.0" />
-    <xacro:property name="noise_stddev" value="0.007" />
     <gazebo reference="${side}_palm_left_camera_frame">
       <sensor name="${side}_palm_stereo_camera" type="multicamera">

Commit message: Test adding contact sensors to palm and fingers

File: ros/sandia_hand_description/urdf/sandia_hand.gazebo.xacro (robot description, xacro)
@@ -195,3 +195,31 @@
     </gazebo>
   </xacro:macro>
+  <xacro:macro name="finger_tactile_sensors_gazebo" params="side idx">
+    <gazebo reference="${side}_f${idx}_1">
+      <sensor name="${side}_f${idx}_tactile" type="contact">
+        <update_rate>30.0</update_rate>
+        <contact>
+          <collision>${side}_f${idx}_1_collision</collision>
+        </contact>
+      </sensor>
+    </gazebo>
+    <gazebo reference="${side}_f${idx}_2">
+      <sensor name="${side}_f${idx}_tactile" type="contact">
+        <update_rate>30.0</update_rate>
+        <contact>
+          <collision>${side}_f${idx}_2_collision</collision>
+        </contact>
+      </sensor>
+    </gazebo>
+  </xacro:macro>
+  <xacro:macro name="sandia_hand_tactile_sensors_gazebo" params="side">
+    <gazebo reference="${side}_palm">
+      <sensor name="${side}_palm_tactile" type="contact">
+        <update_rate>30.0</update_rate>
+        <contact>
+          <collision>${side}_palm_collision</collision>
+        </contact>
+      </sensor>
+    </gazebo>
+  </xacro:macro>
 </robot>

File: ros/sandia_hand_description/urdf/sandia_hand_simple_shapes.urdf.xacro (robot description, xacro)
@@ -263,4 +263,5 @@
     <xacro:finger_transmission side="${side}" idx="${idx}" x="${x}" y="${y}" z="${z}" r="${r}" p="${p}" yaw="${yaw}"/>
     <xacro:finger_gazebo side="${side}" idx="${idx}"/>
+    <xacro:finger_tactile_sensors_gazebo side="${side}" idx="${idx}" />
   </xacro:macro>
   <!--
@@ -425,4 +426,5 @@
     <xacro:sandia_hand_gazebo side="${side}" />
     <xacro:sandia_hand_cameras_gazebo side="${side}" reflect="${reflect}" parent="${parent}" />
+    <xacro:sandia_hand_tactile_sensors_gazebo side="${side}" />
   </xacro:macro>
 </robot>

Commit message: Remove sensor and use plugin

File: ros/sandia_hand_description/urdf/sandia_hand.gazebo.xacro (robot description, xacro)
@@ -46,5 +46,6 @@
   </xacro:macro>
   <xacro:macro name="sandia_hand_gazebo" params="side">
-    <gazebo reference="${side}_palm">
+<!--    <gazebo reference="${side}_palm">-->
+    <gazebo reference="sandia_hand">
       <mu1>0.9</mu1>
       <mu2>0.9</mu2>
@@ -195,5 +196,5 @@
     </gazebo>
   </xacro:macro>
-  <xacro:macro name="finger_tactile_sensors_gazebo" params="side idx">
+<!--  <xacro:macro name="finger_tactile_sensors_gazebo" params="side idx">
     <gazebo reference="${side}_f${idx}_1">
       <sensor name="${side}_f${idx}_tactile" type="contact">
@@ -212,13 +213,34 @@
       </sensor>
     </gazebo>
-  </xacro:macro>
-  <xacro:macro name="sandia_hand_tactile_sensors_gazebo" params="side">
-    <gazebo reference="${side}_palm">
-      <sensor name="${side}_palm_tactile" type="contact">
+  </xacro:macro>-->
+  <xacro:macro name="sandia_hand_tactile_sensors_gazebo" params="side" >
+    <gazebo>
+<!--      <sensor name="${side}_tactile" type="contact">
         <update_rate>30.0</update_rate>
         <contact>
           <collision>${side}_palm_collision</collision>
-        </contact>
-      </sensor>
+          <collision>${side}_f1_1_collision</collision>
+          <collision>${side}_f1_2_collision</collision>
+          <collision>${side}_f2_1_collision</collision>
+          <collision>${side}_f2_2_collision</collision>
+          <collision>${side}_f3_1_collision</collision>
+          <collision>${side}_f3_2_collision</collision>
+        </contact>
+        <plugin filename="libContactPlugin.so" name="sandia_contact_plugin">
+          <alwaysOn>true</alwaysOn>
+          <updateRate>0.0</updateRate>
+        </plugin>
+      </sensor>-->
+      <plugin filename="libContactPlugin.so" name="sandia_contact_plugin">
+         <contact>
+          <collision>${side}_palm::${side}_palm_collision</collision>
+          <collision>${side}_f1_1::${side}_f1_1_collision</collision>
+          <collision>${side}_f1_2::${side}_f1_2_collision</collision>
+          <collision>${side}_f2_1::${side}_f2_1_collision</collision>
+          <collision>${side}_f2_2::${side}_f2_2_collision</collision>
+          <collision>${side}_f3_1::${side}_f3_1_collision</collision>
+          <collision>${side}_f3_2::${side}_f3_2_collision</collision>
+        </contact>
+      </plugin>
     </gazebo>
   </xacro:macro>

File: ros/sandia_hand_description/urdf/sandia_hand_simple_shapes.urdf.xacro (robot description, xacro)
@@ -263,5 +263,5 @@
     <xacro:finger_transmission side="${side}" idx="${idx}" x="${x}" y="${y}" z="${z}" r="${r}" p="${p}" yaw="${yaw}"/>
     <xacro:finger_gazebo side="${side}" idx="${idx}"/>
-    <xacro:finger_tactile_sensors_gazebo side="${side}" idx="${idx}" />
+<!--    <xacro:finger_tactile_sensors_gazebo side="${side}" idx="${idx}" />-->
   </xacro:macro>
   <!--

Commit message: Fix palm collision names

File: ros/sandia_hand_description/urdf/sandia_hand.gazebo.xacro (robot description, xacro)
@@ -196,43 +196,15 @@
     </gazebo>
   </xacro:macro>
-<!--  <xacro:macro name="finger_tactile_sensors_gazebo" params="side idx">
-    <gazebo reference="${side}_f${idx}_1">
-      <sensor name="${side}_f${idx}_tactile" type="contact">
-        <update_rate>30.0</update_rate>
-        <contact>
-          <collision>${side}_f${idx}_1_collision</collision>
-        </contact>
-      </sensor>
-    </gazebo>
-    <gazebo reference="${side}_f${idx}_2">
-      <sensor name="${side}_f${idx}_tactile" type="contact">
-        <update_rate>30.0</update_rate>
-        <contact>
-          <collision>${side}_f${idx}_2_collision</collision>
-        </contact>
-      </sensor>
-    </gazebo>
-  </xacro:macro>-->
-  <xacro:macro name="sandia_hand_tactile_sensors_gazebo" params="side" >
+  <xacro:macro name="sandia_hand_tactile_sensors_gazebo" params="side parent" >
     <gazebo>
-<!--      <sensor name="${side}_tactile" type="contact">
-        <update_rate>30.0</update_rate>
-        <contact>
-          <collision>${side}_palm_collision</collision>
-          <collision>${side}_f1_1_collision</collision>
-          <collision>${side}_f1_2_collision</collision>
-          <collision>${side}_f2_1_collision</collision>
-          <collision>${side}_f2_2_collision</collision>
-          <collision>${side}_f3_1_collision</collision>
-          <collision>${side}_f3_2_collision</collision>
-        </contact>
-        <plugin filename="libContactPlugin.so" name="sandia_contact_plugin">
-          <alwaysOn>true</alwaysOn>
-          <updateRate>0.0</updateRate>
-        </plugin>
-      </sensor>-->
       <plugin filename="libContactPlugin.so" name="sandia_contact_plugin">
          <contact>
-          <collision>${side}_palm::${side}_palm_collision</collision>
+          <collision>${parent}::${parent}_collision_${side}_palm</collision>
+          <collision>${parent}::${parent}_collision_${side}_palm_1</collision>
+          <collision>${parent}::${parent}_collision_${side}_palm_3</collision>
+          <collision>${parent}::${parent}_collision_${side}_palm_4</collision>
+          <collision>${parent}::${parent}_collision_${side}_palm_5</collision>
+          <collision>${side}_f0_1::${side}_f0_1_collision</collision>
+          <collision>${side}_f0_2::${side}_f0_2_collision</collision>
           <collision>${side}_f1_1::${side}_f1_1_collision</collision>
           <collision>${side}_f1_2::${side}_f1_2_collision</collision>

File: ros/sandia_hand_description/urdf/sandia_hand_simple_shapes.urdf.xacro (robot description, xacro)
@@ -426,5 +426,5 @@
     <xacro:sandia_hand_gazebo side="${side}" />
     <xacro:sandia_hand_cameras_gazebo side="${side}" reflect="${reflect}" parent="${parent}" />
-    <xacro:sandia_hand_tactile_sensors_gazebo side="${side}" />
+    <xacro:sandia_hand_tactile_sensors_gazebo side="${side}" parent="${parent}" />
   </xacro:macro>
 </robot>

Commit message: tuning sim contact parameters.

File: ros/sandia_hand_description/urdf/sandia_hand.gazebo.xacro (robot description, xacro)
@@ -9,29 +9,32 @@
       <kd>1.0</kd>
       <maxVel>0.1</maxVel>
-      <minDepth>0.0</minDepth>
+      <minDepth>0.001</minDepth>
     </gazebo>
     <gazebo reference="${side}_f${idx}_0">
       <mu1>0.9</mu1>
       <mu2>0.9</mu2>
-      <kp>1000000000.0</kp>
-      <kd>1.0</kd>
-      <maxVel>0.1</maxVel>
-      <minDepth>0.0</minDepth>
+      <kp>1000000.0</kp>
+      <kd>1.0</kd>
+      <maxVel>0.0</maxVel>
+      <minDepth>0.003</minDepth>
+      <maxContacts>1</maxContacts>
     </gazebo>
     <gazebo reference="${side}_f${idx}_1">
       <mu1>0.9</mu1>
       <mu2>0.9</mu2>
-      <kp>1000000000.0</kp>
-      <kd>1.0</kd>
-      <maxVel>1.0</maxVel>
-      <minDepth>0.0</minDepth>
+      <kp>1000000.0</kp>
+      <kd>1.0</kd>
+      <maxVel>0.0</maxVel>
+      <minDepth>0.003</minDepth>
+      <maxContacts>1</maxContacts>
     </gazebo>
     <gazebo reference="${side}_f${idx}_2">
       <mu1>0.9</mu1>
       <mu2>0.9</mu2>
-      <kp>1000000000.0</kp>
-      <kd>1.0</kd>
-      <maxVel>1.0</maxVel>
-      <minDepth>0.0</minDepth>
+      <kp>1000000.0</kp>
+      <kd>1.0</kd>
+      <maxVel>0.0</maxVel>
+      <minDepth>0.003</minDepth>
+      <maxContacts>1</maxContacts>
     </gazebo>
     <gazebo reference="${side}_f${idx}_j0">

File: ros/sandia_hand_description/urdf/sandia_hand_simple_shapes.urdf.xacro (robot description, xacro)
@@ -8,5 +8,5 @@
   <xacro:property name="damping_coefficient_j1" value="30" />
   <xacro:property name="damping_coefficient_j2" value="30" />
-  <xacro:property name="velocity_limit" value="100" />
+  <xacro:property name="velocity_limit" value="-1" />
   <xacro:macro name="finger" params="idx x y z r p yaw side reflect">
     <link name="${side}_f${idx}_base">

Commit message: Add imu sensor xacro

File: ros/sandia_hand_description/urdf/sandia_hand.gazebo.xacro (robot description, xacro)
@@ -217,3 +217,28 @@
     </gazebo>
   </xacro:macro>
+  <xacro:macro name="sandia_hand_imu_sensor_gazebo" params="parent" >
+  <gazebo reference="${parent}">
+    <sensor name="imu_sensor" type="imu">
+      <always_on>1</always_on>
+      <update_rate>1000.0</update_rate>
+      <imu>
+        <noise>
+          <type>gaussian</type>
+          <rate>
+            <mean>0.0</mean>
+            <stddev>2e-4</stddev>
+            <bias_mean>0.0000075</bias_mean>
+            <bias_stddev>0.0000008</bias_stddev>
+          </rate>
+          <accel>
+            <mean>0.0</mean>
+            <stddev>1.7e-2</stddev>
+            <bias_mean>0.1</bias_mean>
+            <bias_stddev>0.001</bias_stddev>
+          </accel>
+        </noise>
+      </imu>
+    </sensor>
+  </gazebo>
+  </xacro:macro>
 </robot>

File: ros/sandia_hand_description/urdf/sandia_hand_simple_shapes.urdf.xacro (robot description, xacro)
@@ -418,4 +418,5 @@
     <xacro:sandia_hand_cameras_gazebo side="${side}" reflect="${reflect}" parent="${parent}" />
     <xacro:sandia_hand_tactile_sensors_gazebo side="${side}" parent="${parent}" />
+    <xacro:sandia_hand_imu_sensor_gazebo parent="${parent}" />
   </xacro:macro>
 </robot>

Commit message: FlatBlack for sim visual.

File: ros/sandia_hand_description/urdf/sandia_hand.gazebo.xacro (robot description, xacro)
@@ -10,4 +10,5 @@
       <maxVel>0.1</maxVel>
       <minDepth>0.001</minDepth>
+      <material>Gazebo/FlatBlack</material>
     </gazebo>
     <gazebo reference="${side}_f${idx}_0">
@@ -19,4 +20,5 @@
       <minDepth>0.003</minDepth>
       <maxContacts>1</maxContacts>
+      <material>Gazebo/FlatBlack</material>
     </gazebo>
     <gazebo reference="${side}_f${idx}_1">
@@ -28,4 +30,5 @@
       <minDepth>0.003</minDepth>
       <maxContacts>1</maxContacts>
+      <material>Gazebo/FlatBlack</material>
     </gazebo>
     <gazebo reference="${side}_f${idx}_2">
@@ -37,4 +40,5 @@
       <minDepth>0.003</minDepth>
       <maxContacts>1</maxContacts>
+      <material>Gazebo/FlatBlack</material>
     </gazebo>
     <gazebo reference="${side}_f${idx}_j0">
@@ -52,4 +56,5 @@
       <mu1>0.9</mu1>
       <mu2>0.9</mu2>
+      <material>Gazebo/FlatBlack</material>
     </gazebo>
   </xacro:macro>

Commit message: reduce damping to 2 Nms / rad.

File: ros/sandia_hand_description/urdf/sandia_hand.gazebo.xacro (robot description, xacro)
@@ -6,5 +6,5 @@
       <mu1>0.9</mu1>
       <mu2>0.9</mu2>
-      <kp>1000000000.0</kp>
+      <kp>1000000.0</kp>
       <kd>1.0</kd>
       <maxVel>0.1</maxVel>
@@ -17,5 +17,5 @@
       <kp>1000000.0</kp>
       <kd>1.0</kd>
-      <maxVel>0.0</maxVel>
+      <maxVel>0.1</maxVel>
       <minDepth>0.003</minDepth>
       <maxContacts>1</maxContacts>
@@ -27,5 +27,5 @@
       <kp>1000000.0</kp>
       <kd>1.0</kd>
-      <maxVel>0.0</maxVel>
+      <maxVel>0.1</maxVel>
       <minDepth>0.003</minDepth>
       <maxContacts>1</maxContacts>
@@ -37,5 +37,5 @@
       <kp>1000000.0</kp>
       <kd>1.0</kd>
-      <maxVel>0.0</maxVel>
+      <maxVel>0.1</maxVel>
       <minDepth>0.003</minDepth>
       <maxContacts>1</maxContacts>

File: ros/sandia_hand_description/urdf/sandia_hand_simple_shapes.urdf.xacro (robot description, xacro)
@@ -5,7 +5,7 @@
   <include filename="$(find sandia_hand_description)/urdf/sandia_hand.transmission.xacro" />
   <xacro:property name="M_pi" value="3.1415926535897931" />
-  <xacro:property name="damping_coefficient_j0" value="-2.5" />
-  <xacro:property name="damping_coefficient_j1" value="-2.5" />
-  <xacro:property name="damping_coefficient_j2" value="-2.5" />
+  <xacro:property name="damping_coefficient_j0" value="2.0" />
+  <xacro:property name="damping_coefficient_j1" value="2.0" />
+  <xacro:property name="damping_coefficient_j2" value="2.0" />
   <xacro:property name="velocity_limit" value="-1" />
   <xacro:macro name="finger" params="idx x y z r p yaw side reflect">

Commit message: Add soft high friction collision shapes to palm and finger tips

File: ros/sandia_hand_description/urdf/sandia_hand.gazebo.xacro (robot description, xacro)
@@ -42,4 +42,12 @@
       <material>Gazebo/FlatBlack</material>
     </gazebo>
+    <gazebo reference="${side}_f${idx}_2_soft">
+      <mu1>11</mu1>
+      <mu2>11</mu2>
+      <material>Gazebo/FlatBlack</material>
+      <maxContacts>1</maxContacts>
+      <kp>1500</kp>
+      <kd>1</kd>
+    </gazebo>
     <gazebo reference="${side}_f${idx}_j0">
       <cfmDamping>1</cfmDamping>
@@ -56,5 +64,13 @@
       <mu1>0.9</mu1>
       <mu2>0.9</mu2>
-      <material>Gazebo/FlatBlack</material>
+      <minDepth>0.001</minDepth>
+      <material>Gazebo/FlatBlack</material>
+    </gazebo>
+    <gazebo reference="${side}_palm_soft">
+      <mu1>11</mu1>
+      <mu2>11</mu2>
+      <material>Gazebo/FlatBlack</material>
+      <kp>1500</kp>
+      <kd>1</kd>
     </gazebo>
   </xacro:macro>

File: ros/sandia_hand_description/urdf/sandia_hand_simple_shapes.urdf.xacro (robot description, xacro)
@@ -214,4 +214,32 @@
       </inertial>
     </link>
+    <link name="${side}_f${idx}_2_soft">
+      <collision group="default">
+        <origin xyz="0.024 0 0" rpy="0 ${M_pi/2} 0"/>
+        <geometry>
+          <cylinder radius="0.014" length="0.057" />
+        </geometry>
+      </collision>
+      <collision group="other">
+        <origin xyz="0.052 0 0" rpy="0 0 0"/>
+        <geometry>
+          <sphere radius="0.014" />
+        </geometry>
+      </collision>
+      <!--
+      <visual>
+        <origin xyz="0.024 0 0" rpy="0 ${M_pi/2} 0"/>
+        <geometry>
+          <cylinder radius="0.014" length="0.057" />
+        </geometry>
+      </visual>
+      <visual>
+        <origin xyz="0.052 0 0" rpy="0 0 0"/>
+        <geometry>
+          <sphere radius="0.014" />
+        </geometry>
+      </visual>
+      -->
+    </link>
     <joint name="${side}_f${idx}_base" type="fixed">
       <parent link="${side}_palm"/>
@@ -261,4 +289,9 @@
       <origin xyz="0.04 0 0" rpy="-${M_pi/2} 0 0"/>
     </joint>
+    <joint name="${side}_f${idx}_2_soft" type="fixed">
+      <parent link="${side}_f${idx}_2"/>
+      <child link="${side}_f${idx}_2_soft"/>
+      <origin xyz="0 0 0" rpy="0 0 0"/>
+    </joint>
     <xacro:finger_transmission side="${side}" idx="${idx}" x="${x}" y="${y}" z="${z}" r="${r}" p="${p}" yaw="${yaw}"/>
     <xacro:finger_gazebo side="${side}" idx="${idx}"/>
@@ -402,4 +435,35 @@
       <!-   end visual mesh of f2 -->
     </link>
+    <link name="${side}_palm_soft">
+      <collision group="other">
+        <origin xyz="0.069 ${0.016 * reflect} 0.038" rpy="0 ${M_pi/2} ${-0.9 * reflect}"/>
+        <geometry>
+          <cylinder radius="0.018" length="0.100" />
+        </geometry>
+      </collision>
+      <collision group="other">
+        <origin xyz="0.11 ${-0.01*reflect} -0.005" rpy="0 0 ${0.37*reflect}"/>
+        <geometry>
+          <box size="0.09 .03 .07" />
+        </geometry>
+      </collision>
+      <collision group="other">
+        <origin xyz="0.09 ${0.02*reflect} -0.005" rpy="0 0 ${0.37*reflect}"/>
+        <geometry>
+          <box size="0.09 .03 .07" />
+        </geometry>
+      </collision>
+      <collision group="other">
+        <origin xyz="0.060 ${0.050*reflect} -0.005" rpy="0 0 ${0.37*reflect}"/>
+        <geometry>
+          <box size="0.09 .03 .07" />
+        </geometry>
+      </collision>
+    </link>
+    <joint name="${side}_palm_soft_joint" type="fixed">
+      <origin xyz="0 0 0" rpy="0 0 0"/>
+      <parent link="${side}_palm"/>
+      <child link="${side}_palm_soft"/>
+    </joint>
     <joint name="${side}_sandia_hand_joint" type="fixed">
       <parent link="${parent}"/>
