Commit message: Removed collision and visual groups

File: ros/sandia_hand_description/urdf/sandia_hand.gazebo.xacro (robot description, xacro)
@@ -107,5 +107,5 @@
         <inertia ixx="0.0001" ixy="0.0" ixz="0.0" iyy="0.0001" iyz="0.0" izz="0.0001"/>
       </inertial>
-      <visual group="default">
+      <visual>
         <origin xyz="0 0 0" rpy="0 0 0"/>
         <geometry>
@@ -186,5 +186,5 @@
         <inertia ixx="0.0001" ixy="0.0" ixz="0.0" iyy="0.0001" iyz="0.0" izz="0.0001"/>
       </inertial>
-      <visual group="default">
+      <visual>
         <origin xyz="0 0 0" rpy="0 0 0"/>
         <geometry>

File: ros/sandia_hand_description/urdf/sandia_hand_simple_shapes.urdf.xacro (robot description, xacro)
@@ -37,5 +37,5 @@
       </inertial>
       <!-- begin simple shape approximation of f0 -->
-      <collision group="default">
+      <collision"default">
         <origin xyz="0 0 0.003" rpy="0 0 0"/>
         <geometry>
@@ -43,5 +43,5 @@
         </geometry>
       </collision>
-      <collision group="other">
+      <collision"other">
         <origin xyz="0.011 0 0.003" rpy="${M_pi/2} 0 0"/>
         <geometry>
@@ -71,5 +71,5 @@
       <!--   end visual shape approximation of f0 -->
       <!-- begin collision mesh of f0 ->
-      <collision group="default">
+      <collision"default">
         <origin xyz="0 0 0" rpy="0 0 0"/>
         <geometry>
@@ -99,5 +99,5 @@
       </inertial>
       <!-- begin simple shape approximation of f1 -->
-      <collision group="default">
+      <collision"default">
         <origin xyz="0.024 0 0" rpy="0 ${M_pi/2} 0"/>
         <geometry>
@@ -118,5 +118,5 @@
       <!--   end visual shape approximation of f1 -->
       <!-- begin collision mesh of f1 ->
-      <collision group="default">
+      <collision"default">
         <origin xyz="0 0 0" rpy="0 0 0"/>
         <geometry>
@@ -154,5 +154,5 @@
       </inertial>
       <!-- begin simple shape approximation of f2 -->
-      <collision group="default">
+      <collision"default">
         <origin xyz="0.024 0 0" rpy="0 ${M_pi/2} 0"/>
         <geometry>
@@ -160,5 +160,5 @@
         </geometry>
       </collision>
-      <collision group="other">
+      <collision"other">
         <origin xyz="0.052 0 0" rpy="0 0 0"/>
         <geometry>
@@ -187,5 +187,5 @@
       </visual>
       <!-- begin collision mesh of f2    ->
-      <collision group="default">
+      <collision"default">
         <origin xyz="0 0 0" rpy="0 0 0"/>
         <geometry>
@@ -274,5 +274,5 @@
       </inertial>
       <!-- begin simple shape approximation of palm -->
-      <collision group="default">
+      <collision"default">
         <origin xyz="0.069 ${0.016 * reflect} 0.038" rpy="0 ${M_pi/2} ${-0.9 * reflect}"/>
         <geometry>
@@ -280,5 +280,5 @@
         </geometry>
       </collision>
-      <collision group="other">
+      <collision"other">
         <origin xyz="0.064 ${0.008 * reflect} 0.021" rpy="${0.41 * reflect} 0 ${-0.9 * reflect}"/>
         <geometry>
@@ -286,5 +286,5 @@
         </geometry>
       </collision>
-      <collision group="other">
+      <collision"other">
         <origin xyz="0.02 0 -0.005" rpy="0 ${M_pi/2} 0"/>
         <geometry>
@@ -292,5 +292,5 @@
         </geometry>
       </collision>
-      <collision group="other">
+      <collision"other">
         <origin xyz="0.11 ${-0.01*reflect} -0.005" rpy="0 0 ${0.37*reflect}"/>
         <geometry>
@@ -298,5 +298,5 @@
         </geometry>
       </collision>
-      <collision group="other">
+      <collision"other">
         <origin xyz="0.09 ${0.02*reflect} -0.005" rpy="0 0 ${0.37*reflect}"/>
         <geometry>
@@ -304,5 +304,5 @@
         </geometry>
       </collision>
-      <collision group="other">
+      <collision"other">
         <origin xyz="0.060 ${0.050*reflect} -0.005" rpy="0 0 ${0.37*reflect}"/>
         <geometry>
@@ -310,5 +310,5 @@
         </geometry>
       </collision>
-      <collision group="other">
+      <collision"other">
         <origin xyz="0.044 ${-0.04*reflect} -0.005" rpy="0 0 ${0.79*reflect}"/>
         <geometry>
@@ -383,5 +383,5 @@
       <!--   end visual shape approximation of palm -->
       <!-- begin collision mesh of f2 ->
-      <collision group="default">
+      <collision"default">
         <origin xyz="0 0 0" rpy="0 0 0"/>
         <geometry>

Commit message: revert visual group name

File: ros/sandia_hand_description/urdf/sandia_hand.gazebo.xacro (robot description, xacro)
@@ -107,5 +107,5 @@
         <inertia ixx="0.0001" ixy="0.0" ixz="0.0" iyy="0.0001" iyz="0.0" izz="0.0001"/>
       </inertial>
-      <visual>
+      <visual group="default">
         <origin xyz="0 0 0" rpy="0 0 0"/>
         <geometry>
@@ -186,5 +186,5 @@
         <inertia ixx="0.0001" ixy="0.0" ixz="0.0" iyy="0.0001" iyz="0.0" izz="0.0001"/>
       </inertial>
-      <visual>
+      <visual group="default">
         <origin xyz="0 0 0" rpy="0 0 0"/>
         <geometry>
